File: Page 8.sch (KiCad schematic (older format))
At the start: 14 parts

Commit message: Updates
Parts:
- R801, R802, R803, R804, R805: value R22 -> 22K0
- R806: renamed from R906; value R22K0 -> 22K0; Manufacturer (none) -> TE Connectivity
- TP801: renamed from TP901; value TP_SPI_MISO -> TestPoint; symbol Connector:TestPoint -> Name~Plate~Class~Library:TestPoint; Name (none) -> TP_LCD_SPI_MISO
- TP802: renamed from TP902; value TP_FONT_nSELECT -> Test Point; Name (none) -> TP_FONT_nSELECT
- TP803: renamed from TP903; value TP_SPI_CLK -> Test Point; Name (none) -> TP_SPI_CLK
- TP804: renamed from TP904; value TP_SPI_MOSI -> Test Point; Name (none) -> TP_SPI_MOSI
- TP805: renamed from TP905; value TP_DC -> Test Point; Name (none) -> TP_DC
- TP806: renamed from TP906; value TP_LCD_nCS -> Test Point; Name (none) -> TP_LCD_nCS
Changed lines of the file:
@@
 LCD_nCS
 $Comp
-L Connector:TestPoint TP906
+L Connector:TestPoint TP806
 U 1 1 5EB10897
 P 3500 5550
-F 0 "TP906" H 3300 5850 50  0000 L CNN
-F 1 "TP_LCD_nCS" H 3300 5750 50  0000 L CNN
+F 0 "TP806" H 3300 5850 50  0000 L CNN
+F 1 "Test Point" H 3300 5750 50  0000 L CNN
 F 2 "Connector_Wire:SolderWirePad_1x01_SMD_5x10mm" H 3700 5550 50  0001 C CNN
-F 3 "~" H 3700 5550 50  0001 C CNN
+F 3 "None" H 3700 5550 50  0001 C CNN
+F 4 "TP_LCD_nCS" H 3500 5550 50  0001 C CNN "Name"
 	1    3500 5550
 	1    0    0    -1
@@
 AR Path="/5EAC05C2/5EB1088F" Ref="R?"  Part="1"
 AR Path="/5EACA483/5EB1088F" Ref="R?"  Part="1"
-AR Path="/5ECF32A9/5EB1088F" Ref="R906"  Part="1"
-F 0 "R906" V 4000 5650 50  0000 R CNN
-F 1 "R22K0" V 3800 5650 50  0000 R CNN
+AR Path="/5ECF32A9/5EB1088F" Ref="R806"  Part="1"
+F 0 "R806" V 4000 5650 50  0000 R CNN
+F 1 "22K0" V 3800 5650 50  0000 R CNN
 F 2 "Resistor_SMD:R_0603_1608Metric_Pad1.05x0.95mm_HandSolder" V 3830 5550 50  0001 C CNN
 F 3 "https://www.te.com/commerce/DocumentDelivery/DDEController?Action=srchrtrv&DocNm=1773204-3&DocType=DS&DocLang=English" H 3900 5550 50  0001 C CNN
+F 4 "TE Connectivity " H 3900 5550 50  0001 C CNN "Manufacturer"
 	1    3900 5550
 	0    -1   -1   0
 $EndComp
 $Comp
-L Connector:TestPoint TP905
+L Connector:TestPoint TP805
 U 1 1 5EB0F64B
 P 3500 4900
-F 0 "TP905" H 3300 5200 50  0000 L CNN
-F 1 "TP_DC" H 3300 5100 50  0000 L CNN
+F 0 "TP805" H 3300 5200 50  0000 L CNN
+F 1 "Test Point" H 3300 5100 50  0000 L CNN
 F 2 "Connector_Wire:SolderWirePad_1x01_SMD_5x10mm" H 3700 4900 50  0001 C CNN
-F 3 "~" H 3700 4900 50  0001 C CNN
+F 3 "None" H 3700 4900 50  0001 C CNN
+F 4 "TP_DC" H 3500 4900 50  0001 C CNN "Name"
 	1    3500 4900
 	1    0    0    -1
@@
 AR Path="/5ECF32A9/5EB0F643" Ref="R805"  Part="1"
 F 0 "R805" V 4000 5000 50  0000 R CNN
-F 1 "R22" V 3800 5000 50  0000 R CNN
+F 1 "22K0" V 3800 5000 50  0000 R CNN
 F 2 "Resistor_SMD:R_0603_1608Metric_Pad1.05x0.95mm_HandSolder" V 3830 4900 50  0001 C CNN
 F 3 "https://www.te.com/commerce/DocumentDelivery/DDEController?Action=srchrtrv&DocNm=1773204-3&DocType=DS&DocLang=English" H 3900 4900 50  0001 C CNN
@@
 $EndComp
 $Comp
-L Connector:TestPoint TP904
+L Connector:TestPoint TP804
 U 1 1 5EB078C9
 P 3500 4250
-F 0 "TP904" H 3300 4550 50  0000 L CNN
-F 1 "TP_SPI_MOSI" H 3300 4450 50  0000 L CNN
+F 0 "TP804" H 3300 4550 50  0000 L CNN
+F 1 "Test Point" H 3300 4450 50  0000 L CNN
 F 2 "Connector_Wire:SolderWirePad_1x01_SMD_5x10mm" H 3700 4250 50  0001 C CNN
-F 3 "~" H 3700 4250 50  0001 C CNN
+F 3 "None" H 3700 4250 50  0001 C CNN
+F 4 "TP_SPI_MOSI" H 3500 4250 50  0001 C CNN "Name"
 	1    3500 4250
 	1    0    0    -1
@@
 AR Path="/5ECF32A9/5EB078C1" Ref="R804"  Part="1"
 F 0 "R804" V 4000 4350 50  0000 R CNN
-F 1 "R22" V 3800 4350 50  0000 R CNN
+F 1 "22K0" V 3800 4350 50  0000 R CNN
 F 2 "Resistor_SMD:R_0603_1608Metric_Pad1.05x0.95mm_HandSolder" V 3830 4250 50  0001 C CNN
 F 3 "https://www.te.com/commerce/DocumentDelivery/DDEController?Action=srchrtrv&DocNm=1773204-3&DocType=DS&DocLang=English" H 3900 4250 50  0001 C CNN
@@
 $EndComp
 $Comp
-L Connector:TestPoint TP903
+L Connector:TestPoint TP803
 U 1 1 5EB06A11
 P 3500 3600
-F 0 "TP903" H 3300 3900 50  0000 L CNN
-F 1 "TP_SPI_CLK" H 3300 3800 50  0000 L CNN
+F 0 "TP803" H 3300 3900 50  0000 L CNN
+F 1 "Test Point" H 3300 3800 50  0000 L CNN
 F 2 "Connector_Wire:SolderWirePad_1x01_SMD_5x10mm" H 3700 3600 50  0001 C CNN
-F 3 "~" H 3700 3600 50  0001 C CNN
+F 3 "None" H 3700 3600 50  0001 C CNN
+F 4 "TP_SPI_CLK" H 3500 3600 50  0001 C CNN "Name"
 	1    3500 3600
 	1    0    0    -1
@@
 AR Path="/5ECF32A9/5EB06A09" Ref="R803"  Part="1"
 F 0 "R803" V 4000 3700 50  0000 R CNN
-F 1 "R22" V 3800 3700 50  0000 R CNN
+F 1 "22K0" V 3800 3700 50  0000 R CNN
 F 2 "Resistor_SMD:R_0603_1608Metric_Pad1.05x0.95mm_HandSolder" V 3830 3600 50  0001 C CNN
 F 3 "https://www.te.com/commerce/DocumentDelivery/DDEController?Action=srchrtrv&DocNm=1773204-3&DocType=DS&DocLang=English" H 3900 3600 50  0001 C CNN
@@
 $EndComp
 $Comp
-L Connector:TestPoint TP902
+L Connector:TestPoint TP802
 U 1 1 5EB05D05
 P 3500 2950
-F 0 "TP902" H 3300 3250 50  0000 L CNN
-F 1 "TP_FONT_nSELECT" H 3300 3150 50  0000 L CNN
+F 0 "TP802" H 3300 3250 50  0000 L CNN
+F 1 "Test Point" H 3300 3150 50  0001 L CNN
 F 2 "Connector_Wire:SolderWirePad_1x01_SMD_5x10mm" H 3700 2950 50  0001 C CNN
-F 3 "~" H 3700 2950 50  0001 C CNN
+F 3 "None" H 3700 2950 50  0001 C CNN
+F 4 "TP_FONT_nSELECT" H 3300 3150 50  0000 L CNN "Name"
 	1    3500 2950
 	1    0    0    -1
@@
 AR Path="/5ECF32A9/5EB05CFD" Ref="R802"  Part="1"
 F 0 "R802" V 4000 3050 50  0000 R CNN
-F 1 "R22" V 3800 3050 50  0000 R CNN
+F 1 "22K0" V 3800 3050 50  0000 R CNN
 F 2 "Resistor_SMD:R_0603_1608Metric_Pad1.05x0.95mm_HandSolder" V 3830 2950 50  0001 C CNN
 F 3 "https://www.te.com/commerce/DocumentDelivery/DDEController?Action=srchrtrv&DocNm=1773204-3&DocType=DS&DocLang=English" H 3900 2950 50  0001 C CNN
@@
 AR Path="/5ECF32A9/5EAFACC6" Ref="R801"  Part="1"
 F 0 "R801" V 4000 2400 50  0000 R CNN
-F 1 "R22" V 3800 2400 50  0000 R CNN
+F 1 "22K0" V 3800 2400 50  0000 R CNN
 F 2 "Resistor_SMD:R_0603_1608Metric_Pad1.05x0.95mm_HandSolder" V 3830 2300 50  0001 C CNN
 F 3 "https://www.te.com/commerce/DocumentDelivery/DDEController?Action=srchrtrv&DocNm=1773204-3&DocType=DS&DocLang=English" H 3900 2300 50  0001 C CNN
@@
 $EndComp
 $Comp
-L Connector:TestPoint TP901
+L Name~Plate~Class~Library:TestPoint TP801
 U 1 1 5EB012D4
 P 3500 2300
-F 0 "TP901" H 3300 2600 50  0000 L CNN
-F 1 "TP_SPI_MISO" H 3300 2500 50  0000 L CNN
+F 0 "TP801" H 3300 2600 50  0000 L CNN
+F 1 "TestPoint" H 3400 2050 50  0001 L CNN
 F 2 "Connector_Wire:SolderWirePad_1x01_SMD_5x10mm" H 3700 2300 50  0001 C CNN
-F 3 "~" H 3700 2300 50  0001 C CNN
+F 3 "None" H 3700 2300 50  0001 C CNN
+F 4 "TP_LCD_SPI_MISO" H 3300 2500 50  0000 L CNN "Name"
 	1    3500 2300
 	1    0    0    -1

Commit message: Updates to schematic
Switching to ATMega34UF chip.
Parts:
- C801: DigiKey Part No. (none) -> 311-1335-1-ND; Manufacturer (none) -> Yageo; Mftr Part No. Yageo CC0603KPX7R7BB104 -> CC0603KPX7R7BB104
- J801: renamed from LCD1; value LCD 2.4\" -> DNP; footprint Name Plate Class Project:LCD_ER-TFTM024-3 -> Name Plate Class Project:LCD_ER-TFTM024-3_SMD; DigiKey Part No. (none) -> 0713085440-ND; Manufacturer (none) -> Molex; Mftr Part No. (none) -> 0713085440; Name (none) -> ER-TFTM024-3-2847-4SPI-3.3V-3748-2559-3304
- R801, R802, R803, R804, R805: value 22K0 -> 22; DigiKey Part No. (none) -> A130081CT-ND; Manufacturer (none) -> TE Connectivity; Mftr Part No. (none) -> CRGCQ0603J22R
- R806: value 22K0 -> 22; DigiKey Part No. (none) -> A130081CT-ND; Mftr Part No. (none) -> CRGCQ0603J22R
- TP801: value TestPoint -> Test Point; DigiKey Part No. (none) -> None; Manufacturer (none) -> None; Mftr Part No. (none) -> None
- TP802, TP803, TP804, TP805, TP806: symbol Connector:TestPoint -> Name~Plate~Class~Library:TestPoint; DigiKey Part No. (none) -> None; Manufacturer (none) -> None; Mftr Part No. (none) -> None
Changed lines of the file:
@@
 LCD_nCS
 $Comp
-L Connector:TestPoint TP806
+L Name~Plate~Class~Library:TestPoint TP806
 U 1 1 5EB10897
 P 3500 5550
 F 0 "TP806" H 3300 5850 50  0000 L CNN
-F 1 "Test Point" H 3300 5750 50  0000 L CNN
+F 1 "Test Point" H 3300 5750 50  0001 L CNN
 F 2 "Connector_Wire:SolderWirePad_1x01_SMD_5x10mm" H 3700 5550 50  0001 C CNN
 F 3 "None" H 3700 5550 50  0001 C CNN
-F 4 "TP_LCD_nCS" H 3500 5550 50  0001 C CNN "Name"
+F 4 "TP_LCD_nCS" H 3300 5750 50  0000 L CNN "Name"
+F 5 "None" H 3500 5550 50  0001 C CNN "DigiKey Part No."
+F 6 "None" H 3500 5550 50  0001 C CNN "Manufacturer"
+F 7 "None" H 3500 5550 50  0001 C CNN "Mftr Part No."
 	1    3500 5550
 	1    0    0    -1
@@
 AR Path="/5ECF32A9/5EB1088F" Ref="R806"  Part="1"
 F 0 "R806" V 4000 5650 50  0000 R CNN
-F 1 "22K0" V 3800 5650 50  0000 R CNN
+F 1 "22" V 3800 5650 50  0000 R CNN
 F 2 "Resistor_SMD:R_0603_1608Metric_Pad1.05x0.95mm_HandSolder" V 3830 5550 50  0001 C CNN
 F 3 "https://www.te.com/commerce/DocumentDelivery/DDEController?Action=srchrtrv&DocNm=1773204-3&DocType=DS&DocLang=English" H 3900 5550 50  0001 C CNN
 F 4 "TE Connectivity " H 3900 5550 50  0001 C CNN "Manufacturer"
+F 5 "CRGCQ0603J22R" H 3900 5550 50  0001 C CNN "Mftr Part No."
+F 6 "A130081CT-ND" H 3900 5550 50  0001 C CNN "DigiKey Part No."
 	1    3900 5550
 	0    -1   -1   0
 $EndComp
 $Comp
-L Connector:TestPoint TP805
+L Name~Plate~Class~Library:TestPoint TP805
 U 1 1 5EB0F64B
 P 3500 4900
 F 0 "TP805" H 3300 5200 50  0000 L CNN
-F 1 "Test Point" H 3300 5100 50  0000 L CNN
+F 1 "Test Point" H 3300 5100 50  0001 L CNN
 F 2 "Connector_Wire:SolderWirePad_1x01_SMD_5x10mm" H 3700 4900 50  0001 C CNN
 F 3 "None" H 3700 4900 50  0001 C CNN
-F 4 "TP_DC" H 3500 4900 50  0001 C CNN "Name"
+F 4 "TP_DC" H 3300 5100 50  0000 L CNN "Name"
+F 5 "None" H 3500 4900 50  0001 C CNN "DigiKey Part No."
+F 6 "None" H 3500 4900 50  0001 C CNN "Manufacturer"
+F 7 "None" H 3500 4900 50  0001 C CNN "Mftr Part No."
 	1    3500 4900
 	1    0    0    -1
@@
 AR Path="/5ECF32A9/5EB0F643" Ref="R805"  Part="1"
 F 0 "R805" V 4000 5000 50  0000 R CNN
-F 1 "22K0" V 3800 5000 50  0000 R CNN
+F 1 "22" V 3800 5000 50  0000 R CNN
 F 2 "Resistor_SMD:R_0603_1608Metric_Pad1.05x0.95mm_HandSolder" V 3830 4900 50  0001 C CNN
 F 3 "https://www.te.com/commerce/DocumentDelivery/DDEController?Action=srchrtrv&DocNm=1773204-3&DocType=DS&DocLang=English" H 3900 4900 50  0001 C CNN
+F 4 "TE Connectivity " H 3900 4900 50  0001 C CNN "Manufacturer"
+F 5 "CRGCQ0603J22R" H 3900 4900 50  0001 C CNN "Mftr Part No."
+F 6 "A130081CT-ND" H 3900 4900 50  0001 C CNN "DigiKey Part No."
 	1    3900 4900
 	0    -1   -1   0
 $EndComp
 $Comp
-L Connector:TestPoint TP804
+L Name~Plate~Class~Library:TestPoint TP804
 U 1 1 5EB078C9
 P 3500 4250
 F 0 "TP804" H 3300 4550 50  0000 L CNN
-F 1 "Test Point" H 3300 4450 50  0000 L CNN
+F 1 "Test Point" H 3300 4450 50  0001 L CNN
 F 2 "Connector_Wire:SolderWirePad_1x01_SMD_5x10mm" H 3700 4250 50  0001 C CNN
 F 3 "None" H 3700 4250 50  0001 C CNN
-F 4 "TP_SPI_MOSI" H 3500 4250 50  0001 C CNN "Name"
+F 4 "TP_SPI_MOSI" H 3300 4450 50  0000 L CNN "Name"
+F 5 "None" H 3500 4250 50  0001 C CNN "DigiKey Part No."
+F 6 "None" H 3500 4250 50  0001 C CNN "Manufacturer"
+F 7 "None" H 3500 4250 50  0001 C CNN "Mftr Part No."
 	1    3500 4250
 	1    0    0    -1
@@
 AR Path="/5ECF32A9/5EB078C1" Ref="R804"  Part="1"
 F 0 "R804" V 4000 4350 50  0000 R CNN
-F 1 "22K0" V 3800 4350 50  0000 R CNN
+F 1 "22" V 3800 4350 50  0000 R CNN
 F 2 "Resistor_SMD:R_0603_1608Metric_Pad1.05x0.95mm_HandSolder" V 3830 4250 50  0001 C CNN
 F 3 "https://www.te.com/commerce/DocumentDelivery/DDEController?Action=srchrtrv&DocNm=1773204-3&DocType=DS&DocLang=English" H 3900 4250 50  0001 C CNN
+F 4 "TE Connectivity " H 3900 4250 50  0001 C CNN "Manufacturer"
+F 5 "CRGCQ0603J22R" H 3900 4250 50  0001 C CNN "Mftr Part No."
+F 6 "A130081CT-ND" H 3900 4250 50  0001 C CNN "DigiKey Part No."
 	1    3900 4250
 	0    -1   -1   0
 $EndComp
 $Comp
-L Connector:TestPoint TP803
+L Name~Plate~Class~Library:TestPoint TP803
 U 1 1 5EB06A11
 P 3500 3600
 F 0 "TP803" H 3300 3900 50  0000 L CNN
-F 1 "Test Point" H 3300 3800 50  0000 L CNN
+F 1 "Test Point" H 3300 3800 50  0001 L CNN
 F 2 "Connector_Wire:SolderWirePad_1x01_SMD_5x10mm" H 3700 3600 50  0001 C CNN
 F 3 "None" H 3700 3600 50  0001 C CNN
-F 4 "TP_SPI_CLK" H 3500 3600 50  0001 C CNN "Name"
+F 4 "TP_SPI_CLK" H 3300 3800 50  0000 L CNN "Name"
+F 5 "None" H 3500 3600 50  0001 C CNN "DigiKey Part No."
+F 6 "None" H 3500 3600 50  0001 C CNN "Manufacturer"
+F 7 "None" H 3500 3600 50  0001 C CNN "Mftr Part No."
 	1    3500 3600
 	1    0    0    -1
@@
 AR Path="/5ECF32A9/5EB06A09" Ref="R803"  Part="1"
 F 0 "R803" V 4000 3700 50  0000 R CNN
-F 1 "22K0" V 3800 3700 50  0000 R CNN
+F 1 "22" V 3800 3700 50  0000 R CNN
 F 2 "Resistor_SMD:R_0603_1608Metric_Pad1.05x0.95mm_HandSolder" V 3830 3600 50  0001 C CNN
 F 3 "https://www.te.com/commerce/DocumentDelivery/DDEController?Action=srchrtrv&DocNm=1773204-3&DocType=DS&DocLang=English" H 3900 3600 50  0001 C CNN
+F 4 "TE Connectivity " H 3900 3600 50  0001 C CNN "Manufacturer"
+F 5 "CRGCQ0603J22R" H 3900 3600 50  0001 C CNN "Mftr Part No."
+F 6 "A130081CT-ND" H 3900 3600 50  0001 C CNN "DigiKey Part No."
 	1    3900 3600
 	0    -1   -1   0
 $EndComp
 $Comp
-L Connector:TestPoint TP802
+L Name~Plate~Class~Library:TestPoint TP802
 U 1 1 5EB05D05
 P 3500 2950
@@
 F 3 "None" H 3700 2950 50  0001 C CNN
 F 4 "TP_FONT_nSELECT" H 3300 3150 50  0000 L CNN "Name"
+F 5 "None" H 3500 2950 50  0001 C CNN "DigiKey Part No."
+F 6 "None" H 3500 2950 50  0001 C CNN "Manufacturer"
+F 7 "None" H 3500 2950 50  0001 C CNN "Mftr Part No."
 	1    3500 2950
 	1    0    0    -1
@@
 AR Path="/5ECF32A9/5EB05CFD" Ref="R802"  Part="1"
 F 0 "R802" V 4000 3050 50  0000 R CNN
-F 1 "22K0" V 3800 3050 50  0000 R CNN
+F 1 "22" V 3800 3050 50  0000 R CNN
 F 2 "Resistor_SMD:R_0603_1608Metric_Pad1.05x0.95mm_HandSolder" V 3830 2950 50  0001 C CNN
 F 3 "https://www.te.com/commerce/DocumentDelivery/DDEController?Action=srchrtrv&DocNm=1773204-3&DocType=DS&DocLang=English" H 3900 2950 50  0001 C CNN
+F 4 "TE Connectivity " H 3900 2950 50  0001 C CNN "Manufacturer"
+F 5 "CRGCQ0603J22R" H 3900 2950 50  0001 C CNN "Mftr Part No."
+F 6 "A130081CT-ND" H 3900 2950 50  0001 C CNN "DigiKey Part No."
 	1    3900 2950
 	0    -1   -1   0
@@
 AR Path="/5ECF32A9/5EAFACC6" Ref="R801"  Part="1"
 F 0 "R801" V 4000 2400 50  0000 R CNN
-F 1 "22K0" V 3800 2400 50  0000 R CNN
+F 1 "22" V 3800 2400 50  0000 R CNN
 F 2 "Resistor_SMD:R_0603_1608Metric_Pad1.05x0.95mm_HandSolder" V 3830 2300 50  0001 C CNN
 F 3 "https://www.te.com/commerce/DocumentDelivery/DDEController?Action=srchrtrv&DocNm=1773204-3&DocType=DS&DocLang=English" H 3900 2300 50  0001 C CNN
+F 4 "TE Connectivity " H 3900 2300 50  0001 C CNN "Manufacturer"
+F 5 "CRGCQ0603J22R" H 3900 2300 50  0001 C CNN "Mftr Part No."
+F 6 "A130081CT-ND" H 3900 2300 50  0001 C CNN "DigiKey Part No."
 	1    3900 2300
 	0    -1   -1   0
@@
 F 2 "Capacitor_SMD:C_0603_1608Metric_Pad1.05x0.95mm_HandSolder" H 6438 2750 50  0001 C CNN
 F 3 "https://www.yageo.com/upload/media/product/productsearch/datasheet/mlcc/UPY-GPHC_X7R_6.3V-to-50V_18.pdf" H 6400 2900 50  0001 C CNN
-F 4 "Yageo CC0603KPX7R7BB104" H 6400 2900 50  0001 C CNN "Mftr Part No."
+F 4 "CC0603KPX7R7BB104" H 6400 2900 50  0001 C CNN "Mftr Part No."
+F 5 "Yageo" H 6400 2900 50  0001 C CNN "Manufacturer"
+F 6 "311-1335-1-ND" H 6400 2900 50  0001 C CNN "DigiKey Part No."
 	1    6400 2900
 	1    0    0    -1
@@
 P 7400 3650
 AR Path="/5EAC05C2/5EB2A1E3" Ref="LCD?"  Part="1"
-AR Path="/5ECF32A9/5EB2A1E3" Ref="LCD1"  Part="1"
-F 0 "LCD1" H 6900 4750 50  0000 L BNN
-F 1 "LCD 2.4\"" H 6900 2500 50  0000 L BNN
-F 2 "Name Plate Class Project:LCD_ER-TFTM024-3" H 7400 3650 50  0001 C CNN
+AR Path="/5ECF32A9/5EB2A1E3" Ref="J801"  Part="1"
+F 0 "J801" H 6900 4750 50  0000 L BNN
+F 1 "DNP" H 6900 2500 50  0000 L BNN
+F 2 "Name Plate Class Project:LCD_ER-TFTM024-3_SMD" H 7400 3650 50  0001 C CNN
 F 3 "" H 7400 3650 50  0001 C CNN
+F 4 "0713085440-ND" H 7400 3650 50  0001 C CNN "DigiKey Part No."
+F 5 "Molex" H 7400 3650 50  0001 C CNN "Manufacturer"
+F 6 "0713085440" H 7400 3650 50  0001 C CNN "Mftr Part No."
+F 7 "ER-TFTM024-3-2847-4SPI-3.3V-3748-2559-3304" H 7400 3650 50  0001 C CNN "Name"
 	1    7400 3650
 	1    0    0    -1
@@
 P 3500 2300
 F 0 "TP801" H 3300 2600 50  0000 L CNN
-F 1 "TestPoint" H 3400 2050 50  0001 L CNN
+F 1 "Test Point" H 3400 2050 50  0001 L CNN
 F 2 "Connector_Wire:SolderWirePad_1x01_SMD_5x10mm" H 3700 2300 50  0001 C CNN
 F 3 "None" H 3700 2300 50  0001 C CNN
 F 4 "TP_LCD_SPI_MISO" H 3300 2500 50  0000 L CNN "Name"
+F 5 "None" H 3500 2300 50  0001 C CNN "DigiKey Part No."
+F 6 "None" H 3500 2300 50  0001 C CNN "Manufacturer"
+F 7 "None" H 3500 2300 50  0001 C CNN "Mftr Part No."
 	1    3500 2300
 	1    0    0    -1

Commit message: Updates
Parts:
- J801: footprint Name Plate Class Project:LCD_ER-TFTM024-3_SMD -> Name_Plate_Class_Project:LCD_ER-TFTM024-3_SMD; symbol Name~Plate~Class~Library:LCD_ER-TFTM024-3 -> Name_Plate_Class_Project:LCD_ER-TFTM024-3; Name ER-TFTM024-3-2847-4SPI-3.3V-3748-2559-3304 -> (none)
- TP801, TP802, TP803, TP804, TP805, TP806: symbol Name~Plate~Class~Library:TestPoint -> Name_Plate_Class_Project:TestPoint
Changed lines of the file:
@@
 LCD_nCS
 $Comp
-L Name~Plate~Class~Library:TestPoint TP806
+L Name_Plate_Class_Project:TestPoint TP806
 U 1 1 5EB10897
 P 3500 5550
@@
 $EndComp
 $Comp
-L Name~Plate~Class~Library:TestPoint TP805
+L Name_Plate_Class_Project:TestPoint TP805
 U 1 1 5EB0F64B
 P 3500 4900
@@
 $EndComp
 $Comp
-L Name~Plate~Class~Library:TestPoint TP804
+L Name_Plate_Class_Project:TestPoint TP804
 U 1 1 5EB078C9
 P 3500 4250
@@
 $EndComp
 $Comp
-L Name~Plate~Class~Library:TestPoint TP803
+L Name_Plate_Class_Project:TestPoint TP803
 U 1 1 5EB06A11
 P 3500 3600
@@
 $EndComp
 $Comp
-L Name~Plate~Class~Library:TestPoint TP802
+L Name_Plate_Class_Project:TestPoint TP802
 U 1 1 5EB05D05
 P 3500 2950
@@
 $EndComp
 $Comp
-L Name~Plate~Class~Library:LCD_ER-TFTM024-3 LCD?
+L Name_Plate_Class_Project:LCD_ER-TFTM024-3 LCD?
 U 1 1 5EB2A1E3
 P 7400 3650
@@
 F 0 "J801" H 6900 4750 50  0000 L BNN
 F 1 "DNP" H 6900 2500 50  0000 L BNN
-F 2 "Name Plate Class Project:LCD_ER-TFTM024-3_SMD" H 7400 3650 50  0001 C CNN
+F 2 "Name_Plate_Class_Project:LCD_ER-TFTM024-3_SMD" H 7400 3650 50  0001 C CNN
 F 3 "" H 7400 3650 50  0001 C CNN
 F 4 "0713085440-ND" H 7400 3650 50  0001 C CNN "DigiKey Part No."
 F 5 "Molex" H 7400 3650 50  0001 C CNN "Manufacturer"
 F 6 "0713085440" H 7400 3650 50  0001 C CNN "Mftr Part No."
-F 7 "ER-TFTM024-3-2847-4SPI-3.3V-3748-2559-3304" H 7400 3650 50  0001 C CNN "Name"
 	1    7400 3650
 	1    0    0    -1
 $EndComp
 $Comp
-L Name~Plate~Class~Library:TestPoint TP801
+L Name_Plate_Class_Project:TestPoint TP801
 U 1 1 5EB012D4
 P 3500 2300

Commit message: PCB Layout
Parts:
- TP801, TP802, TP803, TP804, TP805, TP806: footprint Connector_Wire:SolderWirePad_1x01_SMD_5x10mm -> FrequentlyUsed:Pad_2.5-2.5
Changed lines of the file:
@@
 F 0 "TP806" H 3300 5850 50  0000 L CNN
 F 1 "Test Point" H 3300 5750 50  0001 L CNN
-F 2 "Connector_Wire:SolderWirePad_1x01_SMD_5x10mm" H 3700 5550 50  0001 C CNN
+F 2 "FrequentlyUsed:Pad_2.5-2.5" H 3700 5550 50  0001 C CNN
 F 3 "None" H 3700 5550 50  0001 C CNN
 F 4 "TP_LCD_nCS" H 3300 5750 50  0000 L CNN "Name"
@@
 F 0 "TP805" H 3300 5200 50  0000 L CNN
 F 1 "Test Point" H 3300 5100 50  0001 L CNN
-F 2 "Connector_Wire:SolderWirePad_1x01_SMD_5x10mm" H 3700 4900 50  0001 C CNN
+F 2 "FrequentlyUsed:Pad_2.5-2.5" H 3700 4900 50  0001 C CNN
 F 3 "None" H 3700 4900 50  0001 C CNN
 F 4 "TP_DC" H 3300 5100 50  0000 L CNN "Name"
@@
 F 0 "TP804" H 3300 4550 50  0000 L CNN
 F 1 "Test Point" H 3300 4450 50  0001 L CNN
-F 2 "Connector_Wire:SolderWirePad_1x01_SMD_5x10mm" H 3700 4250 50  0001 C CNN
+F 2 "FrequentlyUsed:Pad_2.5-2.5" H 3700 4250 50  0001 C CNN
 F 3 "None" H 3700 4250 50  0001 C CNN
 F 4 "TP_SPI_MOSI" H 3300 4450 50  0000 L CNN "Name"
@@
 F 0 "TP803" H 3300 3900 50  0000 L CNN
 F 1 "Test Point" H 3300 3800 50  0001 L CNN
-F 2 "Connector_Wire:SolderWirePad_1x01_SMD_5x10mm" H 3700 3600 50  0001 C CNN
+F 2 "FrequentlyUsed:Pad_2.5-2.5" H 3700 3600 50  0001 C CNN
 F 3 "None" H 3700 3600 50  0001 C CNN
 F 4 "TP_SPI_CLK" H 3300 3800 50  0000 L CNN "Name"
@@
 F 0 "TP802" H 3300 3250 50  0000 L CNN
 F 1 "Test Point" H 3300 3150 50  0001 L CNN
-F 2 "Connector_Wire:SolderWirePad_1x01_SMD_5x10mm" H 3700 2950 50  0001 C CNN
+F 2 "FrequentlyUsed:Pad_2.5-2.5" H 3700 2950 50  0001 C CNN
 F 3 "None" H 3700 2950 50  0001 C CNN
 F 4 "TP_FONT_nSELECT" H 3300 3150 50  0000 L CNN "Name"
@@
 F 0 "TP801" H 3300 2600 50  0000 L CNN
 F 1 "Test Point" H 3400 2050 50  0001 L CNN
-F 2 "Connector_Wire:SolderWirePad_1x01_SMD_5x10mm" H 3700 2300 50  0001 C CNN
+F 2 "FrequentlyUsed:Pad_2.5-2.5" H 3700 2300 50  0001 C CNN
 F 3 "None" H 3700 2300 50  0001 C CNN
 F 4 "TP_LCD_SPI_MISO" H 3300 2500 50  0000 L CNN "Name"

Commit message: PCB Update
Connections:
- net labels added: LCD_DC_R
Changed lines of the file:
@@
 LCD_SPI_MOSI
 Text Label 8100 3900 0    50   ~ 0
-LCD_DC
+LCD_DC_R
 Text Label 8100 3800 0    50   ~ 0
 LCD_nCS
@@
 	3500 4900 3250 4900
 Text Label 4150 4900 0    50   ~ 0
-LCD_DC
+LCD_DC_R
 Wire Wire Line
 	4050 5550 4750 5550

Commit message: PCB Update
Connections:
- net labels added: LCD_nCS_R
Changed lines of the file:
@@
 LCD_DC_R
 Text Label 8100 3800 0    50   ~ 0
-LCD_nCS
+LCD_nCS_R
 Wire Wire Line
 	8000 4300 8650 4300
@@
 	3500 5550 3250 5550
 Text Label 4150 5550 0    50   ~ 0
-LCD_nCS
+LCD_nCS_R
 $Comp
 L Name_Plate_Class_Project:TestPoint TP806

Commit message: PCB Tweaks
Parts:
- J801: DigiKey Part No. 0713085440-ND -> S5690-ND; Manufacturer Molex -> Sullins Connector Solutions; Mftr Part No. 0713085440 -> NPTC202KFMS-RC
Changed lines of the file:
@@
 AR Path="/5EAC05C2/5EB2A1E3" Ref="LCD?"  Part="1"
 AR Path="/5ECF32A9/5EB2A1E3" Ref="J801"  Part="1"
+AR Path="/5ECF31FF/5EB2A1E3" Ref="J801"  Part="1"
 F 0 "J801" H 6900 4750 50  0000 L BNN
 F 1 "DNP" H 6900 2500 50  0000 L BNN
 F 2 "Name_Plate_Class_Project:LCD_ER-TFTM024-3_SMD" H 7400 3650 50  0001 C CNN
-F 3 "" H 7400 3650 50  0001 C CNN
-F 4 "0713085440-ND" H 7400 3650 50  0001 C CNN "DigiKey Part No."
-F 5 "Molex" H 7400 3650 50  0001 C CNN "Manufacturer"
-F 6 "0713085440" H 7400 3650 50  0001 C CNN "Mftr Part No."
+F 3 "https://media.digikey.com/pdf/Data%20Sheets/Sullins%20PDFs/Female_Headers.100_DS.pdf" H 7400 3650 50  0001 C CNN
+F 4 "S5690-ND" H 7400 3650 50  0001 C CNN "DigiKey Part No."
+F 5 "Sullins Connector Solutions" H 7400 3650 50  0001 C CNN "Manufacturer"
+F 6 "NPTC202KFMS-RC" H 7400 3650 50  0001 C CNN "Mftr Part No."
 	1    7400 3650
 	1    0    0    -1
