File: Page 2.sch (KiCad schematic (older format))
At the start: 0 parts

Commit message: Updates
Parts:
- added J1: Battery Connector, symbol Connector_Generic:Conn_01x02
- added S201: Battery Switch, Name Plate Class Project:Switch_JS202011SCQN, symbol Name~Plate~Class~Library:Switch_JS202011SCQN
Changed lines of the file:
@@
 Comment4 ""
 $EndDescr
+$Comp
+L Name~Plate~Class~Library:Switch_JS202011SCQN S201
+U 1 1 5EB4E9F9
+P 2850 3500
+F 0 "S201" H 3180 3546 50  0000 L CNN
+F 1 "Battery Switch" H 3180 3455 50  0000 L CNN
+F 2 "Name Plate Class Project:Switch_JS202011SCQN" H 2000 2700 50  0001 L BNN
+F 3 "https://www.ckswitches.com/media/1422/js.pdf" H 2850 3500 50  0001 L BNN
+	1    2850 3500
+	1    0    0    -1
+$EndComp
+$Comp
+L Connector_Generic:Conn_01x02 J1
+U 1 1 5EB52776
+P 1550 2650
+F 0 "J1" V 1514 2462 50  0000 R CNN
+F 1 "Battery Connector" V 1423 2462 50  0000 R CNN
+F 2 "" H 1550 2650 50  0001 C CNN
+F 3 "~" H 1550 2650 50  0001 C CNN
+	1    1550 2650
+	0    -1   -1   0
+$EndComp
 $EndSCHEMATC

Commit message: Updates
Parts:
- added C201, C203, C204: 0.1uF, Capacitor_SMD:C_0603_1608Metric_Pad1.05x0.95mm_HandSolder, symbol Device:C
- added C202, C205: 22uF, Name Plate Class Project:CAP_430X430N, symbol Device:CP1
- added Q201: BSS138, Package_TO_SOT_SMD:SOT-23, symbol Device:Q_NMOS_GSD
- added R201, R202: R100K0, Resistor_SMD:R_0603_1608Metric_Pad1.05x0.95mm_HandSolder, symbol Device:R
- added TP201: TP_SWITCH_BATTERY, Connector_Wire:SolderWirePad_1x01_SMD_5x10mm, symbol Connector:TestPoint
- added TP202: TP_5V, Connector_Wire:SolderWirePad_1x01_SMD_5x10mm, symbol Connector:TestPoint
- added U201, U?: MIC5219-5.0YM5-TR, SOT-23-5_M5_MCH, symbol Name~Plate~Class~Library:MIC5219-x.xYM5-TR
- J1: footprint (none) -> Name Plate Class Project:JST_PH_w_SolderPoints
Connections:
- net labels added: +3.3V, +5V, GND, VBUS
- wire segments 0 -> 68
- no-connect marks 0 -> 2
Other:
- moved on the sheet: J1

Commit message: Updates
Parts:
- U201: footprint SOT-23-5_M5_MCH -> Package_TO_SOT_SMD:SOT-23-5_HandSoldering
- U202: renamed from U?; footprint SOT-23-5_M5_MCH -> Package_TO_SOT_SMD:SOT-23-5_HandSoldering
Connections:
- wire segments 68 -> 73
Other:
- note added: "Power Switching and Regulators"
- moved on the sheet: J1, TP202
Changed lines of the file:
@@
 $EndComp
 $Comp
-L power:GND #PWR?
+L power:GND #PWR0103
 U 1 1 5EB54C9C
-P 1450 2950
-F 0 "#PWR?" H 1450 2700 50  0001 C CNN
-F 1 "GND" H 1455 2777 50  0000 C CNN
-F 2 "" H 1450 2950 50  0001 C CNN
-F 3 "" H 1450 2950 50  0001 C CNN
-	1    1450 2950
-	1    0    0    -1
-$EndComp
-Wire Wire Line
-	1450 2850 1450 2950
-Wire Wire Line
-	1350 2850 1350 3500
-Wire Wire Line
-	1350 3500 2150 3500
-Wire Wire Line
-	2150 3500 2150 2900
+P 1550 2950
+F 0 "#PWR0103" H 1550 2700 50  0001 C CNN
+F 1 "GND" H 1555 2777 50  0000 C CNN
+F 2 "" H 1550 2950 50  0001 C CNN
+F 3 "" H 1550 2950 50  0001 C CNN
+	1    1550 2950
+	1    0    0    -1
+$EndComp
+Wire Wire Line
+	1450 2850 1450 3500
 Wire Wire Line
 	2150 2900 2650 2900
@@
 Wire Wire Line
 	2650 4100 2150 4100
-Wire Wire Line
-	2150 4100 2150 3500
-Connection ~ 2150 3500
 $Comp
 L Connector_Generic:Conn_01x02 J1
 U 1 1 5EB52776
-P 1350 2650
-F 0 "J1" V 1550 2700 50  0000 R CNN
-F 1 "Battery Connector" V 1450 2700 50  0000 R CNN
-F 2 "Name Plate Class Project:JST_PH_w_SolderPoints" H 1350 2650 50  0001 C CNN
-F 3 "~" H 1350 2650 50  0001 C CNN
-	1    1350 2650
+P 1450 2650
+F 0 "J1" V 1650 2700 50  0000 R CNN
+F 1 "Battery Connector" V 1550 2700 50  0000 R CNN
+F 2 "Name Plate Class Project:JST_PH_w_SolderPoints" H 1450 2650 50  0001 C CNN
+F 3 "~" H 1450 2650 50  0001 C CNN
+	1    1450 2650
 	0    -1   -1   0
 $EndComp
@@
 	2850 4100 2850 4000
 Wire Wire Line
-	3150 3500 3500 3500
+	3150 3500 3350 3500
 Connection ~ 3150 3500
 Wire Wire Line
@@
 	3500 3500 4500 3500
 $Comp
-L power:GND #PWR?
+L power:GND #PWR0104
 U 1 1 5EB58CBE
 P 3750 5150
-F 0 "#PWR?" H 3750 4900 50  0001 C CNN
+F 0 "#PWR0104" H 3750 4900 50  0001 C CNN
 F 1 "GND" H 3755 4977 50  0000 C CNN
 F 2 "" H 3750 5150 50  0001 C CNN
@@
 $EndComp
 Wire Wire Line
-	4000 3150 4000 4300
+	4000 2950 4000 3050
 $Comp
 L Device:C C?
@@
 Wire Wire Line
 	3750 5000 3500 5000
-$Comp
-L Name~Plate~Class~Library:MIC5219-x.xYM5-TR U201
-U 1 1 5EB67A18
-P 5800 3700
-F 0 "U201" H 5450 4150 60  0000 L CNN
-F 1 "MIC5219-5.0YM5-TR" H 5450 4050 60  0000 L CNN
-F 2 "SOT-23-5_M5_MCH" H 5450 3300 60  0001 L CNN
-F 3 "" H 5150 3900 60  0000 C CNN
-	1    5800 3700
-	1    0    0    -1
-$EndComp
 Wire Wire Line
 	4500 4050 5250 4050
@@
 	6450 3600 6450 3700
 $Comp
-L power:GND #PWR?
+L power:GND #PWR0105
 U 1 1 5EB6D89E
 P 6450 4350
-F 0 "#PWR?" H 6450 4100 50  0001 C CNN
+F 0 "#PWR0105" H 6450 4100 50  0001 C CNN
 F 1 "GND" H 6455 4177 50  0000 C CNN
 F 2 "" H 6450 4350 50  0001 C CNN
@@
 	6450 4100 6450 4200
 Wire Wire Line
-	6250 3500 6750 3500
-$Comp
-L Name~Plate~Class~Library:MIC5219-x.xYM5-TR U?
+	6250 3500 6600 3500
+$Comp
+L Name~Plate~Class~Library:MIC5219-x.xYM5-TR U202
 U 1 1 5EB717E5
 P 8400 3700
-F 0 "U?" H 8050 4150 60  0000 L CNN
+F 0 "U202" H 8050 4150 60  0000 L CNN
 F 1 "MIC5219-5.0YM5-TR" H 8050 4050 60  0000 L CNN
-F 2 "SOT-23-5_M5_MCH" H 8050 3300 60  0001 L CNN
-F 3 "" H 7750 3900 60  0000 C CNN
+F 2 "Package_TO_SOT_SMD:SOT-23-5_HandSoldering" H 8050 3300 60  0001 L CNN
+F 3 "http://ww1.microchip.com/downloads/en/DeviceDoc/MIC5219-500mA-Peak-Output-LDO-Regulator-DS20006021A.pdf" H 7750 3900 60  0001 C CNN
 	1    8400 3700
 	1    0    0    -1
@@
 L Connector:TestPoint TP?
 U 1 1 5EB7241E
-P 6750 3500
+P 6850 3500
 AR Path="/5ECF32A9/5EB7241E" Ref="TP?"  Part="1"
 AR Path="/5EACA483/5EB7241E" Ref="TP202"  Part="1"
-F 0 "TP202" H 6700 3800 50  0000 L CNN
-F 1 "TP_5V" H 6700 3700 50  0000 L CNN
-F 2 "Connector_Wire:SolderWirePad_1x01_SMD_5x10mm" H 6950 3500 50  0001 C CNN
-F 3 "~" H 6950 3500 50  0001 C CNN
-	1    6750 3500
-	1    0    0    -1
-$EndComp
-Connection ~ 6750 3500
-Wire Wire Line
-	6750 3500 7100 3500
+F 0 "TP202" H 6800 3800 50  0000 L CNN
+F 1 "TP_5V" H 6800 3700 50  0000 L CNN
+F 2 "Connector_Wire:SolderWirePad_1x01_SMD_5x10mm" H 7050 3500 50  0001 C CNN
+F 3 "~" H 7050 3500 50  0001 C CNN
+	1    6850 3500
+	1    0    0    -1
+$EndComp
 $Comp
 L Device:CP1 C202
@@
 	9050 3600 9050 3700
 $Comp
-L power:GND #PWR?
+L power:GND #PWR0106
 U 1 1 5EB7AD53
 P 9050 4350
-F 0 "#PWR?" H 9050 4100 50  0001 C CNN
+F 0 "#PWR0106" H 9050 4100 50  0001 C CNN
 F 1 "GND" H 9055 4177 50  0000 C CNN
 F 2 "" H 9050 4350 50  0001 C CNN
@@
 	7550 3050 7550 3500
 $Comp
-L power:+5V #PWR?
+L power:+5V #PWR0107
 U 1 1 5EB765CC
 P 7550 3050
-F 0 "#PWR?" H 7550 2900 50  0001 C CNN
+F 0 "#PWR0107" H 7550 2900 50  0001 C CNN
 F 1 "+5V" H 7565 3223 50  0000 C CNN
 F 2 "" H 7550 3050 50  0001 C CNN
@@
 $EndComp
 $Comp
-L power:+3.3V #PWR?
+L power:+3.3V #PWR0108
 U 1 1 5EB828C2
 P 9700 3050
-F 0 "#PWR?" H 9700 2900 50  0001 C CNN
+F 0 "#PWR0108" H 9700 2900 50  0001 C CNN
 F 1 "+3.3V" H 9715 3223 50  0000 C CNN
 F 2 "" H 9700 3050 50  0001 C CNN
@@
 	3750 5000 3750 5150
 $Comp
-L power:VBUS #PWR?
+L power:VBUS #PWR0109
 U 1 1 5EB8783A
-P 4000 3150
-F 0 "#PWR?" H 4000 3000 50  0001 C CNN
-F 1 "VBUS" H 4015 3323 50  0000 C CNN
-F 2 "" H 4000 3150 50  0001 C CNN
-F 3 "" H 4000 3150 50  0001 C CNN
-	1    4000 3150
-	1    0    0    -1
-$EndComp
-$Comp
-L power:+5V #PWR?
-U 1 1 5EB88401
-P 4300 3100
-F 0 "#PWR?" H 4300 2950 50  0001 C CNN
-F 1 "+5V" H 4315 3273 50  0000 C CNN
-F 2 "" H 4300 3100 50  0001 C CNN
-F 3 "" H 4300 3100 50  0001 C CNN
-	1    4300 3100
-	1    0    0    -1
-$EndComp
+P 4000 2950
+F 0 "#PWR0109" H 4000 2800 50  0001 C CNN
+F 1 "VBUS" H 4015 3123 50  0000 C CNN
+F 2 "" H 4000 2950 50  0001 C CNN
+F 3 "" H 4000 2950 50  0001 C CNN
+	1    4000 2950
+	1    0    0    -1
+$EndComp
+Text Notes 4700 5650 0    98   ~ 20
+Power Switching and Regulators
+Connection ~ 6600 3500
+Connection ~ 6850 3500
+Wire Wire Line
+	6850 3500 7100 3500
+Wire Wire Line
+	6600 3500 6850 3500
+Wire Wire Line
+	6600 3050 6600 3500
+Connection ~ 4000 3050
+Wire Wire Line
+	4000 3050 4000 4300
+$Comp
+L Name~Plate~Class~Library:MIC5219-x.xYM5-TR U201
+U 1 1 5EB67A18
+P 5800 3700
+F 0 "U201" H 5450 4150 60  0000 L CNN
+F 1 "MIC5219-5.0YM5-TR" H 5450 4050 60  0000 L CNN
+F 2 "Package_TO_SOT_SMD:SOT-23-5_HandSoldering" H 5450 3300 60  0001 L CNN
+F 3 "http://ww1.microchip.com/downloads/en/DeviceDoc/MIC5219-500mA-Peak-Output-LDO-Regulator-DS20006021A.pdf" H 5150 3900 60  0001 C CNN
+	1    5800 3700
+	1    0    0    -1
+$EndComp
+Wire Wire Line
+	4000 3050 6600 3050
+Wire Wire Line
+	1550 2850 1550 2950
+$Comp
+L power:PWR_FLAG #FLG0102
+U 1 1 5ED8ACEA
+P 3350 3500
+F 0 "#FLG0102" H 3350 3575 50  0001 C CNN
+F 1 "PWR_FLAG" H 3350 3673 50  0000 C CNN
+F 2 "" H 3350 3500 50  0001 C CNN
+F 3 "~" H 3350 3500 50  0001 C CNN
+	1    3350 3500
+	1    0    0    -1
+$EndComp
+Connection ~ 3350 3500
+Wire Wire Line
+	3350 3500 3500 3500
+Wire Wire Line
+	2150 4100 2150 3500
+Wire Wire Line
+	2150 3500 2150 2900
+Connection ~ 2150 3500
+Wire Wire Line
+	1450 3500 2150 3500
 $EndSCHEMATC

Commit message: Updating to Final Revision
Parts:
- added C203: 0.1uF, Capacitor_SMD:C_0603_1608Metric_Pad1.05x0.95mm_HandSolder, symbol Device:C
- added TP203: TP_3V, Connector_Wire:SolderWirePad_1x01_SMD_5x10mm, symbol Connector:TestPoint
- C204: renamed from C205; value 22uF -> 10uF
- C205: renamed from C203; value 0.1uF -> 470pF
- C206: renamed from C204; value 0.1uF -> 470pF
- renumbered J1 to J201, R202 to R203
Connections:
- wire segments 73 -> 77
Changed lines of the file:
@@
 $Descr A4 11693 8268
 encoding utf-8
-Sheet 3 10
+Sheet 3 9
 Title ""
 Date ""
@@
 	2650 4100 2150 4100
 $Comp
-L Connector_Generic:Conn_01x02 J1
+L Connector_Generic:Conn_01x02 J201
 U 1 1 5EB52776
 P 1450 2650
-F 0 "J1" V 1650 2700 50  0000 R CNN
+F 0 "J201" V 1650 2700 50  0000 R CNN
 F 1 "Battery Connector" V 1550 2700 50  0000 R CNN
 F 2 "Name Plate Class Project:JST_PH_w_SolderPoints" H 1450 2650 50  0001 C CNN
@@
 Wire Wire Line
 	4000 2950 4000 3050
-$Comp
-L Device:C C?
-U 1 1 5EB5C47E
-P 6450 3850
-AR Path="/5EB5C47E" Ref="C?"  Part="1"
-AR Path="/5EAC05C2/5EB5C47E" Ref="C?"  Part="1"
-AR Path="/5EACA483/5EB5C47E" Ref="C203"  Part="1"
-F 0 "C203" H 6500 3950 50  0000 L BNN
-F 1 "0.1uF" H 6500 3700 50  0000 L BNN
-F 2 "Capacitor_SMD:C_0603_1608Metric_Pad1.05x0.95mm_HandSolder" H 6488 3700 50  0001 C CNN
-F 3 "https://www.yageo.com/upload/media/product/productsearch/datasheet/mlcc/UPY-GPHC_X7R_6.3V-to-50V_18.pdf" H 6450 3850 50  0001 C CNN
-F 4 "Yageo CC0603KPX7R7BB104" H 6450 3850 50  0001 C CNN "Mftr Part No."
-	1    6450 3850
-	1    0    0    -1
-$EndComp
 $Comp
 L Device:R R?
@@
 AR Path="/5EB5DD15" Ref="R?"  Part="1"
 AR Path="/5EAC05C2/5EB5DD15" Ref="R?"  Part="1"
-AR Path="/5EACA483/5EB5DD15" Ref="R202"  Part="1"
-F 0 "R202" H 4070 4746 50  0000 L CNN
+AR Path="/5EACA483/5EB5DD15" Ref="R203"  Part="1"
+F 0 "R203" H 4070 4746 50  0000 L CNN
 F 1 "R100K0" H 4070 4655 50  0000 L CNN
 F 2 "Resistor_SMD:R_0603_1608Metric_Pad1.05x0.95mm_HandSolder" V 3930 4700 50  0001 C CNN
@@
 AR Path="/5ECE9FD3/5EB74201" Ref="C?"  Part="1"
 AR Path="/5ECEA271/5EB74201" Ref="C?"  Part="1"
-F 0 "C202" H 7250 3850 50  0000 L CNN
-F 1 "22uF" H 7250 3750 50  0000 L CNN
+F 0 "C202" H 7150 3950 50  0000 L CNN
+F 1 "22uF" H 7150 3750 50  0000 L CNN
 F 2 "Name Plate Class Project:CAP_430X430N" H 7100 3850 50  0001 C CNN
 F 3 "https://media.digikey.com/pdf/Data%20Sheets/Panasonic%20Electronic%20Components/S_Series,Type_V_Rev2018.pdf" H 7100 3850 50  0001 C CNN
@@
 AR Path="/5EB7AD4B" Ref="C?"  Part="1"
 AR Path="/5EAC05C2/5EB7AD4B" Ref="C?"  Part="1"
-AR Path="/5EACA483/5EB7AD4B" Ref="C204"  Part="1"
-F 0 "C204" H 9100 3950 50  0000 L BNN
-F 1 "0.1uF" H 9100 3700 50  0000 L BNN
+AR Path="/5EACA483/5EB7AD4B" Ref="C206"  Part="1"
+F 0 "C206" H 9100 3950 50  0000 L BNN
+F 1 "470pF" H 9100 3700 50  0000 L BNN
 F 2 "Capacitor_SMD:C_0603_1608Metric_Pad1.05x0.95mm_HandSolder" H 9088 3700 50  0001 C CNN
 F 3 "https://www.yageo.com/upload/media/product/productsearch/datasheet/mlcc/UPY-GPHC_X7R_6.3V-to-50V_18.pdf" H 9050 3850 50  0001 C CNN
@@
 	9050 4100 9050 4200
 $Comp
-L Device:CP1 C205
+L Device:CP1 C204
 U 1 1 5EB7AD61
 P 9700 3850
-AR Path="/5EACA483/5EB7AD61" Ref="C205"  Part="1"
+AR Path="/5EACA483/5EB7AD61" Ref="C204"  Part="1"
 AR Path="/5ECE9FD3/5EB7AD61" Ref="C?"  Part="1"
 AR Path="/5ECEA271/5EB7AD61" Ref="C?"  Part="1"
-F 0 "C205" H 9850 3850 50  0000 L CNN
-F 1 "22uF" H 9850 3750 50  0000 L CNN
+F 0 "C204" H 9850 3850 50  0000 L CNN
+F 1 "10uF" H 9850 3750 50  0000 L CNN
 F 2 "Name Plate Class Project:CAP_430X430N" H 9700 3850 50  0001 C CNN
 F 3 "https://media.digikey.com/pdf/Data%20Sheets/Panasonic%20Electronic%20Components/S_Series,Type_V_Rev2018.pdf" H 9700 3850 50  0001 C CNN
@@
 	8900 3900 8900 4100
 Wire Wire Line
-	8850 3500 9700 3500
+	8850 3500 9300 3500
 Connection ~ 7550 3500
 Wire Wire Line
-	7550 3500 7800 3500
+	7550 3500 7650 3500
 Wire Wire Line
 	7100 3500 7550 3500
@@
 Wire Wire Line
 	1450 3500 2150 3500
+$Comp
+L Connector:TestPoint TP?
+U 1 1 5ECCF025
+P 9300 3500
+AR Path="/5ECF32A9/5ECCF025" Ref="TP?"  Part="1"
+AR Path="/5EACA483/5ECCF025" Ref="TP203"  Part="1"
+F 0 "TP203" H 9250 3800 50  0000 L CNN
+F 1 "TP_3V" H 9250 3700 50  0000 L CNN
+F 2 "Connector_Wire:SolderWirePad_1x01_SMD_5x10mm" H 9500 3500 50  0001 C CNN
+F 3 "~" H 9500 3500 50  0001 C CNN
+	1    9300 3500
+	1    0    0    -1
+$EndComp
+Connection ~ 9300 3500
+Wire Wire Line
+	9300 3500 9700 3500
+$Comp
+L Device:C C?
+U 1 1 5ECCFF91
+P 7650 3850
+AR Path="/5ECCFF91" Ref="C?"  Part="1"
+AR Path="/5EAC05C2/5ECCFF91" Ref="C?"  Part="1"
+AR Path="/5EACA483/5ECCFF91" Ref="C203"  Part="1"
+F 0 "C203" H 7700 3950 50  0000 L CNN
+F 1 "0.1uF" H 7700 3750 50  0000 L CNN
+F 2 "Capacitor_SMD:C_0603_1608Metric_Pad1.05x0.95mm_HandSolder" H 7688 3700 50  0001 C CNN
+F 3 "https://www.yageo.com/upload/media/product/productsearch/datasheet/mlcc/UPY-GPHC_X7R_6.3V-to-50V_18.pdf" H 7650 3850 50  0001 C CNN
+F 4 "Yageo CC0603KPX7R7BB104" H 7650 3850 50  0001 C CNN "Mftr Part No."
+	1    7650 3850
+	1    0    0    -1
+$EndComp
+$Comp
+L Device:C C?
+U 1 1 5EB5C47E
+P 6450 3850
+AR Path="/5EB5C47E" Ref="C?"  Part="1"
+AR Path="/5EAC05C2/5EB5C47E" Ref="C?"  Part="1"
+AR Path="/5EACA483/5EB5C47E" Ref="C205"  Part="1"
+F 0 "C205" H 6500 3950 50  0000 L CNN
+F 1 "470pF" H 6500 3750 50  0000 L CNN
+F 2 "Capacitor_SMD:C_0603_1608Metric_Pad1.05x0.95mm_HandSolder" H 6488 3700 50  0001 C CNN
+F 3 "https://www.yageo.com/upload/media/product/productsearch/datasheet/mlcc/UPY-GPHC_X7R_6.3V-to-50V_18.pdf" H 6450 3850 50  0001 C CNN
+F 4 "Yageo CC0603KPX7R7BB104" H 6450 3850 50  0001 C CNN "Mftr Part No."
+	1    6450 3850
+	1    0    0    -1
+$EndComp
+Wire Wire Line
+	7650 3700 7650 3500
+Connection ~ 7650 3500
+Wire Wire Line
+	7650 3500 7800 3500
+$Comp
+L power:GND #PWR?
+U 1 1 5ECD2699
+P 7650 4350
+F 0 "#PWR?" H 7650 4100 50  0001 C CNN
+F 1 "GND" H 7655 4177 50  0000 C CNN
+F 2 "" H 7650 4350 50  0001 C CNN
+F 3 "" H 7650 4350 50  0001 C CNN
+	1    7650 4350
+	1    0    0    -1
+$EndComp
+Wire Wire Line
+	7650 4350 7650 4000
 $EndSCHEMATC

Commit message: Updates
Parts:
- added R201: Jumper, Resistor_SMD:R_0603_1608Metric_Pad1.05x0.95mm_HandSolder, symbol Device:R
- R202: renamed from R201; value R100K0 -> 100K0; DigiKey Part No. (none) -> 311-100KGRCT-ND; Manufacturer (none) -> Yageo
- R203: value R100K0 -> 100K0; DigiKey Part No. (none) -> 311-100KGRCT-ND; Manufacturer (none) -> Yageo
- TP201: value TP_SWITCH_BATTERY -> TestPoint; symbol Connector:TestPoint -> Name~Plate~Class~Library:TestPoint; Name (none) -> TP_SWITCH_BATTERY
- TP202: value TP_5V -> Test Point; symbol Connector:TestPoint -> Name~Plate~Class~Library:TestPoint; Name (none) -> TP_5V
- TP203: value TP_3V -> Test Point; symbol Connector:TestPoint -> Name~Plate~Class~Library:TestPoint; Name (none) -> TP_3V
Connections:
- wire segments 77 -> 78
Changed lines of the file:
@@
 AR Path="/5EB5D504" Ref="R?"  Part="1"
 AR Path="/5EAC05C2/5EB5D504" Ref="R?"  Part="1"
-AR Path="/5EACA483/5EB5D504" Ref="R201"  Part="1"
-F 0 "R201" H 4570 3846 50  0000 L CNN
-F 1 "R100K0" H 4570 3755 50  0000 L CNN
+AR Path="/5EACA483/5EB5D504" Ref="R202"  Part="1"
+F 0 "R202" H 4570 3846 50  0000 L CNN
+F 1 "100K0" H 4570 3755 50  0000 L CNN
 F 2 "Resistor_SMD:R_0603_1608Metric_Pad1.05x0.95mm_HandSolder" V 4430 3800 50  0001 C CNN
 F 3 "https://www.yageo.com/upload/media/product/productsearch/datasheet/rchip/PYu-RC_Group_51_RoHS_L_10.pdf" H 4500 3800 50  0001 C CNN
+F 4 "311-100KGRCT-ND" H 4500 3800 50  0001 C CNN "DigiKey Part No."
+F 5 "Yageo" H 4500 3800 50  0001 C CNN "Manufacturer"
 	1    4500 3800
 	1    0    0    1
@@
 AR Path="/5EACA483/5EB5DD15" Ref="R203"  Part="1"
 F 0 "R203" H 4070 4746 50  0000 L CNN
-F 1 "R100K0" H 4070 4655 50  0000 L CNN
+F 1 "100K0" H 4070 4655 50  0000 L CNN
 F 2 "Resistor_SMD:R_0603_1608Metric_Pad1.05x0.95mm_HandSolder" V 3930 4700 50  0001 C CNN
 F 3 "https://www.yageo.com/upload/media/product/productsearch/datasheet/rchip/PYu-RC_Group_51_RoHS_L_10.pdf" H 4000 4700 50  0001 C CNN
+F 4 "311-100KGRCT-ND" H 4000 4700 50  0001 C CNN "DigiKey Part No."
+F 5 "Yageo" H 4000 4700 50  0001 C CNN "Manufacturer"
 	1    4000 4700
 	1    0    0    -1
@@
 	4500 4050 4500 4100
 $Comp
-L Connector:TestPoint TP?
+L Name~Plate~Class~Library:TestPoint TP?
 U 1 1 5EB6B8BD
 P 5250 4050
@@
 AR Path="/5EACA483/5EB6B8BD" Ref="TP201"  Part="1"
 F 0 "TP201" H 5300 4300 50  0000 R CNN
-F 1 "TP_SWITCH_BATTERY" H 5300 4400 50  0000 R CNN
+F 1 "TestPoint" H 5300 4400 50  0000 R CNN
 F 2 "Connector_Wire:SolderWirePad_1x01_SMD_5x10mm" H 5450 4050 50  0001 C CNN
-F 3 "~" H 5450 4050 50  0001 C CNN
+F 3 "None" H 5450 4050 50  0001 C CNN
+F 4 "TP_SWITCH_BATTERY" H 5250 4050 50  0001 C CNN "Name"
 	1    5250 4050
 	-1   0    0    1
@@
 $EndComp
 $Comp
-L Connector:TestPoint TP?
+L Name~Plate~Class~Library:TestPoint TP?
 U 1 1 5EB7241E
 P 6850 3500
@@
 AR Path="/5EACA483/5EB7241E" Ref="TP202"  Part="1"
 F 0 "TP202" H 6800 3800 50  0000 L CNN
-F 1 "TP_5V" H 6800 3700 50  0000 L CNN
+F 1 "Test Point" H 6800 3700 50  0001 L CNN
 F 2 "Connector_Wire:SolderWirePad_1x01_SMD_5x10mm" H 7050 3500 50  0001 C CNN
-F 3 "~" H 7050 3500 50  0001 C CNN
+F 3 "None" H 7050 3500 50  0001 C CNN
+F 4 "TP_5V" H 6800 3700 50  0000 L CNN "Name"
 	1    6850 3500
 	1    0    0    -1
@@
 $EndComp
 Wire Wire Line
-	4000 3050 6600 3050
+	4000 3050 6200 3050
 Wire Wire Line
 	1550 2850 1550 2950
@@
 	1450 3500 2150 3500
 $Comp
-L Connector:TestPoint TP?
+L Name~Plate~Class~Library:TestPoint TP?
 U 1 1 5ECCF025
 P 9300 3500
@@
 AR Path="/5EACA483/5ECCF025" Ref="TP203"  Part="1"
 F 0 "TP203" H 9250 3800 50  0000 L CNN
-F 1 "TP_3V" H 9250 3700 50  0000 L CNN
+F 1 "Test Point" H 9250 3700 50  0001 L CNN
 F 2 "Connector_Wire:SolderWirePad_1x01_SMD_5x10mm" H 9500 3500 50  0001 C CNN
-F 3 "~" H 9500 3500 50  0001 C CNN
+F 3 "None" H 9500 3500 50  0001 C CNN
+F 4 "TP_3V" H 9250 3700 50  0000 L CNN "Name"
 	1    9300 3500
 	1    0    0    -1
@@
 Wire Wire Line
 	7650 4350 7650 4000
+Wire Wire Line
+	6500 3050 6600 3050
+$Comp
+L Device:R R?
+U 1 1 5EC13512
+P 6350 3050
+AR Path="/5EC13512" Ref="R?"  Part="1"
+AR Path="/5EAC05C2/5EC13512" Ref="R?"  Part="1"
+AR Path="/5EACA483/5EC13512" Ref="R201"  Part="1"
+F 0 "R201" V 6550 2950 50  0000 L CNN
+F 1 "Jumper" V 6450 2950 50  0000 L CNN
+F 2 "Resistor_SMD:R_0603_1608Metric_Pad1.05x0.95mm_HandSolder" V 6280 3050 50  0001 C CNN
+F 3 "https://www.yageo.com/upload/media/product/productsearch/datasheet/rchip/PYu-RC_Group_51_RoHS_L_10.pdf" H 6350 3050 50  0001 C CNN
+F 4 "Yageo" H 6350 3050 50  0001 C CNN "Manufacturer"
+	1    6350 3050
+	0    1    -1   0
+$EndComp
 $EndSCHEMATC
