File: Page 2.sch (KiCad schematic (older format))
At the start: 17 parts, among them J201 Battery Connector, Q201 BSS138, U201 MIC5219-5.0YM5-TR, U202 MIC5219-3.3YM5-TR

Commit message: Updates
Parts:
- C202, C204: footprint Name Plate Class Project:CAP_430X430N -> Name_Plate_Class_Project:CAP_430X430N
- J201: footprint Name Plate Class Project:JST_PH_w_SolderPoints -> Name_Plate_Class_Project:JST_PH_w_SolderPoints
- Q201: symbol Name~Plate~Class~Library:Q_NMOS_GSD -> Name_Plate_Class_Project:Q_NMOS_GSD
- S201: footprint Name Plate Class Project:Switch_JS202011SCQN -> Name_Plate_Class_Project:Switch_JS202011SCQN; symbol Name~Plate~Class~Library:Switch_JS202011SCQN -> Name_Plate_Class_Project:Switch_JS202011SCQN
- TP201, TP202, TP203: symbol Name~Plate~Class~Library:TestPoint -> Name_Plate_Class_Project:TestPoint
- U201, U202: symbol Name~Plate~Class~Library:MIC5219-x.xYM5-TR -> Name_Plate_Class_Project:MIC5219-x.xYM5-TR
Connections:
- wire segments 78 -> 75
Changed lines of the file:
@@
 $EndDescr
 $Comp
-L Name~Plate~Class~Library:Switch_JS202011SCQN S201
+L Name_Plate_Class_Project:Switch_JS202011SCQN S201
 U 1 1 5EB4E9F9
 P 2650 3500
 F 0 "S201" H 2400 4300 50  0000 L CNN
 F 1 "Battery Switch" H 2400 4200 50  0000 L CNN
-F 2 "Name Plate Class Project:Switch_JS202011SCQN" H 1800 2700 50  0001 L BNN
+F 2 "Name_Plate_Class_Project:Switch_JS202011SCQN" H 1800 2700 50  0001 L BNN
 F 3 "https://www.ckswitches.com/media/1422/js.pdf" H 2650 3500 50  0001 L BNN
 F 4 "401-2002-2-ND" H 2650 3500 50  0001 C CNN "DigiKey Part No."
@@
 F 0 "J201" V 1650 2700 50  0000 R CNN
 F 1 "Battery Connector" V 1550 2700 50  0000 R CNN
-F 2 "Name Plate Class Project:JST_PH_w_SolderPoints" H 1450 2650 50  0001 C CNN
+F 2 "Name_Plate_Class_Project:JST_PH_w_SolderPoints" H 1450 2650 50  0001 C CNN
 F 3 "http://www.jst-mfg.com/product/pdf/eng/ePH.pdf" H 1450 2650 50  0001 C CNN
 F 4 "JST Sales America Inc." H 1450 2650 50  0001 C CNN "Manufacturer"
@@
 $EndComp
 $Comp
-L Name~Plate~Class~Library:Q_NMOS_GSD Q201
+L Name_Plate_Class_Project:Q_NMOS_GSD Q201
 U 1 1 5EB6003E
 P 4400 4300
@@
 	3750 5000 3500 5000
 Wire Wire Line
-	4500 4050 5250 4050
-Wire Wire Line
 	5300 4050 5300 3600
 Wire Wire Line
@@
 	4500 4050 4500 4100
 $Comp
-L Name~Plate~Class~Library:TestPoint TP?
+L Name_Plate_Class_Project:TestPoint TP?
 U 1 1 5EB6B8BD
 P 5250 4050
 AR Path="/5ECF32A9/5EB6B8BD" Ref="TP?"  Part="1"
 AR Path="/5EACA483/5EB6B8BD" Ref="TP201"  Part="1"
+AR Path="/5EB6B8BD" Ref="TP201"  Part="1"
 F 0 "TP201" H 5300 4300 50  0000 R CNN
 F 1 "Test Point" H 5300 4400 50  0001 R CNN
@@
 	-1   0    0    1
 $EndComp
-Connection ~ 5250 4050
-Wire Wire Line
-	5250 4050 5300 4050
 Wire Wire Line
 	6250 3600 6450 3600
@@
 	6250 3500 6600 3500
 $Comp
-L Name~Plate~Class~Library:MIC5219-x.xYM5-TR U202
+L Name_Plate_Class_Project:MIC5219-x.xYM5-TR U202
 U 1 1 5EB717E5
 P 8400 3700
@@
 $EndComp
 $Comp
-L Name~Plate~Class~Library:TestPoint TP?
+L Name_Plate_Class_Project:TestPoint TP?
 U 1 1 5EB7241E
 P 6850 3500
 AR Path="/5ECF32A9/5EB7241E" Ref="TP?"  Part="1"
 AR Path="/5EACA483/5EB7241E" Ref="TP202"  Part="1"
+AR Path="/5EB7241E" Ref="TP202"  Part="1"
 F 0 "TP202" H 6800 3800 50  0000 L CNN
 F 1 "Test Point" H 6800 3700 50  0001 L CNN
@@
 F 0 "C202" H 7150 3950 50  0000 L CNN
 F 1 "10uF" H 7150 3750 50  0000 L CNN
-F 2 "Name Plate Class Project:CAP_430X430N" H 7100 3850 50  0001 C CNN
+F 2 "Name_Plate_Class_Project:CAP_430X430N" H 7100 3850 50  0001 C CNN
 F 3 "https://media.digikey.com/pdf/Data%20Sheets/Panasonic%20Electronic%20Components/S_Series,Type_V_Rev2018.pdf" H 7100 3850 50  0001 C CNN
-F 4 "" H 7100 3850 50  0001 C CNN "Field4"
-F 5 "399-11437-1-ND" H 7100 3850 50  0001 C CNN "DigiKey Part No."
-F 6 "T491A106K010AT" H 7100 3850 50  0001 C CNN "Mftr Part No."
-F 7 "" H 7100 3850 50  0001 C CNN "URL"
-F 8 "Kemet" H 7100 3850 50  0001 C CNN "Manufacturer"
+F 4 "399-11437-1-ND" H 7100 3850 50  0001 C CNN "DigiKey Part No."
+F 5 "T491A106K010AT" H 7100 3850 50  0001 C CNN "Mftr Part No."
+F 6 "Kemet" H 7100 3850 50  0001 C CNN "Manufacturer"
 	1    7100 3850
 	1    0    0    -1
@@
 F 0 "C204" H 9850 3850 50  0000 L CNN
 F 1 "10uF" H 9850 3750 50  0000 L CNN
-F 2 "Name Plate Class Project:CAP_430X430N" H 9700 3850 50  0001 C CNN
+F 2 "Name_Plate_Class_Project:CAP_430X430N" H 9700 3850 50  0001 C CNN
 F 3 "https://media.digikey.com/pdf/Data%20Sheets/Panasonic%20Electronic%20Components/S_Series,Type_V_Rev2018.pdf" H 9700 3850 50  0001 C CNN
-F 4 "" H 9700 3850 50  0001 C CNN "Field4"
-F 5 "399-11437-1-ND" H 9700 3850 50  0001 C CNN "DigiKey Part No."
-F 6 "T491A106K010AT" H 9700 3850 50  0001 C CNN "Mftr Part No."
-F 7 "" H 9700 3850 50  0001 C CNN "URL"
-F 8 "Kemet" H 9700 3850 50  0001 C CNN "Manufacturer"
+F 4 "399-11437-1-ND" H 9700 3850 50  0001 C CNN "DigiKey Part No."
+F 5 "T491A106K010AT" H 9700 3850 50  0001 C CNN "Mftr Part No."
+F 6 "Kemet" H 9700 3850 50  0001 C CNN "Manufacturer"
 	1    9700 3850
 	1    0    0    -1
@@
 Wire Wire Line
 	8900 3900 8900 4100
-Wire Wire Line
-	8850 3500 9300 3500
 Connection ~ 7550 3500
 Wire Wire Line
@@
 Power Switching and Regulators
 Connection ~ 6600 3500
-Connection ~ 6850 3500
-Wire Wire Line
-	6850 3500 7100 3500
-Wire Wire Line
-	6600 3500 6850 3500
 Wire Wire Line
 	6600 3050 6600 3500
@@
 	4000 3050 4000 4300
 $Comp
-L Name~Plate~Class~Library:MIC5219-x.xYM5-TR U201
+L Name_Plate_Class_Project:MIC5219-x.xYM5-TR U201
 U 1 1 5EB67A18
 P 5800 3700
@@
 	1450 3500 2150 3500
 $Comp
-L Name~Plate~Class~Library:TestPoint TP?
+L Name_Plate_Class_Project:TestPoint TP?
 U 1 1 5ECCF025
 P 9300 3500
 AR Path="/5ECF32A9/5ECCF025" Ref="TP?"  Part="1"
 AR Path="/5EACA483/5ECCF025" Ref="TP203"  Part="1"
+AR Path="/5ECCF025" Ref="TP203"  Part="1"
 F 0 "TP203" H 9250 3800 50  0000 L CNN
 F 1 "Test Point" H 9250 3700 50  0001 L CNN
@@
 	1    0    0    -1
 $EndComp
-Connection ~ 9300 3500
-Wire Wire Line
-	9300 3500 9700 3500
 $Comp
 L Device:C C?
@@
 	0    1    -1   0
 $EndComp
+Wire Wire Line
+	4500 4050 5300 4050
+Wire Wire Line
+	8850 3500 9700 3500
+Wire Wire Line
+	6600 3500 7100 3500
 $EndSCHEMATC

Commit message: Update Page 2.sch
Parts:
- S201: DigiKey Part No. 401-2002-2-ND -> 401-2002-1-ND
Changed lines of the file:
@@
 F 2 "Name_Plate_Class_Project:Switch_JS202011SCQN" H 1800 2700 50  0001 L BNN
 F 3 "https://www.ckswitches.com/media/1422/js.pdf" H 2650 3500 50  0001 L BNN
-F 4 "401-2002-2-ND" H 2650 3500 50  0001 C CNN "DigiKey Part No."
+F 4 "401-2002-1-ND" H 2650 3500 50  0001 C CNN "DigiKey Part No."
 F 5 "C&K" H 2650 3500 50  0001 C CNN "Manufacturer"
 F 6 "JS202011SCQN" H 2650 3500 50  0001 C CNN "Mftr Part No."

Commit message: PCB Layout
Parts:
- C202, C204: footprint Name_Plate_Class_Project:CAP_430X430N -> Name_Plate_Class_Project:T491A106K010AT; DigiKey Part No. 399-11437-1-ND -> 399-3684-1-ND
- TP201, TP202, TP203: footprint Connector_Wire:SolderWirePad_1x01_SMD_5x10mm -> FrequentlyUsed:Pad_2.5-2.5
Connections:
- net B+: now reaches J201.1 (Pin_1), S201.2, S201.5
- net BSWO: now reaches C201.1, R202.2, S201.3, S201.6, U201.1 (IN)
- net at Q201.3 (D), R202.1, U201.3 (EN): now also TP201.1
Other:
- moved on the sheet: TP201
Changed lines of the file:
@@
 L Name_Plate_Class_Project:TestPoint TP?
 U 1 1 5EB6B8BD
-P 5250 4050
+P 5200 4050
 AR Path="/5ECF32A9/5EB6B8BD" Ref="TP?"  Part="1"
 AR Path="/5EACA483/5EB6B8BD" Ref="TP201"  Part="1"
 AR Path="/5EB6B8BD" Ref="TP201"  Part="1"
-F 0 "TP201" H 5300 4300 50  0000 R CNN
-F 1 "Test Point" H 5300 4400 50  0001 R CNN
-F 2 "Connector_Wire:SolderWirePad_1x01_SMD_5x10mm" H 5450 4050 50  0001 C CNN
-F 3 "None" H 5450 4050 50  0001 C CNN
-F 4 "TP_SWITCH_BATTERY" H 5300 4400 50  0000 R CNN "Name"
-F 5 "None" H 5250 4050 50  0001 C CNN "DigiKey Part No."
-F 6 "None" H 5250 4050 50  0001 C CNN "Manufacturer"
-F 7 "None" H 5250 4050 50  0001 C CNN "Mftr Part No."
-	1    5250 4050
+F 0 "TP201" H 5250 4300 50  0000 R CNN
+F 1 "Test Point" H 5250 4400 50  0001 R CNN
+F 2 "FrequentlyUsed:Pad_2.5-2.5" H 5400 4050 50  0001 C CNN
+F 3 "None" H 5400 4050 50  0001 C CNN
+F 4 "TP_SWITCH_BATTERY" H 5250 4400 50  0000 R CNN "Name"
+F 5 "None" H 5200 4050 50  0001 C CNN "DigiKey Part No."
+F 6 "None" H 5200 4050 50  0001 C CNN "Manufacturer"
+F 7 "None" H 5200 4050 50  0001 C CNN "Mftr Part No."
+	1    5200 4050
 	-1   0    0    1
 $EndComp
@@
 F 0 "TP202" H 6800 3800 50  0000 L CNN
 F 1 "Test Point" H 6800 3700 50  0001 L CNN
-F 2 "Connector_Wire:SolderWirePad_1x01_SMD_5x10mm" H 7050 3500 50  0001 C CNN
+F 2 "FrequentlyUsed:Pad_2.5-2.5" H 7050 3500 50  0001 C CNN
 F 3 "None" H 7050 3500 50  0001 C CNN
 F 4 "TP_5V" H 6800 3700 50  0000 L CNN "Name"
@@
 F 0 "C202" H 7150 3950 50  0000 L CNN
 F 1 "10uF" H 7150 3750 50  0000 L CNN
-F 2 "Name_Plate_Class_Project:CAP_430X430N" H 7100 3850 50  0001 C CNN
-F 3 "https://media.digikey.com/pdf/Data%20Sheets/Panasonic%20Electronic%20Components/S_Series,Type_V_Rev2018.pdf" H 7100 3850 50  0001 C CNN
-F 4 "399-11437-1-ND" H 7100 3850 50  0001 C CNN "DigiKey Part No."
+F 2 "Name_Plate_Class_Project:T491A106K010AT" H 7100 3850 50  0001 C CNN
+F 3 "https://content.kemet.com/datasheets/KEM_T2005_T491.pdf" H 7100 3850 50  0001 C CNN
+F 4 "399-3684-1-ND" H 7100 3850 50  0001 C CNN "DigiKey Part No."
 F 5 "T491A106K010AT" H 7100 3850 50  0001 C CNN "Mftr Part No."
 F 6 "Kemet" H 7100 3850 50  0001 C CNN "Manufacturer"
@@
 F 0 "C204" H 9850 3850 50  0000 L CNN
 F 1 "10uF" H 9850 3750 50  0000 L CNN
-F 2 "Name_Plate_Class_Project:CAP_430X430N" H 9700 3850 50  0001 C CNN
-F 3 "https://media.digikey.com/pdf/Data%20Sheets/Panasonic%20Electronic%20Components/S_Series,Type_V_Rev2018.pdf" H 9700 3850 50  0001 C CNN
-F 4 "399-11437-1-ND" H 9700 3850 50  0001 C CNN "DigiKey Part No."
+F 2 "Name_Plate_Class_Project:T491A106K010AT" H 9700 3850 50  0001 C CNN
+F 3 "https://content.kemet.com/datasheets/KEM_T2005_T491.pdf" H 9700 3850 50  0001 C CNN
+F 4 "399-3684-1-ND" H 9700 3850 50  0001 C CNN "DigiKey Part No."
 F 5 "T491A106K010AT" H 9700 3850 50  0001 C CNN "Mftr Part No."
 F 6 "Kemet" H 9700 3850 50  0001 C CNN "Manufacturer"
@@
 F 0 "TP203" H 9250 3800 50  0000 L CNN
 F 1 "Test Point" H 9250 3700 50  0001 L CNN
-F 2 "Connector_Wire:SolderWirePad_1x01_SMD_5x10mm" H 9500 3500 50  0001 C CNN
+F 2 "FrequentlyUsed:Pad_2.5-2.5" H 9500 3500 50  0001 C CNN
 F 3 "None" H 9500 3500 50  0001 C CNN
 F 4 "TP_3V" H 9250 3700 50  0000 L CNN "Name"
@@
 $EndComp
 Wire Wire Line
-	4500 4050 5300 4050
+	4500 4050 5200 4050
 Wire Wire Line
 	8850 3500 9700 3500
 Wire Wire Line
 	6600 3500 7100 3500
+Text Label 1600 3500 0    50   ~ 0
+B+
+Text Label 3650 3500 0    50   ~ 0
+BSWO
+Connection ~ 5200 4050
+Wire Wire Line
+	5200 4050 5300 4050
 $EndSCHEMATC

Commit message: PCB Update
Connections:
- net +3V3: now also TP203.1
- net +5V: now also TP202.1
Changed lines of the file:
@@
 	4500 4050 5200 4050
 Wire Wire Line
-	8850 3500 9700 3500
+	8850 3500 9300 3500
 Wire Wire Line
-	6600 3500 7100 3500
+	6600 3500 6850 3500
 Text Label 1600 3500 0    50   ~ 0
 B+
@@
 Wire Wire Line
 	5200 4050 5300 4050
+Connection ~ 6850 3500
+Wire Wire Line
+	6850 3500 7100 3500
+Connection ~ 9300 3500
+Wire Wire Line
+	9300 3500 9700 3500
 $EndSCHEMATC

Commit message: Updates
Parts:
- U201, U202: footprint Package_TO_SOT_SMD:SOT-23-5_HandSoldering -> Package_TO_SOT_SMD:SOT-23-5
Changed lines of the file:
@@
 F 0 "U202" H 8050 4150 60  0000 L CNN
 F 1 "MIC5219-3.3YM5-TR" H 8050 4050 60  0000 L CNN
-F 2 "Package_TO_SOT_SMD:SOT-23-5_HandSoldering" H 8050 3300 60  0001 L CNN
+F 2 "Package_TO_SOT_SMD:SOT-23-5" H 8050 3300 60  0001 L CNN
 F 3 "http://ww1.microchip.com/downloads/en/DeviceDoc/MIC5219-500mA-Peak-Output-LDO-Regulator-DS20006021A.pdf" H 7750 3900 60  0001 C CNN
 F 4 "576-1281-6-ND" H 8400 3700 50  0001 C CNN "DigiKey Part No."
@@
 F 0 "U201" H 5450 4150 60  0000 L CNN
 F 1 "MIC5219-5.0YM5-TR" H 5450 4050 60  0000 L CNN
-F 2 "Package_TO_SOT_SMD:SOT-23-5_HandSoldering" H 5450 3300 60  0001 L CNN
+F 2 "Package_TO_SOT_SMD:SOT-23-5" H 5450 3300 60  0001 L CNN
 F 3 "http://ww1.microchip.com/downloads/en/DeviceDoc/MIC5219-500mA-Peak-Output-LDO-Regulator-DS20006021A.pdf" H 5150 3900 60  0001 C CNN
 F 4 "576-2770-6-ND" H 5800 3700 50  0001 C CNN "DigiKey Part No."
