File: Page 5.sch (KiCad schematic (older format))
At the start: 0 parts

Commit message: Updates
Parts:
- added C501: 0.1uF, Capacitor_SMD:C_0603_1608Metric_Pad1.05x0.95mm_HandSolder, symbol Device:C
- added R501: R10K0, Resistor_SMD:R_0603_1608Metric_Pad1.05x0.95mm_HandSolder, symbol Device:R
- added R502, R503: R1K0, Resistor_SMD:R_0603_1608Metric_Pad1.05x0.95mm_HandSolder, symbol Device:R
- added U501: ATSAMD11C14A-SS, Package_SO:SOIC-14_3.9x8.7mm_P1.27mm, symbol MCU_Microchip_SAMD:ATSAMD11C14A-SS
Connections:
- new net +3V3: C501.1, U501.12 (VDD)
- new net GND: C501.2, U501.11 (GND)
- no-connect marks 0 -> 4
Changed lines of the file:
@@
 Comment4 ""
 $EndDescr
+$Comp
+L MCU_Microchip_SAMD:ATSAMD11C14A-SS U501
+U 1 1 5EBC098A
+P 4000 2800
+F 0 "U501" H 4200 3550 50  0000 L CNN
+F 1 "ATSAMD11C14A-SS" H 4200 3450 50  0000 L CNN
+F 2 "Package_SO:SOIC-14_3.9x8.7mm_P1.27mm" H 4000 1750 50  0001 C CNN
+F 3 "http://ww1.microchip.com/downloads/en/DeviceDoc/Atmel-42363-SAM-D11_Datasheet.pdf" H 4000 2100 50  0001 C CNN
+	1    4000 2800
+	1    0    0    -1
+$EndComp
+NoConn ~ 4500 2500
+NoConn ~ 3500 3000
+NoConn ~ 4500 2800
+NoConn ~ 4500 2900
+$Comp
+L Device:C C?
+U 1 1 5EBC3CA5
+P 2950 3550
+AR Path="/5EBC3CA5" Ref="C?"  Part="1"
+AR Path="/5EAC05C2/5EBC3CA5" Ref="C?"  Part="1"
+AR Path="/5EACA483/5EBC3CA5" Ref="C?"  Part="1"
+AR Path="/5ECEA271/5EBC3CA5" Ref="C?"  Part="1"
+AR Path="/5ECF2F45/5EBC3CA5" Ref="C?"  Part="1"
+AR Path="/5ECF2FE7/5EBC3CA5" Ref="C501"  Part="1"
+F 0 "C501" H 3100 3600 50  0000 L BNN
+F 1 "0.1uF" H 3100 3500 50  0000 L BNN
+F 2 "Capacitor_SMD:C_0603_1608Metric_Pad1.05x0.95mm_HandSolder" H 2988 3400 50  0001 C CNN
+F 3 "https://www.yageo.com/upload/media/product/productsearch/datasheet/mlcc/UPY-GPHC_X7R_6.3V-to-50V_18.pdf" H 2950 3550 50  0001 C CNN
+F 4 "Yageo CC0603KPX7R7BB104" H 2950 3550 50  0001 C CNN "Mftr Part No."
+	1    2950 3550
+	1    0    0    -1
+$EndComp
+Wire Wire Line
+	2950 3700 2950 3800
+$Comp
+L power:GND #PWR?
+U 1 1 5EBC43AB
+P 3450 3900
+F 0 "#PWR?" H 3450 3650 50  0001 C CNN
+F 1 "GND" H 3455 3727 50  0000 C CNN
+F 2 "" H 3450 3900 50  0001 C CNN
+F 3 "" H 3450 3900 50  0001 C CNN
+	1    3450 3900
+	1    0    0    -1
+$EndComp
+Wire Wire Line
+	4000 3500 4000 3800
+Wire Wire Line
+	4000 3800 3450 3800
+Wire Wire Line
+	3450 3800 3450 3900
+Wire Wire Line
+	2950 3400 2950 2000
+Wire Wire Line
+	4000 2000 4000 2100
+Connection ~ 3450 3800
+Wire Wire Line
+	3450 3800 2950 3800
+$Comp
+L power:+3.3V #PWR?
+U 1 1 5EBC5389
+P 3500 1900
+F 0 "#PWR?" H 3500 1750 50  0001 C CNN
+F 1 "+3.3V" H 3515 2073 50  0000 C CNN
+F 2 "" H 3500 1900 50  0001 C CNN
+F 3 "" H 3500 1900 50  0001 C CNN
+	1    3500 1900
+	1    0    0    -1
+$EndComp
+Wire Wire Line
+	2950 2000 3500 2000
+Wire Wire Line
+	3500 1900 3500 2000
+Connection ~ 3500 2000
+Wire Wire Line
+	3500 2000 4000 2000
+$Comp
+L Device:R R?
+U 1 1 5EBC6EB0
+P 6350 2400
+AR Path="/5EBC6EB0" Ref="R?"  Part="1"
+AR Path="/5EAC05C2/5EBC6EB0" Ref="R?"  Part="1"
+AR Path="/5EACA483/5EBC6EB0" Ref="R?"  Part="1"
+AR Path="/5ECF2FE7/5EBC6EB0" Ref="R501"  Part="1"
+F 0 "R501" H 6420 2446 50  0000 L CNN
+F 1 "R10K0" H 6420 2355 50  0000 L CNN
+F 2 "Resistor_SMD:R_0603_1608Metric_Pad1.05x0.95mm_HandSolder" V 6280 2400 50  0001 C CNN
+F 3 "https://www.yageo.com/upload/media/product/productsearch/datasheet/rchip/PYu-RC_Group_51_RoHS_L_10.pdf" H 6350 2400 50  0001 C CNN
+F 4 "311-10KGRCT-ND" H 6350 2400 50  0001 C CNN "DigiKey Part No."
+F 5 "Yageo RC0603JR-0710KL" H 6350 2400 50  0001 C CNN "Mftr Part No."
+	1    6350 2400
+	1    0    0    -1
+$EndComp
+$Comp
+L Device:R R?
+U 1 1 5EBC7901
+P 7050 2400
+AR Path="/5EBC7901" Ref="R?"  Part="1"
+AR Path="/5EAC05C2/5EBC7901" Ref="R?"  Part="1"
+AR Path="/5EACA483/5EBC7901" Ref="R?"  Part="1"
+AR Path="/5ECF2FE7/5EBC7901" Ref="R502"  Part="1"
+F 0 "R502" V 6950 2300 50  0000 L CNN
+F 1 "R1K0" V 7150 2300 50  0000 L CNN
+F 2 "Resistor_SMD:R_0603_1608Metric_Pad1.05x0.95mm_HandSolder" V 6980 2400 50  0001 C CNN
+F 3 "https://www.yageo.com/upload/media/product/productsearch/datasheet/rchip/PYu-RC_Group_51_RoHS_L_10.pdf" H 7050 2400 50  0001 C CNN
+F 4 "311-1.0KGRCT-ND" H 7050 2400 50  0001 C CNN "DigiKey Part No."
+F 5 "Yageo RC0603JR-071KL" H 7050 2400 50  0001 C CNN "Mftr Part No."
+	1    7050 2400
+	0    1    1    0
+$EndComp
+$Comp
+L Device:R R?
+U 1 1 5EBC8A3C
+P 7050 2850
+AR Path="/5EBC8A3C" Ref="R?"  Part="1"
+AR Path="/5EAC05C2/5EBC8A3C" Ref="R?"  Part="1"
+AR Path="/5EACA483/5EBC8A3C" Ref="R?"  Part="1"
+AR Path="/5ECF2FE7/5EBC8A3C" Ref="R503"  Part="1"
+F 0 "R503" V 6950 2750 50  0000 L CNN
+F 1 "R1K0" V 7150 2750 50  0000 L CNN
+F 2 "Resistor_SMD:R_0603_1608Metric_Pad1.05x0.95mm_HandSolder" V 6980 2850 50  0001 C CNN
+F 3 "https://www.yageo.com/upload/media/product/productsearch/datasheet/rchip/PYu-RC_Group_51_RoHS_L_10.pdf" H 7050 2850 50  0001 C CNN
+F 4 "311-1.0KGRCT-ND" H 7050 2850 50  0001 C CNN "DigiKey Part No."
+F 5 "Yageo RC0603JR-071KL" H 7050 2850 50  0001 C CNN "Mftr Part No."
+	1    7050 2850
+	0    1    1    0
+$EndComp
 $EndSCHEMATC

Commit message: Updates
Parts:
- added C502: 4.7uF, Capacitor_SMD:C_0603_1608Metric_Pad1.05x0.95mm_HandSolder, symbol Device:C
- added D501: PRTR5V0U2X, Package_TO_SOT_SMD:SOT-143, symbol Power_Protection:PRTR5V0U2X
- added J501: USB_B_Mini, Name Plate Class Project:Molex_USB_Mini_B_548190572, symbol Connector:USB_B_Mini
- added J502: SAMD11 Header, Name Plate Class Project:Molex_PinHeader_2x05, symbol Connector_Generic:Conn_02x05_Odd_Even
- added R504: R1M0, Resistor_SMD:R_0603_1608Metric_Pad1.05x0.95mm_HandSolder, symbol Device:R
- added TP501: TP_SAMD11_nRST, Connector_Wire:SolderWirePad_1x01_SMD_5x10mm, symbol Connector:TestPoint
- added TP502: TP_MEGA_nRST, Connector_Wire:SolderWirePad_1x01_SMD_5x10mm, symbol Connector:TestPoint
- added TP503: TP_SAMD11_TX_MEGA_RX, Connector_Wire:SolderWirePad_1x01_SMD_5x10mm, symbol Connector:TestPoint
- added TP504: TP_SAMD11_RX_MEGA_TX, Connector_Wire:SolderWirePad_1x01_SMD_5x10mm, symbol Connector:TestPoint
- added TP505: TP_SAMD11_SWCLK, Connector_Wire:SolderWirePad_1x01_SMD_5x10mm, symbol Connector:TestPoint
- added TP506: TP_SAMD11_SWDIO, Connector_Wire:SolderWirePad_1x01_SMD_5x10mm, symbol Connector:TestPoint
Connections:
- net +3V3: now also R501.1, J502.1 (Pin_1)
- net GND: now also C502.2, D501.1 (GND), J501.5 (GND), J502.3 (Pin_3), J502.5 (Pin_5), R504.2
- net SAMD11_RX: now reaches U501.1 (PA05)
- net SAMD11_RX: now also R503.2
- net USB_DP: now reaches U501.10 (PA25)
- net USB_DP: now also D501.2 (I/O1), J501.3 (D+)
- net SAMD11_TX: now reaches U501.14 (PA04)
- net SAMD11_TX: now also R502.2
- net MEGA_nRST: now reaches U501.3 (PA09/XOUT)
- net MEGA_nRST: now also TP502.1
- net SAMD11_nRST: now reaches U501.6 (PA28/~RST)
- net SAMD11_nRST: now also R501.2, J502.10 (Pin_10), TP501.1
- net SAMD11_SWCLK: now reaches U501.7 (PA30/SWCLK)
- net SAMD11_SWCLK: now also J502.4 (Pin_4), TP505.1
- net SAMD11_SWDIO: now reaches U501.8 (PA31/SWDIO)
- net SAMD11_SWDIO: now also J502.2 (Pin_2), TP506.1
- net USB_DM: now reaches U501.9 (PA24)
- net USB_DM: now also D501.3 (I/O2), J501.2 (D-)
- net MEGA_RX: now reaches R502.1
- net MEGA_RX: now also TP503.1
- net MEGA_TX: now reaches R503.1
- net MEGA_TX: now also TP504.1
- new net: C502.1, J501.6 (Shield), R504.1
- new net VBUS: D501.4 (VCC), J501.1 (VBUS)
- no-connect marks 4 -> 9
Other:
- note added: "SAMD11 Microcontroller and Connector"
- note added: "USB Connector"
- moved on the sheet: C501, R501, R502, R503, U501

Commit message: Switched to Hierarchical
Parts:
- J501: symbol Connector:USB_B_Mini -> Name~Plate~Class~Library:USB_B_Mini
Connections:
- net labels added: SAMD11_RX_MEGA_TX, SAMD11_TX_MEGA_RX
- net labels removed: MEGA_RX, MEGA_TX
Other:
- moved on the sheet: R501, TP501, TP502, TP505, TP506
Changed lines of the file:
@@
 $EndComp
 $Comp
-L Connector:USB_B_Mini J501
+L Name~Plate~Class~Library:USB_B_Mini J501
 U 1 1 5EBEA16E
 P 2650 6300
@@
 Wire Wire Line
 	8850 1950 9650 1950
-Text GLabel 9650 2350 2    50   Output ~ 0
-SAMD11_nRST
 Text Label 8950 2350 0    50   ~ 0
 SAMD11_nRST
-Text GLabel 9650 2050 2    50   Output ~ 0
-SAMD11_SWCLK
-Text GLabel 9650 1950 2    50   BiDi ~ 0
-SAMD11_SWDIO
 Text Label 8950 1950 0    50   ~ 0
 SAMD11_SWDIO
@@
 	1    0    0    -1
 $EndComp
-Text GLabel 4500 6400 2    50   BiDi ~ 0
-USB_DM
-Text GLabel 3550 6300 2    50   BiDi ~ 0
-USB_DP
 Wire Wire Line
 	2950 6300 3200 6300
@@
 Connection ~ 3200 6300
 Wire Wire Line
-	3200 6300 3550 6300
+	3200 6300 3700 6300
 Wire Wire Line
 	4150 5350 4300 5350
@@
 Connection ~ 4300 6400
 Wire Wire Line
-	4300 6400 4500 6400
+	4300 6400 4800 6400
 Wire Wire Line
 	4100 4850 4100 4900
@@
 	1    0    0    -1
 $EndComp
-Text Label 2800 2050 0    50   ~ 0
+Text Label 1750 2050 0    50   ~ 0
 SAMD11_SWCLK
-Text Label 2800 2150 0    50   ~ 0
+Text Label 1750 2150 0    50   ~ 0
 SAMD11_SWDIO
-Text GLabel 5900 2450 2    50   BiDi ~ 0
-USB_DP
-Text GLabel 5900 2350 2    50   BiDi ~ 0
-USB_DM
 Text Label 4900 2450 0    50   ~ 0
 USB_DP
@@
 	1    0    0    -1
 $EndComp
-Text GLabel 6650 2050 2    50   UnSpc ~ 0
-MEGA_TX
-Text GLabel 6650 1950 2    50   UnSpc ~ 0
-MEGA_RX
 Text Label 4900 2050 0    50   ~ 0
 SAMD11_RX
@@
 SAMD11_TX
 Wire Wire Line
-	4700 2450 5900 2450
-Wire Wire Line
-	4700 2350 5900 2350
+	4700 2450 5200 2450
+Wire Wire Line
+	4700 2350 5200 2350
 Wire Wire Line
 	5750 2050 6350 2050
@@
 	4200 2850 4200 3400
 Wire Wire Line
-	2050 2150 2050 2350
-Wire Wire Line
-	2050 2850 1900 2850
-Connection ~ 2050 2850
-Wire Wire Line
-	2050 2950 2050 2850
+	2400 2150 2400 2350
+Wire Wire Line
+	2400 2950 2400 2850
 $Comp
 L Connector:TestPoint TP?
 U 1 1 5EBD98BA
-P 2050 2950
+P 2400 2950
 AR Path="/5ECF32A9/5EBD98BA" Ref="TP?"  Part="1"
 AR Path="/5ECF2FE7/5EBD98BA" Ref="TP502"  Part="1"
-F 0 "TP502" H 2000 3050 50  0000 R CNN
-F 1 "TP_MEGA_nRST" H 2000 3150 50  0000 R CNN
-F 2 "Connector_Wire:SolderWirePad_1x01_SMD_5x10mm" H 2250 2950 50  0001 C CNN
-F 3 "~" H 2250 2950 50  0001 C CNN
-	1    2050 2950
+F 0 "TP502" H 2350 3050 50  0000 R CNN
+F 1 "TP_MEGA_nRST" H 2350 3150 50  0000 R CNN
+F 2 "Connector_Wire:SolderWirePad_1x01_SMD_5x10mm" H 2600 2950 50  0001 C CNN
+F 3 "~" H 2600 2950 50  0001 C CNN
+	1    2400 2950
 	-1   0    0    1
 $EndComp
@@
 L Connector:TestPoint TP?
 U 1 1 5EBCF6F7
-P 2650 2200
+P 2800 2200
 AR Path="/5ECF32A9/5EBCF6F7" Ref="TP?"  Part="1"
 AR Path="/5ECF2FE7/5EBCF6F7" Ref="TP505"  Part="1"
-F 0 "TP505" H 2850 2450 50  0000 R CNN
-F 1 "TP_SAMD11_SWCLK" H 2850 2550 50  0000 R CNN
-F 2 "Connector_Wire:SolderWirePad_1x01_SMD_5x10mm" H 2850 2200 50  0001 C CNN
-F 3 "~" H 2850 2200 50  0001 C CNN
-	1    2650 2200
+F 0 "TP505" H 3000 2450 50  0000 R CNN
+F 1 "TP_SAMD11_SWCLK" H 3000 2550 50  0000 R CNN
+F 2 "Connector_Wire:SolderWirePad_1x01_SMD_5x10mm" H 3000 2200 50  0001 C CNN
+F 3 "~" H 3000 2200 50  0001 C CNN
+	1    2800 2200
 	-1   0    0    1
 $EndComp
 Wire Wire Line
-	2650 2200 2650 2050
-Wire Wire Line
-	3550 2850 2050 2850
-Wire Wire Line
-	3700 2050 2650 2050
-Wire Wire Line
-	1900 2050 2650 2050
-Connection ~ 2650 2050
+	3550 2850 2400 2850
+Wire Wire Line
+	3700 2050 2800 2050
+Wire Wire Line
+	1750 2050 2800 2050
+Connection ~ 2800 2050
 $Comp
 L Connector:TestPoint TP?
 U 1 1 5EBCD7DB
-P 2050 2350
+P 2400 2350
 AR Path="/5ECF32A9/5EBCD7DB" Ref="TP?"  Part="1"
 AR Path="/5ECF2FE7/5EBCD7DB" Ref="TP506"  Part="1"
-F 0 "TP506" H 2800 2350 50  0000 R CNN
-F 1 "TP_SAMD11_SWDIO" H 2800 2450 50  0000 R CNN
-F 2 "Connector_Wire:SolderWirePad_1x01_SMD_5x10mm" H 2250 2350 50  0001 C CNN
-F 3 "~" H 2250 2350 50  0001 C CNN
-	1    2050 2350
+F 0 "TP506" H 3150 2350 50  0000 R CNN
+F 1 "TP_SAMD11_SWDIO" H 3150 2450 50  0000 R CNN
+F 2 "Connector_Wire:SolderWirePad_1x01_SMD_5x10mm" H 2600 2350 50  0001 C CNN
+F 3 "~" H 2600 2350 50  0001 C CNN
+	1    2400 2350
 	-1   0    0    1
 $EndComp
-Text GLabel 1900 2850 0    50   UnSpc ~ 0
-MEGA_nRST
 Text Label 2800 2850 0    50   ~ 0
 MEGA_nRST
@@
 Connection ~ 3400 1000
 Wire Wire Line
-	2650 1000 2650 1250
-Wire Wire Line
-	3400 1000 2650 1000
+	2950 1000 2950 1250
+Wire Wire Line
+	3400 1000 2950 1000
 Wire Wire Line
 	4200 1000 4200 1450
 Wire Wire Line
-	2650 1850 3700 1850
-Connection ~ 2650 1850
-Wire Wire Line
-	2650 1550 2650 1850
-Wire Wire Line
-	2050 2150 3700 2150
-Connection ~ 2050 2150
-Wire Wire Line
-	1900 2150 2050 2150
-Wire Wire Line
-	2050 1850 2650 1850
-Wire Wire Line
-	2050 1850 1900 1850
-Connection ~ 2050 1850
-Text GLabel 1900 1850 0    50   Input ~ 0
-SAMD11_nRST
+	2950 1550 2950 1850
 $Comp
 L Connector:TestPoint TP?
 U 1 1 5EBCAF81
-P 2050 1850
+P 2400 1850
 AR Path="/5ECF32A9/5EBCAF81" Ref="TP?"  Part="1"
 AR Path="/5ECF2FE7/5EBCAF81" Ref="TP501"  Part="1"
-F 0 "TP501" H 1850 2150 50  0000 L CNN
-F 1 "TP_SAMD11_nRST" H 1850 2050 50  0000 L CNN
-F 2 "Connector_Wire:SolderWirePad_1x01_SMD_5x10mm" H 2250 1850 50  0001 C CNN
-F 3 "~" H 2250 1850 50  0001 C CNN
-	1    2050 1850
-	1    0    0    -1
-$EndComp
-Text GLabel 1900 2050 0    50   Input ~ 0
-SAMD11_SWCLK
-Text Label 2800 1850 0    50   ~ 0
+F 0 "TP501" H 2200 2150 50  0000 L CNN
+F 1 "TP_SAMD11_nRST" H 2200 2050 50  0000 L CNN
+F 2 "Connector_Wire:SolderWirePad_1x01_SMD_5x10mm" H 2600 1850 50  0001 C CNN
+F 3 "~" H 2600 1850 50  0001 C CNN
+	1    2400 1850
+	1    0    0    -1
+$EndComp
+Text Label 1750 1850 0    50   ~ 0
 SAMD11_nRST
-Text GLabel 1900 2150 0    50   BiDi ~ 0
-SAMD11_SWDIO
 Wire Wire Line
 	3400 1000 3700 1000
@@
 L Device:R R?
 U 1 1 5EBC6EB0
-P 2650 1400
+P 2950 1400
 AR Path="/5EBC6EB0" Ref="R?"  Part="1"
 AR Path="/5EAC05C2/5EBC6EB0" Ref="R?"  Part="1"
 AR Path="/5EACA483/5EBC6EB0" Ref="R?"  Part="1"
 AR Path="/5ECF2FE7/5EBC6EB0" Ref="R501"  Part="1"
-F 0 "R501" H 2720 1446 50  0000 L CNN
-F 1 "R10K0" H 2720 1355 50  0000 L CNN
-F 2 "Resistor_SMD:R_0603_1608Metric_Pad1.05x0.95mm_HandSolder" V 2580 1400 50  0001 C CNN
-F 3 "https://www.yageo.com/upload/media/product/productsearch/datasheet/rchip/PYu-RC_Group_51_RoHS_L_10.pdf" H 2650 1400 50  0001 C CNN
-F 4 "311-10KGRCT-ND" H 2650 1400 50  0001 C CNN "DigiKey Part No."
-F 5 "Yageo RC0603JR-0710KL" H 2650 1400 50  0001 C CNN "Mftr Part No."
-	1    2650 1400
+F 0 "R501" H 3020 1446 50  0000 L CNN
+F 1 "R10K0" H 3020 1355 50  0000 L CNN
+F 2 "Resistor_SMD:R_0603_1608Metric_Pad1.05x0.95mm_HandSolder" V 2880 1400 50  0001 C CNN
+F 3 "https://www.yageo.com/upload/media/product/productsearch/datasheet/rchip/PYu-RC_Group_51_RoHS_L_10.pdf" H 2950 1400 50  0001 C CNN
+F 4 "311-10KGRCT-ND" H 2950 1400 50  0001 C CNN "DigiKey Part No."
+F 5 "Yageo RC0603JR-0710KL" H 2950 1400 50  0001 C CNN "Mftr Part No."
+	1    2950 1400
 	1    0    0    -1
 $EndComp
@@
 Wire Wire Line
 	3750 4900 3750 4950
+Text Label 4500 6400 0    50   ~ 0
+USB_DM
+Text Label 3400 6300 0    50   ~ 0
+USB_DP
+Text HLabel 2200 2850 0    50   Input ~ 0
+MEGA_nRST
+Text HLabel 6650 1950 2    50   Input ~ 0
+SAMD11_TX_MEGA_RX
+Text HLabel 6650 2050 2    50   Input ~ 0
+SAMD11_RX_MEGA_TX
+Connection ~ 2400 2150
+Wire Wire Line
+	1750 2150 2400 2150
+Wire Wire Line
+	2800 2050 2800 2200
+Wire Wire Line
+	2400 2150 3700 2150
+Connection ~ 2950 1850
+Wire Wire Line
+	2950 1850 3700 1850
+Connection ~ 2400 1850
+Wire Wire Line
+	2400 1850 2950 1850
+Wire Wire Line
+	1750 1850 2400 1850
+Connection ~ 2400 2850
+Wire Wire Line
+	2200 2850 2400 2850
 $EndSCHEMATC

Commit message: Updates
Parts:
- R501: value R10K0 -> 10K0; Manufacturer (none) -> Yageo
- R502, R503: value R1K0 -> 1K0
- R504: value R1M0 -> 1M0
- TP501: value TP_SAMD11_nRST -> Test Point; Name (none) -> TP_SAMD11_nRST
- TP502: value TP_MEGA_nRST -> Test Point; Name (none) -> TP_MEGA_nRST
- TP503: value TP_SAMD11_TX_MEGA_RX -> Test Point; Name (none) -> TP_SAMD11_TX_MEGA_RX
- TP504: value TP_SAMD11_RX_MEGA_TX -> Test Point; Name (none) -> TP_SAMD11_RX_MEGA_TX
- TP505: value TP_SAMD11_SWCLK -> Test Point; Name (none) -> TP_SAMD11_SWCLK
- TP506: value TP_SAMD11_SWDIO -> Test Point; Name (none) -> TP_SAMD11_SWDIO
Changed lines of the file:
@@
 AR Path="/5ECF2FE7/5EC05B2C" Ref="R504"  Part="1"
 F 0 "R504" H 1470 6446 50  0000 L CNN
-F 1 "R1M0" H 1470 6355 50  0000 L CNN
+F 1 "1M0" H 1470 6355 50  0000 L CNN
 F 2 "Resistor_SMD:R_0603_1608Metric_Pad1.05x0.95mm_HandSolder" V 1330 6400 50  0001 C CNN
 F 3 "https://www.te.com/commerce/DocumentDelivery/DDEController?Action=srchrtrv&DocNm=1773204-3&DocType=DS&DocLang=English" H 1400 6400 50  0001 C CNN
@@
 AR Path="/5ECF2FE7/5EBE3E2F" Ref="TP504"  Part="1"
 F 0 "TP504" H 6150 2200 50  0000 L CNN
-F 1 "TP_SAMD11_RX_MEGA_TX" H 6150 2100 50  0000 L CNN
+F 1 "Test Point" H 6150 2100 50  0000 L CNN
 F 2 "Connector_Wire:SolderWirePad_1x01_SMD_5x10mm" H 6550 1900 50  0001 C CNN
-F 3 "~" H 6550 1900 50  0001 C CNN
+F 3 "None" H 6550 1900 50  0001 C CNN
+F 4 "TP_SAMD11_RX_MEGA_TX" H 6350 1900 50  0001 C CNN "Name"
 	1    6350 1900
 	1    0    0    -1
@@
 AR Path="/5ECF2FE7/5EBE32F4" Ref="TP503"  Part="1"
 F 0 "TP503" H 5750 1900 50  0000 L CNN
-F 1 "TP_SAMD11_TX_MEGA_RX" H 5750 1800 50  0000 L CNN
+F 1 "Test Point" H 5750 1800 50  0000 L CNN
 F 2 "Connector_Wire:SolderWirePad_1x01_SMD_5x10mm" H 6150 1600 50  0001 C CNN
-F 3 "~" H 6150 1600 50  0001 C CNN
+F 3 "None" H 6150 1600 50  0001 C CNN
+F 4 "TP_SAMD11_TX_MEGA_RX" H 5950 1600 50  0001 C CNN "Name"
 	1    5950 1600
 	1    0    0    -1
@@
 AR Path="/5ECF2FE7/5EBD98BA" Ref="TP502"  Part="1"
 F 0 "TP502" H 2350 3050 50  0000 R CNN
-F 1 "TP_MEGA_nRST" H 2350 3150 50  0000 R CNN
+F 1 "Test Point" H 2350 3150 50  0000 R CNN
 F 2 "Connector_Wire:SolderWirePad_1x01_SMD_5x10mm" H 2600 2950 50  0001 C CNN
-F 3 "~" H 2600 2950 50  0001 C CNN
+F 3 "None" H 2600 2950 50  0001 C CNN
+F 4 "TP_MEGA_nRST" H 2400 2950 50  0001 C CNN "Name"
 	1    2400 2950
 	-1   0    0    1
@@
 AR Path="/5ECF2FE7/5EBCF6F7" Ref="TP505"  Part="1"
 F 0 "TP505" H 3000 2450 50  0000 R CNN
-F 1 "TP_SAMD11_SWCLK" H 3000 2550 50  0000 R CNN
+F 1 "Test Point" H 3000 2550 50  0000 R CNN
 F 2 "Connector_Wire:SolderWirePad_1x01_SMD_5x10mm" H 3000 2200 50  0001 C CNN
-F 3 "~" H 3000 2200 50  0001 C CNN
+F 3 "None" H 3000 2200 50  0001 C CNN
+F 4 "TP_SAMD11_SWCLK" H 2800 2200 50  0001 C CNN "Name"
 	1    2800 2200
 	-1   0    0    1
@@
 AR Path="/5ECF2FE7/5EBCD7DB" Ref="TP506"  Part="1"
 F 0 "TP506" H 3150 2350 50  0000 R CNN
-F 1 "TP_SAMD11_SWDIO" H 3150 2450 50  0000 R CNN
+F 1 "Test Point" H 3150 2450 50  0000 R CNN
 F 2 "Connector_Wire:SolderWirePad_1x01_SMD_5x10mm" H 2600 2350 50  0001 C CNN
-F 3 "~" H 2600 2350 50  0001 C CNN
+F 3 "None" H 2600 2350 50  0001 C CNN
+F 4 "TP_SAMD11_SWDIO" H 2400 2350 50  0001 C CNN "Name"
 	1    2400 2350
 	-1   0    0    1
@@
 AR Path="/5ECF2FE7/5EBCAF81" Ref="TP501"  Part="1"
 F 0 "TP501" H 2200 2150 50  0000 L CNN
-F 1 "TP_SAMD11_nRST" H 2200 2050 50  0000 L CNN
+F 1 "Test Point" H 2200 2050 50  0000 L CNN
 F 2 "Connector_Wire:SolderWirePad_1x01_SMD_5x10mm" H 2600 1850 50  0001 C CNN
-F 3 "~" H 2600 1850 50  0001 C CNN
+F 3 "None" H 2600 1850 50  0001 C CNN
+F 4 "TP_SAMD11_nRST" H 2400 1850 50  0001 C CNN "Name"
 	1    2400 1850
 	1    0    0    -1
@@
 AR Path="/5ECF2FE7/5EBC8A3C" Ref="R503"  Part="1"
 F 0 "R503" V 5700 1950 50  0000 L CNN
-F 1 "R1K0" V 5800 1950 50  0000 L CNN
+F 1 "1K0" V 5800 1950 50  0000 L CNN
 F 2 "Resistor_SMD:R_0603_1608Metric_Pad1.05x0.95mm_HandSolder" V 5530 2050 50  0001 C CNN
 F 3 "https://www.yageo.com/upload/media/product/productsearch/datasheet/rchip/PYu-RC_Group_51_RoHS_L_10.pdf" H 5600 2050 50  0001 C CNN
@@
 AR Path="/5ECF2FE7/5EBC7901" Ref="R502"  Part="1"
 F 0 "R502" V 5400 1850 50  0000 L CNN
-F 1 "R1K0" V 5500 1850 50  0000 L CNN
+F 1 "1K0" V 5500 1850 50  0000 L CNN
 F 2 "Resistor_SMD:R_0603_1608Metric_Pad1.05x0.95mm_HandSolder" V 5530 1950 50  0001 C CNN
 F 3 "https://www.yageo.com/upload/media/product/productsearch/datasheet/rchip/PYu-RC_Group_51_RoHS_L_10.pdf" H 5600 1950 50  0001 C CNN
@@
 AR Path="/5ECF2FE7/5EBC6EB0" Ref="R501"  Part="1"
 F 0 "R501" H 3020 1446 50  0000 L CNN
-F 1 "R10K0" H 3020 1355 50  0000 L CNN
+F 1 "10K0" H 3020 1355 50  0000 L CNN
 F 2 "Resistor_SMD:R_0603_1608Metric_Pad1.05x0.95mm_HandSolder" V 2880 1400 50  0001 C CNN
 F 3 "https://www.yageo.com/upload/media/product/productsearch/datasheet/rchip/PYu-RC_Group_51_RoHS_L_10.pdf" H 2950 1400 50  0001 C CNN
 F 4 "311-10KGRCT-ND" H 2950 1400 50  0001 C CNN "DigiKey Part No."
 F 5 "Yageo RC0603JR-0710KL" H 2950 1400 50  0001 C CNN "Mftr Part No."
+F 6 "Yageo" H 2950 1400 50  0001 C CNN "Manufacturer"
 	1    2950 1400
 	1    0    0    -1

Commit message: Updates to schematic
Switching to ATMega34UF chip.
Parts:
- C501: DigiKey Part No. (none) -> 311-1335-1-ND; Manufacturer (none) -> Yageo; Mftr Part No. Yageo CC0603KPX7R7BB104 -> CC0603KPX7R7BB104
- C502: Manufacturer (none) -> Kemet; Mftr Part No. KEMET C0805C472KDRACTU -> C0805C472KDRACTU
- D501: value PRTR5V0U2X -> PRTR5V0U2X,215; DigiKey Part No. (none) -> 1727-3884-6-ND; Manufacturer (none) -> Philips/NXP; Mftr Part No. (none) -> PRTR5V0U2X,215
- J501: DigiKey Part No. (none) -> WM17116DKR-ND; Manufacturer (none) -> Molex; Mftr Part No. (none) -> 548190572
- J502: DigiKey Part No. (none) -> SAM1157-05-ND; Manufacturer (none) -> Samtec; Mftr Part No. (none) -> FTS-105-01-L-DV
- R501: value 10K0 -> 10k; Mftr Part No. Yageo RC0603JR-0710KL -> RC0603JR-0710KL
- R502, R503: value 1K0 -> 1k; Manufacturer (none) -> Yageo; Mftr Part No. Yageo RC0603JR-071KL -> RC0603JR-071KL
- R504: value 1M0 -> 1M; DigiKey Part No. A130109CT-ND -> 311-1.00MHRCT-ND; Manufacturer (none) -> TE Connectivity; Mftr Part No. TE Connectivity CRGCQ0603J1M0 -> RC0603FR-071ML
- TP501, TP502, TP503, TP504, TP505, TP506: symbol Connector:TestPoint -> Name~Plate~Class~Library:TestPoint; DigiKey Part No. (none) -> None; Manufacturer (none) -> None; Mftr Part No. (none) -> None
- U501: DigiKey Part No. (none) -> ATSAMD11C14A-SSNTDKR-ND; Manufacturer (none) -> Atmel; Mftr Part No. (none) -> ATSAMD11C14A-SSNT
