File: Page 4.sch (KiCad schematic (older format))
At the start: 25 parts

Commit message: Updates
Connections:
- net labels added: SW4
Other:
- note added: "Switches"
- moved on the sheet: C401, C402, C403, C404, C405, R401, R402, R403, R404, R405, R406, R407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

Commit message: Switched to Hierarchical
Changed lines of the file:
@@
 Wire Wire Line
 	3350 1500 3500 1500
-Text GLabel 5100 1500 2    50   UnSpc ~ 0
-SW1
 $Comp
 L power:GND #PWR0110
@@
 Wire Wire Line
 	7000 1500 7150 1500
-Text GLabel 8750 1500 2    50   UnSpc ~ 0
-SW2
 $Comp
 L power:GND #PWR0113
@@
 Wire Wire Line
 	3350 3300 3500 3300
-Text GLabel 5100 3300 2    50   UnSpc ~ 0
-SW3
 $Comp
 L power:GND #PWR0116
@@
 Wire Wire Line
 	7000 3300 7150 3300
-Text GLabel 8750 3300 2    50   UnSpc ~ 0
-SW4
 $Comp
 L power:GND #PWR0119
@@
 Wire Wire Line
 	5350 5050 5500 5050
-Text GLabel 7100 5050 2    50   UnSpc ~ 0
-SW5
 $Comp
 L power:GND #PWR0122
@@
 Wire Wire Line
 	7150 3300 7400 3300
+Text HLabel 5100 1500 2    50   Input ~ 0
+SW1
+Text HLabel 8750 1500 2    50   Input ~ 0
+SW2
+Text HLabel 8750 3300 2    50   Input ~ 0
+SW4
+Text HLabel 7100 5050 2    50   Input ~ 0
+SW5
+Text HLabel 5100 3300 2    50   Input ~ 0
+SW3
 $EndSCHEMATC

Commit message: Updating to Final Revision
Parts:
- renumbered R403 to R402, R402 to R403
Changed lines of the file:
@@
 $Descr A4 11693 8268
 encoding utf-8
-Sheet 5 10
+Sheet 5 9
 Title ""
 Date ""
@@
 AR Path="/5EAC05C2/5EB93212" Ref="R?"  Part="1"
 AR Path="/5EACA483/5EB93212" Ref="R?"  Part="1"
-AR Path="/5ECF2F45/5EB93212" Ref="R402"  Part="1"
-F 0 "R402" V 4350 1400 50  0000 L CNN
+AR Path="/5ECF2F45/5EB93212" Ref="R403"  Part="1"
+F 0 "R403" V 4350 1400 50  0000 L CNN
 F 1 "R43K0" V 4150 1350 50  0000 L CNN
 F 2 "Resistor_SMD:R_0603_1608Metric_Pad1.05x0.95mm_HandSolder" V 4180 1500 50  0001 C CNN
@@
 AR Path="/5EAC05C2/5EBA7594" Ref="R?"  Part="1"
 AR Path="/5EACA483/5EBA7594" Ref="R?"  Part="1"
-AR Path="/5ECF2F45/5EBA7594" Ref="R403"  Part="1"
-F 0 "R403" H 7470 1296 50  0000 L CNN
+AR Path="/5ECF2F45/5EBA7594" Ref="R402"  Part="1"
+F 0 "R402" H 7470 1296 50  0000 L CNN
 F 1 "R12K0" H 7470 1205 50  0000 L CNN
 F 2 "Resistor_SMD:R_0603_1608Metric_Pad1.05x0.95mm_HandSolder" V 7330 1250 50  0001 C CNN

Commit message: Updates
Parts:
- R401, R402, R405, R407, R409: value R12K0 -> 12K0
- R403, R404, R406, R408, R410: value R43K0 -> 43K0
- TP401: value TP_SW1 -> Test Point; Name (none) -> TP_SW1
- TP402: value TP_SW1 -> Test Point; Name (none) -> TP_SW2
- TP403: value TP_SW1 -> Test Point; Name (none) -> TP_SW3
- TP404: value TP_SW1 -> Test Point; Name (none) -> TP_SW4
- TP405: value TP_SW1 -> Test Point; Name (none) -> TP_SW5
Changed lines of the file:
@@
 AR Path="/5ECF2F45/5EB9319E" Ref="R401"  Part="1"
 F 0 "R401" H 3820 1296 50  0000 L CNN
-F 1 "R12K0" H 3820 1205 50  0000 L CNN
+F 1 "12K0" H 3820 1205 50  0000 L CNN
 F 2 "Resistor_SMD:R_0603_1608Metric_Pad1.05x0.95mm_HandSolder" V 3680 1250 50  0001 C CNN
 F 3 "https://www.yageo.com/upload/media/product/productsearch/datasheet/rchip/PYu-RC_Group_51_RoHS_L_10.pdf" H 3750 1250 50  0001 C CNN
@@
 AR Path="/5ECF2F45/5EB93212" Ref="R403"  Part="1"
 F 0 "R403" V 4350 1400 50  0000 L CNN
-F 1 "R43K0" V 4150 1350 50  0000 L CNN
+F 1 "43K0" V 4150 1350 50  0000 L CNN
 F 2 "Resistor_SMD:R_0603_1608Metric_Pad1.05x0.95mm_HandSolder" V 4180 1500 50  0001 C CNN
 F 3 "https://www.yageo.com/upload/media/product/productsearch/datasheet/rchip/PYu-RC_Group_51_RoHS_L_10.pdf" H 4250 1500 50  0001 C CNN
@@
 	1    0    0    -1
 $EndComp
-$Comp
-L Connector:TestPoint TP?
-U 1 1 5EB966B9
-P 4600 1500
-AR Path="/5ECF32A9/5EB966B9" Ref="TP?"  Part="1"
-AR Path="/5ECF2F45/5EB966B9" Ref="TP401"  Part="1"
-F 0 "TP401" H 4500 1800 50  0000 L CNN
-F 1 "TP_SW1" H 4500 1700 50  0000 L CNN
-F 2 "Connector_Wire:SolderWirePad_1x01_SMD_5x10mm" H 4800 1500 50  0001 C CNN
-F 3 "~" H 4800 1500 50  0001 C CNN
-	1    4600 1500
-	1    0    0    -1
-$EndComp
 Wire Wire Line
 	4800 1650 4800 1500
@@
 AR Path="/5ECF2F45/5EBA7594" Ref="R402"  Part="1"
 F 0 "R402" H 7470 1296 50  0000 L CNN
-F 1 "R12K0" H 7470 1205 50  0000 L CNN
+F 1 "12K0" H 7470 1205 50  0000 L CNN
 F 2 "Resistor_SMD:R_0603_1608Metric_Pad1.05x0.95mm_HandSolder" V 7330 1250 50  0001 C CNN
 F 3 "https://www.yageo.com/upload/media/product/productsearch/datasheet/rchip/PYu-RC_Group_51_RoHS_L_10.pdf" H 7400 1250 50  0001 C CNN
@@
 AR Path="/5ECF2F45/5EBA75BA" Ref="TP402"  Part="1"
 F 0 "TP402" H 8150 1800 50  0000 L CNN
-F 1 "TP_SW1" H 8150 1700 50  0000 L CNN
+F 1 "Test Point" H 8150 1700 50  0001 L CNN
 F 2 "Connector_Wire:SolderWirePad_1x01_SMD_5x10mm" H 8450 1500 50  0001 C CNN
-F 3 "~" H 8450 1500 50  0001 C CNN
+F 3 "None" H 8450 1500 50  0001 C CNN
+F 4 "TP_SW2" H 8150 1700 50  0000 L CNN "Name"
 	1    8250 1500
 	1    0    0    -1
@@
 AR Path="/5ECF2F45/5EBAED97" Ref="R405"  Part="1"
 F 0 "R405" H 3820 3096 50  0000 L CNN
-F 1 "R12K0" H 3820 3005 50  0000 L CNN
+F 1 "12K0" H 3820 3005 50  0000 L CNN
 F 2 "Resistor_SMD:R_0603_1608Metric_Pad1.05x0.95mm_HandSolder" V 3680 3050 50  0001 C CNN
 F 3 "https://www.yageo.com/upload/media/product/productsearch/datasheet/rchip/PYu-RC_Group_51_RoHS_L_10.pdf" H 3750 3050 50  0001 C CNN
@@
 AR Path="/5ECF2F45/5EBAED9D" Ref="R406"  Part="1"
 F 0 "R406" V 4350 3200 50  0000 L CNN
-F 1 "R43K0" V 4150 3150 50  0000 L CNN
+F 1 "43K0" V 4150 3150 50  0000 L CNN
 F 2 "Resistor_SMD:R_0603_1608Metric_Pad1.05x0.95mm_HandSolder" V 4180 3300 50  0001 C CNN
 F 3 "https://www.yageo.com/upload/media/product/productsearch/datasheet/rchip/PYu-RC_Group_51_RoHS_L_10.pdf" H 4250 3300 50  0001 C CNN
@@
 AR Path="/5ECF2F45/5EBAEDBD" Ref="TP403"  Part="1"
 F 0 "TP403" H 4500 3600 50  0000 L CNN
-F 1 "TP_SW1" H 4500 3500 50  0000 L CNN
+F 1 "Test Point" H 4500 3500 50  0001 L CNN
 F 2 "Connector_Wire:SolderWirePad_1x01_SMD_5x10mm" H 4800 3300 50  0001 C CNN
-F 3 "~" H 4800 3300 50  0001 C CNN
+F 3 "None" H 4800 3300 50  0001 C CNN
+F 4 "TP_SW3" H 4500 3500 50  0000 L CNN "Name"
 	1    4600 3300
 	1    0    0    -1
@@
 AR Path="/5ECF2F45/5EBB48B3" Ref="R407"  Part="1"
 F 0 "R407" H 7470 3096 50  0000 L CNN
-F 1 "R12K0" H 7470 3005 50  0000 L CNN
+F 1 "12K0" H 7470 3005 50  0000 L CNN
 F 2 "Resistor_SMD:R_0603_1608Metric_Pad1.05x0.95mm_HandSolder" V 7330 3050 50  0001 C CNN
 F 3 "https://www.yageo.com/upload/media/product/productsearch/datasheet/rchip/PYu-RC_Group_51_RoHS_L_10.pdf" H 7400 3050 50  0001 C CNN
@@
 AR Path="/5ECF2F45/5EBB48B9" Ref="R408"  Part="1"
 F 0 "R408" V 8000 3200 50  0000 L CNN
-F 1 "R43K0" V 7800 3150 50  0000 L CNN
+F 1 "43K0" V 7800 3150 50  0000 L CNN
 F 2 "Resistor_SMD:R_0603_1608Metric_Pad1.05x0.95mm_HandSolder" V 7830 3300 50  0001 C CNN
 F 3 "https://www.yageo.com/upload/media/product/productsearch/datasheet/rchip/PYu-RC_Group_51_RoHS_L_10.pdf" H 7900 3300 50  0001 C CNN
@@
 AR Path="/5ECF2F45/5EBB48D9" Ref="TP404"  Part="1"
 F 0 "TP404" H 8150 3600 50  0000 L CNN
-F 1 "TP_SW1" H 8150 3500 50  0000 L CNN
+F 1 "Test Point" H 8150 3500 50  0001 L CNN
 F 2 "Connector_Wire:SolderWirePad_1x01_SMD_5x10mm" H 8450 3300 50  0001 C CNN
-F 3 "~" H 8450 3300 50  0001 C CNN
+F 3 "None" H 8450 3300 50  0001 C CNN
+F 4 "TP_SW4" H 8150 3500 50  0000 L CNN "Name"
 	1    8250 3300
 	1    0    0    -1
@@
 AR Path="/5ECF2F45/5EBBC6F7" Ref="R409"  Part="1"
 F 0 "R409" H 5820 4846 50  0000 L CNN
-F 1 "R12K0" H 5820 4755 50  0000 L CNN
+F 1 "12K0" H 5820 4755 50  0000 L CNN
 F 2 "Resistor_SMD:R_0603_1608Metric_Pad1.05x0.95mm_HandSolder" V 5680 4800 50  0001 C CNN
 F 3 "https://www.yageo.com/upload/media/product/productsearch/datasheet/rchip/PYu-RC_Group_51_RoHS_L_10.pdf" H 5750 4800 50  0001 C CNN
@@
 AR Path="/5ECF2F45/5EBBC6FD" Ref="R410"  Part="1"
 F 0 "R410" V 6350 4950 50  0000 L CNN
-F 1 "R43K0" V 6150 4900 50  0000 L CNN
+F 1 "43K0" V 6150 4900 50  0000 L CNN
 F 2 "Resistor_SMD:R_0603_1608Metric_Pad1.05x0.95mm_HandSolder" V 6180 5050 50  0001 C CNN
 F 3 "https://www.yageo.com/upload/media/product/productsearch/datasheet/rchip/PYu-RC_Group_51_RoHS_L_10.pdf" H 6250 5050 50  0001 C CNN
@@
 AR Path="/5ECF2F45/5EBBC71D" Ref="TP405"  Part="1"
 F 0 "TP405" H 6500 5350 50  0000 L CNN
-F 1 "TP_SW1" H 6500 5250 50  0000 L CNN
+F 1 "Test Point" H 6500 5250 50  0001 L CNN
 F 2 "Connector_Wire:SolderWirePad_1x01_SMD_5x10mm" H 6800 5050 50  0001 C CNN
-F 3 "~" H 6800 5050 50  0001 C CNN
+F 3 "None" H 6800 5050 50  0001 C CNN
+F 4 "TP_SW5" H 6500 5250 50  0000 L CNN "Name"
 	1    6600 5050
 	1    0    0    -1
@@
 AR Path="/5ECF2F45/5EBA759A" Ref="R404"  Part="1"
 F 0 "R404" V 8000 1400 50  0000 L CNN
-F 1 "R43K0" V 7800 1350 50  0000 L CNN
+F 1 "43K0" V 7800 1350 50  0000 L CNN
 F 2 "Resistor_SMD:R_0603_1608Metric_Pad1.05x0.95mm_HandSolder" V 7830 1500 50  0001 C CNN
 F 3 "https://www.yageo.com/upload/media/product/productsearch/datasheet/rchip/PYu-RC_Group_51_RoHS_L_10.pdf" H 7900 1500 50  0001 C CNN
@@
 Text HLabel 5100 3300 2    50   Input ~ 0
 SW3
+$Comp
+L Connector:TestPoint TP?
+U 1 1 5EB966B9
+P 4600 1500
+AR Path="/5ECF32A9/5EB966B9" Ref="TP?"  Part="1"
+AR Path="/5ECF2F45/5EB966B9" Ref="TP401"  Part="1"
+F 0 "TP401" H 4500 1800 50  0000 L CNN
+F 1 "Test Point" H 4500 1700 50  0001 L CNN
+F 2 "Connector_Wire:SolderWirePad_1x01_SMD_5x10mm" H 4800 1500 50  0001 C CNN
+F 3 "None" H 4800 1500 50  0001 C CNN
+F 4 "TP_SW1" H 4500 1700 50  0000 L CNN "Name"
+	1    4600 1500
+	1    0    0    -1
+$EndComp
 $EndSCHEMATC

Commit message: Updates to schematic
Switching to ATMega34UF chip.
Parts:
- C401, C402, C403, C404, C405: DigiKey Part No. (none) -> 311-1335-1-ND; Manufacturer (none) -> Yageo; Mftr Part No. Yageo CC0603KPX7R7BB104 -> CC0603KPX7R7BB104
- R401, R402, R405, R407, R409: value 12K0 -> 12k; DigiKey Part No. (none) -> 311-12KGRCT-ND; Manufacturer (none) -> Bourns; Mftr Part No. (none) -> RC0603JR-0712KL
- R403, R404, R406, R408, R410: value 43K0 -> 43k; DigiKey Part No. (none) -> 311-43KGRCT-ND; Manufacturer (none) -> Yageo; Mftr Part No. (none) -> RC0603JR-0743KL
- S401, S402, S403, S404, S405: DigiKey Part No. (none) -> SW423DKR-ND; Manufacturer (none) -> OMRON; Mftr Part No. (none) -> B3FS-1000P
- TP401, TP402, TP403, TP404, TP405: symbol Connector:TestPoint -> Name~Plate~Class~Library:TestPoint; DigiKey Part No. (none) -> None; Manufacturer (none) -> None; Mftr Part No. (none) -> None

Commit message: Updates
Parts:
- S401, S402, S403, S404, S405: footprint Name Plate Class Project:Button B3FS-1000P -> Name_Plate_Class_Project:Button B3FS-1000P; symbol Name~Plate~Class~Library:Button_B3FS-1000P -> Name_Plate_Class_Project:Button_B3FS-1000P
- TP401, TP402, TP403, TP404, TP405: symbol Name~Plate~Class~Library:TestPoint -> Name_Plate_Class_Project:TestPoint
Changed lines of the file:
@@
 $EndDescr
 $Comp
-L Name~Plate~Class~Library:Button_B3FS-1000P S401
+L Name_Plate_Class_Project:Button_B3FS-1000P S401
 U 1 1 5EB92598
 P 3050 1550
 F 0 "S401" H 2850 1850 50  0000 L CNN
 F 1 "Button B3FS" H 2850 1750 50  0000 L CNN
-F 2 "Name Plate Class Project:Button B3FS-1000P" H 2850 1350 50  0001 L CNN
+F 2 "Name_Plate_Class_Project:Button B3FS-1000P" H 2850 1350 50  0001 L CNN
 F 3 "https://www.omron.co.jp/ecb/products/pdf/b3fs.pdf" H 2850 1250 50  0001 L CNN
 F 4 "SW423DKR-ND" H 3050 1550 50  0001 C CNN "DigiKey Part No."
@@
 	3500 1500 3750 1500
 $Comp
-L Name~Plate~Class~Library:Button_B3FS-1000P S402
+L Name_Plate_Class_Project:Button_B3FS-1000P S402
 U 1 1 5EBA758E
 P 6700 1550
 F 0 "S402" H 6500 1850 50  0000 L CNN
 F 1 "Button B3FS" H 6500 1750 50  0000 L CNN
-F 2 "Name Plate Class Project:Button B3FS-1000P" H 6500 1350 50  0001 L CNN
+F 2 "Name_Plate_Class_Project:Button B3FS-1000P" H 6500 1350 50  0001 L CNN
 F 3 "https://www.omron.co.jp/ecb/products/pdf/b3fs.pdf" H 6500 1250 50  0001 L CNN
 F 4 "SW423DKR-ND" H 6700 1550 50  0001 C CNN "DigiKey Part No."
@@
 $EndComp
 $Comp
-L Name~Plate~Class~Library:TestPoint TP?
+L Name_Plate_Class_Project:TestPoint TP?
 U 1 1 5EBA75BA
 P 8250 1500
 AR Path="/5ECF32A9/5EBA75BA" Ref="TP?"  Part="1"
 AR Path="/5ECF2F45/5EBA75BA" Ref="TP402"  Part="1"
+AR Path="/5EBA75BA" Ref="TP402"  Part="1"
 F 0 "TP402" H 8150 1800 50  0000 L CNN
 F 1 "Test Point" H 8150 1700 50  0001 L CNN
@@
 	7150 1500 7400 1500
 $Comp
-L Name~Plate~Class~Library:Button_B3FS-1000P S403
+L Name_Plate_Class_Project:Button_B3FS-1000P S403
 U 1 1 5EBAED91
 P 3050 3350
 F 0 "S403" H 2850 3650 50  0000 L CNN
 F 1 "Button B3FS" H 2850 3550 50  0000 L CNN
-F 2 "Name Plate Class Project:Button B3FS-1000P" H 2850 3150 50  0001 L CNN
+F 2 "Name_Plate_Class_Project:Button B3FS-1000P" H 2850 3150 50  0001 L CNN
 F 3 "https://www.omron.co.jp/ecb/products/pdf/b3fs.pdf" H 2850 3050 50  0001 L CNN
 F 4 "SW423DKR-ND" H 3050 3350 50  0001 C CNN "DigiKey Part No."
@@
 $EndComp
 $Comp
-L Name~Plate~Class~Library:TestPoint TP?
+L Name_Plate_Class_Project:TestPoint TP?
 U 1 1 5EBAEDBD
 P 4600 3300
 AR Path="/5ECF32A9/5EBAEDBD" Ref="TP?"  Part="1"
 AR Path="/5ECF2F45/5EBAEDBD" Ref="TP403"  Part="1"
+AR Path="/5EBAEDBD" Ref="TP403"  Part="1"
 F 0 "TP403" H 4500 3600 50  0000 L CNN
 F 1 "Test Point" H 4500 3500 50  0001 L CNN
@@
 	3500 3300 3750 3300
 $Comp
-L Name~Plate~Class~Library:Button_B3FS-1000P S404
+L Name_Plate_Class_Project:Button_B3FS-1000P S404
 U 1 1 5EBB48AD
 P 6700 3350
 F 0 "S404" H 6500 3650 50  0000 L CNN
 F 1 "Button B3FS" H 6500 3550 50  0000 L CNN
-F 2 "Name Plate Class Project:Button B3FS-1000P" H 6500 3150 50  0001 L CNN
+F 2 "Name_Plate_Class_Project:Button B3FS-1000P" H 6500 3150 50  0001 L CNN
 F 3 "https://www.omron.co.jp/ecb/products/pdf/b3fs.pdf" H 6500 3050 50  0001 L CNN
 F 4 "SW423DKR-ND" H 6700 3350 50  0001 C CNN "DigiKey Part No."
@@
 $EndComp
 $Comp
-L Name~Plate~Class~Library:TestPoint TP?
+L Name_Plate_Class_Project:TestPoint TP?
 U 1 1 5EBB48D9
 P 8250 3300
 AR Path="/5ECF32A9/5EBB48D9" Ref="TP?"  Part="1"
 AR Path="/5ECF2F45/5EBB48D9" Ref="TP404"  Part="1"
+AR Path="/5EBB48D9" Ref="TP404"  Part="1"
 F 0 "TP404" H 8150 3600 50  0000 L CNN
 F 1 "Test Point" H 8150 3500 50  0001 L CNN
@@
 Connection ~ 7150 3300
 $Comp
-L Name~Plate~Class~Library:Button_B3FS-1000P S405
+L Name_Plate_Class_Project:Button_B3FS-1000P S405
 U 1 1 5EBBC6F1
 P 5050 5100
 F 0 "S405" H 4850 5400 50  0000 L CNN
 F 1 "Button B3FS" H 4850 5300 50  0000 L CNN
-F 2 "Name Plate Class Project:Button B3FS-1000P" H 4850 4900 50  0001 L CNN
+F 2 "Name_Plate_Class_Project:Button B3FS-1000P" H 4850 4900 50  0001 L CNN
 F 3 "https://www.omron.co.jp/ecb/products/pdf/b3fs.pdf" H 4850 4800 50  0001 L CNN
 F 4 "SW423DKR-ND" H 5050 5100 50  0001 C CNN "DigiKey Part No."
@@
 $EndComp
 $Comp
-L Name~Plate~Class~Library:TestPoint TP?
+L Name_Plate_Class_Project:TestPoint TP?
 U 1 1 5EBBC71D
 P 6600 5050
 AR Path="/5ECF32A9/5EBBC71D" Ref="TP?"  Part="1"
 AR Path="/5ECF2F45/5EBBC71D" Ref="TP405"  Part="1"
+AR Path="/5EBBC71D" Ref="TP405"  Part="1"
 F 0 "TP405" H 6500 5350 50  0000 L CNN
 F 1 "Test Point" H 6500 5250 50  0001 L CNN
@@
 SW3
 $Comp
-L Name~Plate~Class~Library:TestPoint TP?
+L Name_Plate_Class_Project:TestPoint TP?
 U 1 1 5EB966B9
 P 4600 1500
 AR Path="/5ECF32A9/5EB966B9" Ref="TP?"  Part="1"
 AR Path="/5ECF2F45/5EB966B9" Ref="TP401"  Part="1"
+AR Path="/5EB966B9" Ref="TP401"  Part="1"
 F 0 "TP401" H 4500 1800 50  0000 L CNN
 F 1 "Test Point" H 4500 1700 50  0001 L CNN

Commit message: PCB Layout
Parts:
- S401, S402, S403, S404, S405: footprint Name_Plate_Class_Project:Button B3FS-1000P -> Name_Plate_Class_Project:Button_B3FS-1000P
- TP401, TP402, TP403, TP404, TP405: footprint Connector_Wire:SolderWirePad_1x01_SMD_5x10mm -> FrequentlyUsed:Pad_2.5-2.5
Changed lines of the file:
@@
 F 0 "S401" H 2850 1850 50  0000 L CNN
 F 1 "Button B3FS" H 2850 1750 50  0000 L CNN
-F 2 "Name_Plate_Class_Project:Button B3FS-1000P" H 2850 1350 50  0001 L CNN
+F 2 "Name_Plate_Class_Project:Button_B3FS-1000P" H 2850 1350 50  0001 L CNN
 F 3 "https://www.omron.co.jp/ecb/products/pdf/b3fs.pdf" H 2850 1250 50  0001 L CNN
 F 4 "SW423DKR-ND" H 3050 1550 50  0001 C CNN "DigiKey Part No."
@@
 F 0 "S402" H 6500 1850 50  0000 L CNN
 F 1 "Button B3FS" H 6500 1750 50  0000 L CNN
-F 2 "Name_Plate_Class_Project:Button B3FS-1000P" H 6500 1350 50  0001 L CNN
+F 2 "Name_Plate_Class_Project:Button_B3FS-1000P" H 6500 1350 50  0001 L CNN
 F 3 "https://www.omron.co.jp/ecb/products/pdf/b3fs.pdf" H 6500 1250 50  0001 L CNN
 F 4 "SW423DKR-ND" H 6700 1550 50  0001 C CNN "DigiKey Part No."
@@
 F 0 "TP402" H 8150 1800 50  0000 L CNN
 F 1 "Test Point" H 8150 1700 50  0001 L CNN
-F 2 "Connector_Wire:SolderWirePad_1x01_SMD_5x10mm" H 8450 1500 50  0001 C CNN
+F 2 "FrequentlyUsed:Pad_2.5-2.5" H 8450 1500 50  0001 C CNN
 F 3 "None" H 8450 1500 50  0001 C CNN
 F 4 "TP_SW2" H 8150 1700 50  0000 L CNN "Name"
@@
 F 0 "S403" H 2850 3650 50  0000 L CNN
 F 1 "Button B3FS" H 2850 3550 50  0000 L CNN
-F 2 "Name_Plate_Class_Project:Button B3FS-1000P" H 2850 3150 50  0001 L CNN
+F 2 "Name_Plate_Class_Project:Button_B3FS-1000P" H 2850 3150 50  0001 L CNN
 F 3 "https://www.omron.co.jp/ecb/products/pdf/b3fs.pdf" H 2850 3050 50  0001 L CNN
 F 4 "SW423DKR-ND" H 3050 3350 50  0001 C CNN "DigiKey Part No."
@@
 F 0 "TP403" H 4500 3600 50  0000 L CNN
 F 1 "Test Point" H 4500 3500 50  0001 L CNN
-F 2 "Connector_Wire:SolderWirePad_1x01_SMD_5x10mm" H 4800 3300 50  0001 C CNN
+F 2 "FrequentlyUsed:Pad_2.5-2.5" H 4800 3300 50  0001 C CNN
 F 3 "None" H 4800 3300 50  0001 C CNN
 F 4 "TP_SW3" H 4500 3500 50  0000 L CNN "Name"
@@
 F 0 "S404" H 6500 3650 50  0000 L CNN
 F 1 "Button B3FS" H 6500 3550 50  0000 L CNN
-F 2 "Name_Plate_Class_Project:Button B3FS-1000P" H 6500 3150 50  0001 L CNN
+F 2 "Name_Plate_Class_Project:Button_B3FS-1000P" H 6500 3150 50  0001 L CNN
 F 3 "https://www.omron.co.jp/ecb/products/pdf/b3fs.pdf" H 6500 3050 50  0001 L CNN
 F 4 "SW423DKR-ND" H 6700 3350 50  0001 C CNN "DigiKey Part No."
@@
 F 0 "TP404" H 8150 3600 50  0000 L CNN
 F 1 "Test Point" H 8150 3500 50  0001 L CNN
-F 2 "Connector_Wire:SolderWirePad_1x01_SMD_5x10mm" H 8450 3300 50  0001 C CNN
+F 2 "FrequentlyUsed:Pad_2.5-2.5" H 8450 3300 50  0001 C CNN
 F 3 "None" H 8450 3300 50  0001 C CNN
 F 4 "TP_SW4" H 8150 3500 50  0000 L CNN "Name"
@@
 F 0 "S405" H 4850 5400 50  0000 L CNN
 F 1 "Button B3FS" H 4850 5300 50  0000 L CNN
-F 2 "Name_Plate_Class_Project:Button B3FS-1000P" H 4850 4900 50  0001 L CNN
+F 2 "Name_Plate_Class_Project:Button_B3FS-1000P" H 4850 4900 50  0001 L CNN
 F 3 "https://www.omron.co.jp/ecb/products/pdf/b3fs.pdf" H 4850 4800 50  0001 L CNN
 F 4 "SW423DKR-ND" H 5050 5100 50  0001 C CNN "DigiKey Part No."
@@
 F 0 "TP405" H 6500 5350 50  0000 L CNN
 F 1 "Test Point" H 6500 5250 50  0001 L CNN
-F 2 "Connector_Wire:SolderWirePad_1x01_SMD_5x10mm" H 6800 5050 50  0001 C CNN
+F 2 "FrequentlyUsed:Pad_2.5-2.5" H 6800 5050 50  0001 C CNN
 F 3 "None" H 6800 5050 50  0001 C CNN
 F 4 "TP_SW5" H 6500 5250 50  0000 L CNN "Name"
@@
 F 0 "TP401" H 4500 1800 50  0000 L CNN
 F 1 "Test Point" H 4500 1700 50  0001 L CNN
-F 2 "Connector_Wire:SolderWirePad_1x01_SMD_5x10mm" H 4800 1500 50  0001 C CNN
+F 2 "FrequentlyUsed:Pad_2.5-2.5" H 4800 1500 50  0001 C CNN
 F 3 "None" H 4800 1500 50  0001 C CNN
 F 4 "TP_SW1" H 4500 1700 50  0000 L CNN "Name"
