File: Page 6.sch (KiCad schematic (older format))
At the start: 17 parts, among them U601 BNO055, U602 BME280, Y601 32.7680 kHz

Commit message: PCB Layout
Parts:
- TP601, TP602, TP603, TP604: footprint Connector_Wire:SolderWirePad_1x01_SMD_5x10mm -> FrequentlyUsed:Pad_2.5-2.5
Changed lines of the file:
@@
 F 0 "TP604" H 2000 3750 50  0000 R CNN
 F 1 "Test Point" H 2000 3850 50  0001 R CNN
-F 2 "Connector_Wire:SolderWirePad_1x01_SMD_5x10mm" H 2250 3700 50  0001 C CNN
+F 2 "FrequentlyUsed:Pad_2.5-2.5" H 2250 3700 50  0001 C CNN
 F 3 "None" H 2250 3700 50  0001 C CNN
 F 4 "TP_SCL" H 2000 3850 50  0000 R CNN "Name"
@@
 F 0 "TP603" H 2100 3750 50  0000 L CNN
 F 1 "Test Point" H 2100 3650 50  0001 L CNN
-F 2 "Connector_Wire:SolderWirePad_1x01_SMD_5x10mm" H 2250 3600 50  0001 C CNN
+F 2 "FrequentlyUsed:Pad_2.5-2.5" H 2250 3600 50  0001 C CNN
 F 3 "None" H 2250 3600 50  0001 C CNN
 F 4 "TP_SDA" H 2100 3650 50  0000 L CNN "Name"
@@
 F 0 "TP602" H 2100 3250 50  0000 L CNN
 F 1 "Test Point" H 2100 3150 50  0001 L CNN
-F 2 "Connector_Wire:SolderWirePad_1x01_SMD_5x10mm" H 2250 3100 50  0001 C CNN
+F 2 "FrequentlyUsed:Pad_2.5-2.5" H 2250 3100 50  0001 C CNN
 F 3 "None" H 2250 3100 50  0001 C CNN
 F 4 "TP_IMU_INT" H 2100 3150 50  0000 L CNN "Name"
@@
 F 0 "TP601" H 2100 3050 50  0000 L CNN
 F 1 "Test Point" H 2100 2950 50  0001 L CNN
-F 2 "Connector_Wire:SolderWirePad_1x01_SMD_5x10mm" H 2250 2900 50  0001 C CNN
+F 2 "FrequentlyUsed:Pad_2.5-2.5" H 2250 2900 50  0001 C CNN
 F 3 "None" H 2250 2900 50  0001 C CNN
 F 4 "TP_nRST" H 2100 2950 50  0000 L CNN "Name"
