File: Name Plate Class Project.kicad_pcb (KiCad board)
At the start: 2 copper layers, 77.5 x 60 mm, 24 parts, among them J101 CONN HEADER SMD 6POS 2.54MM, U1 ATmega328P-AU, U801 MCP7940N-xSN, Y101 16.00 MHz, Y801 32.7680 kHz

Commit message: Updates
Parts:
- removed U801: MCP7940N-xSN, Package_SO:SOIC-8_3.9x4.9mm_P1.27mm
- added C201: 0.1uF, Capacitor_SMD:C_0603_1608Metric_Pad1.05x0.95mm_HandSolder, F.Cu at (393.2, 7.85)
- added C202: 22uF, Name Plate Class Project:CAP_430X430N, F.Cu at (400.9, 4.81)
- added C203: 0.1uF, Capacitor_SMD:C_0603_1608Metric_Pad1.05x0.95mm_HandSolder, F.Cu at (407.1, 7.79)
- added C204: 0.1uF, Capacitor_SMD:C_0603_1608Metric_Pad1.05x0.95mm_HandSolder, F.Cu at (412.9, 2.09)
- added C205: 22uF, Name Plate Class Project:CAP_430X430N, F.Cu at (414.0, -6.74)
- added C301: 10uF, Capacitor_SMD:C_0805_2012Metric_Pad1.15x1.40mm_HandSolder, F.Cu at (401.2, 27.4)
- added C305: 0.1uF, Capacitor_SMD:C_0603_1608Metric_Pad1.05x0.95mm_HandSolder, F.Cu at (424.4, 15.7)
- added C306: 0.1uF, Capacitor_SMD:C_0603_1608Metric_Pad1.05x0.95mm_HandSolder, F.Cu at (414.5, 28.9)
- added C307: 0.1uF, Capacitor_SMD:C_0603_1608Metric_Pad1.05x0.95mm_HandSolder, F.Cu at (424.4, 18.2)
- added C308: 0.1uF, Capacitor_SMD:C_0603_1608Metric_Pad1.05x0.95mm_HandSolder, F.Cu at (405.8, 28.9)
- added C401: 0.1uF, Capacitor_SMD:C_0603_1608Metric_Pad1.05x0.95mm_HandSolder, F.Cu at (394.0, -15.2)
- added C402: 0.1uF, Capacitor_SMD:C_0603_1608Metric_Pad1.05x0.95mm_HandSolder, F.Cu at (398.3, -17.7)
- added C403: 0.1uF, Capacitor_SMD:C_0603_1608Metric_Pad1.05x0.95mm_HandSolder, F.Cu at (389.6, -17.7)
- added C404: 0.1uF, Capacitor_SMD:C_0603_1608Metric_Pad1.05x0.95mm_HandSolder, F.Cu at (394.0, -17.7)
- added C405: 0.1uF, Capacitor_SMD:C_0603_1608Metric_Pad1.05x0.95mm_HandSolder, F.Cu at (420.1, -37.0)
- added C501: 0.1uF, Capacitor_SMD:C_0603_1608Metric_Pad1.05x0.95mm_HandSolder, F.Cu at (325.6, 41.2)
- added C502: 4.7uF, Capacitor_SMD:C_0603_1608Metric_Pad1.05x0.95mm_HandSolder, F.Cu at (325.6, 43.7)
- added C601: 0.1uF, Capacitor_SMD:C_0603_1608Metric_Pad1.05x0.95mm_HandSolder, F.Cu at (383.1, 15.7)
- added C602: 0.1uF, Capacitor_SMD:C_0603_1608Metric_Pad1.05x0.95mm_HandSolder, F.Cu at (383.1, 18.2)
- added C701: 0.1uF, Capacitor_SMD:C_0603_1608Metric_Pad1.05x0.95mm_HandSolder, F.Cu at (391.7, 31.2)
- added C702: 6.8nF, Capacitor_SMD:C_0603_1608Metric_Pad1.05x0.95mm_HandSolder, F.Cu at (385.0, 43.2)
- added C703: 0.12uF, Capacitor_SMD:C_0805_2012Metric_Pad1.15x1.40mm_HandSolder, F.Cu at (385.2, 40.5)
- added C704: 0.1uF, Capacitor_SMD:C_0603_1608Metric_Pad1.05x0.95mm_HandSolder, F.Cu at (391.7, 33.7)
- added C705: 10pF, Capacitor_SMD:C_0603_1608Metric_Pad1.05x0.95mm_HandSolder, F.Cu at (389.8, 40.3)
- added C706: 10pF, Capacitor_SMD:C_0603_1608Metric_Pad1.05x0.95mm_HandSolder, F.Cu at (391.7, 36.2)
- added C901: 0.1uF, Capacitor_SMD:C_0603_1608Metric_Pad1.05x0.95mm_HandSolder, F.Cu at (268.6, 20.3)
- added D301: WS2812B, LED_SMD:LED_WS2812B_PLCC4_5.0x5.0mm_P3.2mm, F.Cu at (409.6, 17.7)
- added D302: WS2812B, LED_SMD:LED_WS2812B_PLCC4_5.0x5.0mm_P3.2mm, F.Cu at (409.6, 24.3)
- added D303: WS2812B, LED_SMD:LED_WS2812B_PLCC4_5.0x5.0mm_P3.2mm, F.Cu at (418.0, 17.7)
- added D304: WS2812B, LED_SMD:LED_WS2812B_PLCC4_5.0x5.0mm_P3.2mm, F.Cu at (418.0, 24.3)
- added D501: PRTR5V0U2X, Package_TO_SOT_SMD:SOT-143, F.Cu at (353.7, 39.9)
- added J1: Battery Connector, Name Plate Class Project:JST_PH_w_SolderPoints, F.Cu at (389.6, -3.81)
- added J501: USB_B_Mini, Name Plate Class Project:Molex_USB_Mini_B_548190572, F.Cu at (323.6, 33.7)
- added J502: SAMD11 Header, Name Plate Class Project:Molex_PinHeader_2x05, F.Cu at (346.3, 43.2)
- added Q201: BSS138, Package_TO_SOT_SMD:SOT-23, F.Cu at (393.3, 4.32)
- added R201: R100K0, Resistor_SMD:R_0603_1608Metric_Pad1.05x0.95mm_HandSolder, F.Cu at (397.6, 8.99)
- added R202: R100K0, Resistor_SMD:R_0603_1608Metric_Pad1.05x0.95mm_HandSolder, F.Cu at (401.9, 8.99)
- added R301: R22K0, Resistor_SMD:R_0603_1608Metric_Pad1.05x0.95mm_HandSolder, F.Cu at (410.1, 28.9)
- added R401: R12K0, Resistor_SMD:R_0603_1608Metric_Pad1.05x0.95mm_HandSolder, F.Cu at (389.6, -15.2)
- added R402: R43K0, Resistor_SMD:R_0603_1608Metric_Pad1.05x0.95mm_HandSolder, F.Cu at (422.2, -29.4)
- added R403: R12K0, Resistor_SMD:R_0603_1608Metric_Pad1.05x0.95mm_HandSolder, F.Cu at (422.2, -34.5)
- added R404: R43K0, Resistor_SMD:R_0603_1608Metric_Pad1.05x0.95mm_HandSolder, F.Cu at (422.2, -21.9)
- added R405: R12K0, Resistor_SMD:R_0603_1608Metric_Pad1.05x0.95mm_HandSolder, F.Cu at (422.2, -24.4)
- added R406: R43K0, Resistor_SMD:R_0603_1608Metric_Pad1.05x0.95mm_HandSolder, F.Cu at (422.2, -26.9)
- added R407: R12K0, Resistor_SMD:R_0603_1608Metric_Pad1.05x0.95mm_HandSolder, F.Cu at (402.7, -15.2)
- added R408: R43K0, Resistor_SMD:R_0603_1608Metric_Pad1.05x0.95mm_HandSolder, F.Cu at (398.3, -15.2)
- added R409: R12K0, Resistor_SMD:R_0603_1608Metric_Pad1.05x0.95mm_HandSolder, F.Cu at (402.7, -17.7)
- added R410: R43K0, Resistor_SMD:R_0603_1608Metric_Pad1.05x0.95mm_HandSolder, F.Cu at (420.1, -32.0)
- added R501: R10K0, Resistor_SMD:R_0603_1608Metric_Pad1.05x0.95mm_HandSolder, F.Cu at (343.6, 48.7)
- added R502: R1K0, Resistor_SMD:R_0603_1608Metric_Pad1.05x0.95mm_HandSolder, F.Cu at (353.3, 43.5)
- added R503: R1K0, Resistor_SMD:R_0603_1608Metric_Pad1.05x0.95mm_HandSolder, F.Cu at (325.6, 48.7)
- added R504: R1M0, Resistor_SMD:R_0603_1608Metric_Pad1.05x0.95mm_HandSolder, F.Cu at (325.6, 46.2)
- added R701: R10K0, Resistor_SMD:R_0603_1608Metric_Pad1.05x0.95mm_HandSolder, F.Cu at (391.7, 28.7)
- added R702: R10K0, Resistor_SMD:R_0603_1608Metric_Pad1.05x0.95mm_HandSolder, F.Cu at (389.4, 43.2)
- added R901: R22K0, Resistor_SMD:R_0603_1608Metric_Pad1.05x0.95mm_HandSolder, F.Cu at (273.0, 20.3)
- added R902: R22K0, Resistor_SMD:R_0603_1608Metric_Pad1.05x0.95mm_HandSolder, F.Cu at (277.3, 20.3)
- added R903: R22K0, Resistor_SMD:R_0603_1608Metric_Pad1.05x0.95mm_HandSolder, F.Cu at (281.7, 20.3)
- added R904: R22K0, Resistor_SMD:R_0603_1608Metric_Pad1.05x0.95mm_HandSolder, F.Cu at (286.0, 20.3)
- added R905: R22K0, Resistor_SMD:R_0603_1608Metric_Pad1.05x0.95mm_HandSolder, F.Cu at (290.4, 20.3)
- added R906: R22K0, Resistor_SMD:R_0603_1608Metric_Pad1.05x0.95mm_HandSolder, F.Cu at (294.7, 20.3)
- added S201: Battery Switch, Name Plate Class Project:Switch_JS202011SCQN, F.Cu at (386.0, 6.54)
- added S401: Button B3FS, Name Plate Class Project:Button B3FS-1000P, F.Cu at (392.8, -22.9)
- added S402: Button B3FS, Name Plate Class Project:Button B3FS-1000P, F.Cu at (403.6, -22.9)
- added S403: Button B3FS, Name Plate Class Project:Button B3FS-1000P, F.Cu at (412.4, -34.5)
- added S404: Button B3FS, Name Plate Class Project:Button B3FS-1000P, F.Cu at (414.5, -26.8)
- added S405: Button B3FS, Name Plate Class Project:Button B3FS-1000P, F.Cu at (414.5, -19.1)
- added TP201: TP_SWITCH_BATTERY, Connector_Wire:SolderWirePad_1x01_SMD_5x10mm, F.Cu at (399.5, -3.89)
- added TP202: TP_5V, Connector_Wire:SolderWirePad_1x01_SMD_5x10mm, F.Cu at (406.0, -3.89)
- added TP301: TP_ADDR_LED, Connector_Wire:SolderWirePad_1x01_SMD_5x10mm, F.Cu at (402.1, 20.2)
- added TP401: TP_SW1, Connector_Wire:SolderWirePad_1x01_SMD_5x10mm, F.Cu at (397.3, -32.5)
- added TP402: TP_SW1, Connector_Wire:SolderWirePad_1x01_SMD_5x10mm, F.Cu at (390.7, -32.5)
- added TP403: TP_SW1, Connector_Wire:SolderWirePad_1x01_SMD_5x10mm, F.Cu at (384.2, -20.9)
- added TP404: TP_SW1, Connector_Wire:SolderWirePad_1x01_SMD_5x10mm, F.Cu at (384.2, -32.5)
- added TP405: TP_SW1, Connector_Wire:SolderWirePad_1x01_SMD_5x10mm, F.Cu at (403.8, -32.5)
- added TP501: TP_SAMD11_nRST, Connector_Wire:SolderWirePad_1x01_SMD_5x10mm, F.Cu at (338.2, 44.8)
- added TP502: TP_MEGA_nRST, Connector_Wire:SolderWirePad_1x01_SMD_5x10mm, F.Cu at (331.6, 44.8)
- added TP503: TP_SAMD11_TX_MEGA_RX, Connector_Wire:SolderWirePad_1x01_SMD_5x10mm, F.Cu at (338.2, 33.2)
- added TP504: TP_SAMD11_RX_MEGA_TX, Connector_Wire:SolderWirePad_1x01_SMD_5x10mm, F.Cu at (331.6, 33.2)
- added TP505: TP_SAMD11_SWCLK, Connector_Wire:SolderWirePad_1x01_SMD_5x10mm, F.Cu at (320.2, 45.7)
- added TP506: TP_SAMD11_SWDIO, Connector_Wire:SolderWirePad_1x01_SMD_5x10mm, F.Cu at (344.7, 33.2)
- added TP701: TP_nRST, Connector_Wire:SolderWirePad_1x01_SMD_5x10mm, F.Cu at (366.0, 38.9)
- added TP702: TP_IMU_INT, Connector_Wire:SolderWirePad_1x01_SMD_5x10mm, F.Cu at (379.7, 33.2)
- added TP703: TP_SDA, Connector_Wire:SolderWirePad_1x01_SMD_5x10mm, F.Cu at (372.6, 38.9)
- added TP704: TP_SCL, Connector_Wire:SolderWirePad_1x01_SMD_5x10mm, F.Cu at (386.2, 33.2)
- added TP901: TP_SPI_MISO, Connector_Wire:SolderWirePad_1x01_SMD_5x10mm, F.Cu at (350.3, -20.9)
- added TP902: TP_FONT_nSELECT, Connector_Wire:SolderWirePad_1x01_SMD_5x10mm, F.Cu at (356.8, -32.5)
- added TP903: TP_SPI_CLK, Connector_Wire:SolderWirePad_1x01_SMD_5x10mm, F.Cu at (343.7, -9.35)
- added TP904: TP_SPI_MOSI, Connector_Wire:SolderWirePad_1x01_SMD_5x10mm, F.Cu at (350.3, -32.5)
- added TP905: TP_DC, Connector_Wire:SolderWirePad_1x01_SMD_5x10mm, F.Cu at (343.7, -32.5)
- added TP906: TP_LCD_nCS, Connector_Wire:SolderWirePad_1x01_SMD_5x10mm, F.Cu at (343.7, -20.9)
- added U201: MIC5219-5.0YM5-TR, Package_TO_SOT_SMD:SOT-23-5_HandSoldering, F.Cu at (407.9, 4.21)
- added U202: MIC5219-5.0YM5-TR, Package_TO_SOT_SMD:SOT-23-5_HandSoldering, F.Cu at (412.2, -1.49)
- added U3: MCP7940N-xSN, Package_SO:SOIC-8_3.9x4.9mm_P1.27mm, F.Cu at (303.0, 36.3)
- added U501: ATSAMD11C14A-SS, Package_SO:SOIC-14_3.9x8.7mm_P1.27mm, F.Cu at (352.2, 32.6)
- added U601: BME280, Package_LGA:Bosch_LGA-8_2.5x2.5mm_P0.65mm_ClockwisePinNumbering, F.Cu at (387.2, 16.5)
- added U701: BNO055, Package_LGA:LGA-28_5.2x3.8mm_P0.5mm, F.Cu at (379.3, 41.8)
- added Y701: 32.7680 kHz, Name Plate Class Project:Oscillator_MC-405_32.7680K-D__ROHS, F.Cu at (369.6, 30.3)
- C309: value 22uF -> 2.2uF
- J101: value CONN HEADER SMD 6POS 2.54MM -> Conn Header SMD
- LCD1: value LCD 2.4" SPI ER-TFTM024-3 -> LCD 2.4"
- moved C803 154.4 mm to (268.6, 50.1)
- moved R801 150.1 mm to (277.3, 50.1)
- moved B801 145.8 mm to (282.6, 37.5)
- moved C802 145.8 mm to (273.0, 50.1)
- moved Y801 145.8 mm to (305.6, 30.3)
- moved C801 132.8 mm to (281.7, 50.1)
- moved LCD1 0.64 mm to (112.0, 125.4)
Connections:
- net /Page 1/MISO renamed SPI_MISO
- net /Page 1/MOSI renamed SPI_MOSI
- net /Page 1/SCK renamed SPI_CLK
- C309 pad 1: (no net) -> BUZZER
- LCD1 pad 1: (no net) -> GND
- LCD1 pad 23: (no net) -> LCD_nCS
- LCD1 pad 24: /Page 1/LCD_CLK -> /Page 9/LCD_SPI_CLK
- LCD1 pad 25: (no net) -> LCD_DC
- LCD1 pad 27: (no net) -> /Page 9/LCD_SPI_MOSI
- LCD1 pad 28: (no net) -> /Page 9/LCD_SPI_MISO
- LCD1 pad 32: (no net) -> /Page 9/LCD_SPI_MISO
- LCD1 pad 33: /Page 1/LCD_CLK -> (no net)
- LCD1 pad 34: (no net) -> /Page 9/LCD_SPI_MOSI
- LCD1 pad 36: (no net) -> /Page 9/LCD_FONT_nCS
- R101 pad 1: +3V3 -> Net-(R101-Pad1)
- R102 pad 1: +3V3 -> Net-(R101-Pad1)
- R103 pad 1: +3V3 -> Net-(R101-Pad1)
- R801 pad 2: /Page 9/RTC_INT -> /Page 8/RTC_INT
- U1 pad 1: (no net) -> SW1
- U1 pad 11: (no net) -> SW5
- U1 pad 13: (no net) -> BUZZER
- U1 pad 14: (no net) -> LCD_DC
- U1 pad 2: (no net) -> SW2
- U1 pad 23: (no net) -> IMU_INT
- U1 pad 25: (no net) -> LCD_FONT_nSELECT
- U1 pad 26: (no net) -> ADDR_LED
- U1 pad 30: (no net) -> MEGA_RX
- U1 pad 31: (no net) -> MEGA_TX
- U1 pad 32: (no net) -> LCD_nCS
- U1 pad 9: (no net) -> SW3
- Y801 pad 1: Net-(C802-Pad2) -> Net-(C803-Pad2)
- Y801 pad 2: Net-(C803-Pad2) -> Net-(C802-Pad2)

Commit message: Updates
Parts:
- removed the C301 at (401.2, 27.4)
- removed the C701 at (391.7, 31.2)
- removed the C702 at (385.0, 43.2)
- removed the C703 at (385.2, 40.5)
- removed C704: 0.1uF, Capacitor_SMD:C_0603_1608Metric_Pad1.05x0.95mm_HandSolder
- removed C705, C706: 10pF, Capacitor_SMD:C_0603_1608Metric_Pad1.05x0.95mm_HandSolder
- removed R701, R702: R10K0, Resistor_SMD:R_0603_1608Metric_Pad1.05x0.95mm_HandSolder
- removed the R801 at (277.3, 50.1)
- removed TP701: TP_nRST, Connector_Wire:SolderWirePad_1x01_SMD_5x10mm
- removed TP702: TP_IMU_INT, Connector_Wire:SolderWirePad_1x01_SMD_5x10mm
- removed TP703: TP_SDA, Connector_Wire:SolderWirePad_1x01_SMD_5x10mm
- removed TP704: TP_SCL, Connector_Wire:SolderWirePad_1x01_SMD_5x10mm
- removed the U701 at (379.3, 41.8)
- removed the Y701 at (369.6, 30.3)
- added C203: 0.1uF, Capacitor_SMD:C_0603_1608Metric_Pad1.05x0.95mm_HandSolder, F.Cu at (238.3, -15.0)
- added C302: 10uF, Name_Plate_Class_Project:CAP_430X430N, F.Cu at (270.4, -35.0)
- added C601: 0.1uF, Capacitor_SMD:C_0603_1608Metric_Pad1.05x0.95mm_HandSolder, F.Cu at (256.2, -22.1)
- added C602: 6.8nF, Capacitor_SMD:C_0603_1608Metric_Pad1.05x0.95mm_HandSolder, F.Cu at (258.5, -31.6)
- added C603: 0.12uF, Capacitor_SMD:C_0805_2012Metric_HandSolder, F.Cu at (252.1, -24.9)
- added C604: 0.1uF, Capacitor_SMD:C_0603_1608Metric_Pad1.05x0.95mm_HandSolder, F.Cu at (251.9, -22.1)
- added C607: 10pF, Capacitor_SMD:C_0603_1608Metric_Pad1.05x0.95mm_HandSolder, F.Cu at (258.5, -36.6)
- added C608: 10pF, Capacitor_SMD:C_0603_1608Metric_Pad1.05x0.95mm_HandSolder, F.Cu at (258.5, -34.1)
- added R104: 10k, Resistor_SMD:R_0603_1608Metric_Pad1.05x0.95mm_HandSolder, F.Cu at (256.0, -12.5)
- added R105: 10k, Resistor_SMD:R_0603_1608Metric_Pad1.05x0.95mm_HandSolder, F.Cu at (256.0, -15.0)
- added R201: Jumper, Resistor_SMD:R_0603_1608Metric_Pad1.05x0.95mm_HandSolder, F.Cu at (242.7, -15.0)
- added R601: 10k, Resistor_SMD:R_0603_1608Metric_Pad1.05x0.95mm_HandSolder, F.Cu at (256.6, -25.1)
- added R602: 10k, Resistor_SMD:R_0603_1608Metric_Pad1.05x0.95mm_HandSolder, F.Cu at (258.5, -29.1)
- added TP203: Test Point, Connector_Wire:SolderWirePad_1x01_SMD_5x10mm, F.Cu at (232.8, -10.5)
- added TP601: Test Point, Connector_Wire:SolderWirePad_1x01_SMD_5x10mm, F.Cu at (232.8, -26.4)
- added TP602: Test Point, Connector_Wire:SolderWirePad_1x01_SMD_5x10mm, F.Cu at (246.5, -32.1)
- added TP603: Test Point, Connector_Wire:SolderWirePad_1x01_SMD_5x10mm, F.Cu at (239.4, -26.4)
- added TP604: Test Point, Connector_Wire:SolderWirePad_1x01_SMD_5x10mm, F.Cu at (253.1, -32.1)
- added U601: BNO055, Package_LGA:LGA-28_5.2x3.8mm_P0.5mm, F.Cu at (246.2, -23.6)
- added Y601: 32.7680 kHz, Name_Plate_Class_Project:Oscillator_MC-405_32.7680K-D__ROHS, F.Cu at (236.4, -35.0)
- B701: renamed from B801; footprint Name Plate Class Project:BAT_BK-883 -> Name_Plate_Class_Project:BAT_BK-883
- C202: value 22uF -> 10uF; footprint Name Plate Class Project:CAP_430X430N -> Name_Plate_Class_Project:CAP_430X430N
- C204: renamed from C205; value 22uF -> 10uF; footprint Name Plate Class Project:CAP_430X430N -> Name_Plate_Class_Project:CAP_430X430N
- C205: renamed from C203; value 0.1uF -> 470pF
- C206: renamed from C204; value 0.1uF -> 470pF
- C301: renamed from C309; value 2.2uF -> 10uF; footprint Name Plate Class Project:CAP_430X430N -> Name_Plate_Class_Project:CAP_430X430N
- D305: footprint Name Plate Class Project:LED_G-GX -> Name_Plate_Class_Project:LED_G-GX
- D501: value PRTR5V0U2X -> PRTR5V0U2X,215
- J101: footprint Name Plate Class Project:Molex_PinHeader_2x03 -> Name_Plate_Class_Project:Molex_PinHeader_2x03
- J201: renamed from J1; footprint Name Plate Class Project:JST_PH_w_SolderPoints -> Name_Plate_Class_Project:JST_PH_w_SolderPoints
- J501: footprint Name Plate Class Project:Molex_USB_Mini_B_548190572 -> Name_Plate_Class_Project:Molex_USB_Mini_B_548190572
- J502: footprint Name Plate Class Project:Molex_PinHeader_2x05 -> Name_Plate_Class_Project:Molex_PinHeader_2x05
- J801: renamed from LCD1; value LCD 2.4" -> DNP; footprint Name Plate Class Project:LCD_ER-TFTM024-3 -> Name_Plate_Class_Project:LCD_ER-TFTM024-3_SMD
- LS301: footprint Name Plate Class Project:Buzzer_TDK_PS1240P02BT_D12.2mm_H6.5mm -> Name_Plate_Class_Project:Buzzer_TDK_PS1240P02BT_D12.2mm_H6.5mm
- R101: renamed from R103; value R10K0 -> 10k
- R102: renamed from R101; value R4k75 -> 4.75k
- R103: renamed from R102; value R4k75 -> 4.75k
- R202: renamed from R201; value R100K0 -> 100k
- R203: renamed from R202; value R100K0 -> 100k
- R301: value R22K0 -> 22
- R302: value 470k -> 470
- R401, R405, R407, R409: value R12K0 -> 12k
- R402: renamed from R403; value R12K0 -> 12k
- R403: renamed from R402; value R43K0 -> 43k
- R404, R406, R408, R410: value R43K0 -> 43k
- R501: value R10K0 -> 10k
- R502, R503: value R1K0 -> 1k
- R504: value R1M0 -> 1M
- R801: renamed from R901; value R22K0 -> 22
- R802: renamed from R902; value R22K0 -> 22
- R803: renamed from R903; value R22K0 -> 22
- R804: renamed from R904; value R22K0 -> 22
- R805: renamed from R905; value R22K0 -> 22
- R806: renamed from R906; value R22K0 -> 22
- S201: footprint Name Plate Class Project:Switch_JS202011SCQN -> Name_Plate_Class_Project:Switch_JS202011SCQN
- S401, S402, S403, S404, S405: footprint Name Plate Class Project:Button B3FS-1000P -> Name_Plate_Class_Project:Button B3FS-1000P
- TP201: value TP_SWITCH_BATTERY -> Test Point
- TP202: value TP_5V -> Test Point
- TP301: value TP_ADDR_LED -> Test Point
- TP401, TP402, TP403, TP404, TP405: value TP_SW1 -> Test Point
- TP501: value TP_SAMD11_nRST -> Test Point
- TP502: value TP_MEGA_nRST -> Test Point
- TP503: value TP_SAMD11_TX_MEGA_RX -> Test Point
- TP504: value TP_SAMD11_RX_MEGA_TX -> Test Point
- TP505: value TP_SAMD11_SWCLK -> Test Point
- TP506: value TP_SAMD11_SWDIO -> Test Point
- TP801: renamed from TP901; value TP_SPI_MISO -> Test Point
- TP802: renamed from TP902; value TP_FONT_nSELECT -> Test Point
- TP803: renamed from TP903; value TP_SPI_CLK -> Test Point
- TP804: renamed from TP904; value TP_SPI_MOSI -> Test Point
- TP805: renamed from TP905; value TP_DC -> Test Point
- TP806: renamed from TP906; value TP_LCD_nCS -> Test Point
- U202: value MIC5219-5.0YM5-TR -> MIC5219-3.3YM5-TR
- Y101: footprint Name Plate Class Project:Oscillator_ABM3-16.000MHZ-B2-T -> Name_Plate_Class_Project:Oscillator_ABM3-16.000MHZ-B2-T
- Y701: renamed from Y801; footprint Name Plate Class Project:Oscillator_MC-405_32.7680K-D__ROHS -> Name_Plate_Class_Project:Oscillator_MC-405_32.7680K-D__ROHS
- renumbered C106 to C103, C105 to C104, C103 to C105, C104 to C106, C305 to C303, C306 to C304, C307 to C305, C308 to C306, C602 to C605, C601 to C606, C801 to C701, C802 to C702, C803 to C703, C901 to C801, U1 to U101, U601 to U602, U3 to U701
Connections:
- net /Page 9/LCD_FONT_nCS renamed /Page 8/LCD_FONT_nCS
- net /Page 9/LCD_SPI_MISO renamed /Page 8/LCD_SPI_MISO
- net /Page 9/LCD_SPI_MOSI renamed /Page 8/LCD_SPI_MOSI
- net ADDR_LED renamed /Page 1/ADDR_LED
- net BUZZER renamed /Page 1/BUZZER
- net LCD_DC renamed /Page 1/LCD_DC
- net LCD_FONT_nSELECT renamed /Page 1/LCD_FONT_nSELECT
- net LCD_nCS renamed /Page 1/LCD_nCS
- net LED_IND renamed /Page 1/LED_IND
- net MEGA_RX renamed /Page 1/SAMD11_TX_MEGA_RX
- net MEGA_TX renamed /Page 1/SAMD11_RX_MEGA_TX
- net SAMD11_SWCLK renamed /Page 5/SAMD11_SWCLK
- net SAMD11_SWDIO renamed /Page 5/SAMD11_SWDIO
- net SCL renamed /Page 1/SCL
- net SDA renamed /Page 1/SDA
- net SPI_CLK renamed /Page 1/SPI_CLK
- net SPI_MISO renamed /Page 1/SPI_MISO
- net SPI_MOSI renamed /Page 1/SPI_MOSI
- net SW2 renamed /Page 1/SW2
- net SW3 renamed /Page 1/SW3
- net SW5 renamed /Page 1/SW5
- net USB_DM renamed /Page 5/USB_DM
- net USB_DP renamed /Page 5/USB_DP
- C401 pad 1: SW1 -> /Page 1/SW1
- C404 pad 1: SW1 -> /Page 1/SW4
- D501 pad 4: +5V -> VBUS
- J101 pad 5: MEGA_nRST -> /Page 1/MEGA_nRST
- J501 pad 1: +5V -> VBUS
- J502 pad 10: SAMD11_nRST -> /Page 5/SAMD11_nRST
- J801 pad 24: /Page 9/LCD_SPI_CLK -> /Page 8/LCD_SPI_CLK
- J801 pad 33: (no net) -> /Page 8/LCD_SPI_CLK
- Q201 pad 1: +5V -> VBUS
- Q201 pad 2: Net-(Q201-Pad2) -> GND
- Q201 pad 3: GND -> Net-(Q201-Pad3)
- R101 pad 1: Net-(R101-Pad1) -> +3V3
- R101 pad 2: MEGA_nRST -> /Page 1/RTC_INT
- R102 pad 1: Net-(R101-Pad1) -> +3V3
- R103 pad 1: Net-(R101-Pad1) -> +3V3
- R202 pad 1: Net-(Q201-Pad2) -> Net-(Q201-Pad3)
- R203 pad 1: +5V -> VBUS
- R403 pad 2: SW1 -> /Page 1/SW1
- R408 pad 2: SW1 -> /Page 1/SW4
- R501 pad 2: SAMD11_nRST -> /Page 5/SAMD11_nRST
- R803 pad 2: /Page 9/LCD_SPI_CLK -> /Page 8/LCD_SPI_CLK
- TP201 pad 1: Net-(Q201-Pad2) -> (no net)
- TP202 pad 1: +5V -> (no net)
- TP401 pad 1: SW1 -> /Page 1/SW1
- TP404 pad 1: SW1 -> /Page 1/SW4
- TP501 pad 1: SAMD11_nRST -> (no net)
- TP502 pad 1: MEGA_nRST -> /Page 1/MEGA_nRST
- U101 pad 1: SW1 -> /Page 1/SW1
- U101 pad 10: (no net) -> /Page 1/SW4
- U101 pad 23: IMU_INT -> /Page 1/IMU_INT
- U101 pad 24: (no net) -> /Page 1/RTC_INT
- U101 pad 29: MEGA_nRST -> /Page 1/MEGA_nRST
- U201 pad 3: Net-(Q201-Pad2) -> Net-(Q201-Pad3)
- U501 pad 3: MEGA_nRST -> /Page 1/MEGA_nRST
- U501 pad 6: SAMD11_nRST -> /Page 5/SAMD11_nRST
- U701 pad 7: /Page 8/RTC_INT -> /Page 1/RTC_INT

Commit message: PCB Layout
Parts:
- B701, C201, C203, C205, C206, C501, C502, J101, J201, J501, LS301, Q201, R201, R202, R203, R501, R504, S201, U201, U202, U501: moved to B.Cu
- C202, C204: footprint Name_Plate_Class_Project:CAP_430X430N -> Name_Plate_Class_Project:T491A106K010AT; moved to B.Cu
- C301, C302: footprint Name_Plate_Class_Project:CAP_430X430N -> Name_Plate_Class_Project:T491A106K010AT
- D501: footprint Package_TO_SOT_SMD:SOT-143 -> Name_Plate_Class_Project:SOT-143-4; moved to B.Cu
- J502: footprint Name_Plate_Class_Project:Molex_PinHeader_2x05 -> Name_Plate_Class_Project:SAMTEC-FTS-105-01-X-DV; moved to B.Cu
- S401, S402, S403, S404, S405: footprint Name_Plate_Class_Project:Button B3FS-1000P -> Name_Plate_Class_Project:Button_B3FS-1000P
- TP201, TP301, TP401, TP402, TP403, TP404, TP405, TP505, TP506: footprint Connector_Wire:SolderWirePad_1x01_SMD_5x10mm -> FrequentlyUsed:Pad_2.5-2.5; moved to B.Cu
- TP202, TP203, TP501, TP502, TP503, TP504, TP601, TP602, TP603, TP604, TP801, TP802, TP803, TP804, TP805, TP806: footprint Connector_Wire:SolderWirePad_1x01_SMD_5x10mm -> FrequentlyUsed:Pad_2.5-2.5
- moved C303 315.4 mm to (128.1, 123.8), turned to 90 degrees
- moved D301 300.6 mm to (130.5, 129.4)
- moved J201 300.0 mm to (114.5, 116.0)
- moved U201 300.0 mm to (130.5, 118.5)
- moved S201 296.5 mm to (115.5, 128.0)
- moved TP201 296.2 mm to (126.4, 110.9)
- moved C205 296.1 mm to (131.0, 114.8), turned to 180 degrees
- moved U202 292.6 mm to (145.3, 118.5)
- moved R202 292.4 mm to (126.4, 118.3), turned to 270 degrees
- moved C204 291.4 mm to (151.3, 119.5)
- moved C201 291.3 mm to (123.7, 118.3), turned to 90 degrees
- moved C304 287.0 mm to (143.6, 123.8), turned to 90 degrees
- moved R301 287.0 mm to (138.5, 121.8), turned to 180 degrees
- moved C202 286.5 mm to (138.1, 118.8), turned to 90 degrees
- moved C405 286.4 mm to (179.0, 117.6), turned to 90 degrees
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Connections:
- net Net-(C201-Pad1) renamed /Page 2/BSWO
- net Net-(J201-Pad1) renamed /Page 2/B+
- C502 pad 1: Net-(C502-Pad1) -> GND
- C502 pad 2: GND -> Net-(C502-Pad2)
- R504 pad 1: Net-(C502-Pad1) -> GND
- R504 pad 2: GND -> Net-(C502-Pad2)
- TP201 pad 1: (no net) -> Net-(Q201-Pad3)
- TP301 pad 1: /Page 1/ADDR_LED -> Net-(D301-Pad4)
Routing:
- net GND: track 0.00 -> 68.8 mm, vias 0 -> 15
- net +5V: track 0.00 -> 59.4 mm
- net Net-(C502-Pad2): track 0.00 -> 23.6 mm
- net Net-(D303-Pad2): track 0.00 -> 22.7 mm
- net Net-(D301-Pad2): track 0.00 -> 22.7 mm
- net Net-(D302-Pad2): track 0.00 -> 22.5 mm
- net /Page 2/BSWO: track 0.00 -> 21.6 mm
- net /Page 2/B+: track 0.00 -> 20.2 mm
- net /Page 5/SAMD11_SWDIO: track 0.00 -> 19.9 mm
- net /Page 5/SAMD11_SWCLK: track 0.00 -> 19.3 mm
- net /Page 5/SAMD11_nRST: track 0.00 -> 16.5 mm, vias 0 -> 2
- net Net-(D301-Pad4): track 0.00 -> 13.7 mm, vias 0 -> 2
- net Net-(Q201-Pad3): track 0.00 -> 13.2 mm
- net VBUS: track 0.00 -> 12.0 mm
- net /Page 1/SW3: track 0.00 -> 11.9 mm, vias 0 -> 1
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- added copper zone on F.Cu, net +3V3
- added copper zone on B.Cu, net GND
Other:
- board size 77.5 x 60 mm -> 83.5 x 66 mm
- net class Power Main added: clearance 0.2, trace_width 0.5, via_dia 0.8, via_drill 0.4
- board text added: "SAMD11"

Commit message: PCB Update
Parts:
- C701, C702, C703, TP202, TP805, TP806, U701, Y701: moved to B.Cu
- moved R302 223.8 mm to (122.9, 129.5), turned to 270 degrees
- moved D305 220.8 mm to (117.6, 129.3), turned to 180 degrees
- moved TP805 189.6 mm to (139.4, 95.2)
- moved R806 187.8 mm to (123.8, 98.0)
- moved TP806 185.3 mm to (139.3, 99.2)
- moved R805 182.8 mm to (123.8, 95.4), turned to 180 degrees
- moved C801 176.4 mm to (123.2, 120.2)
- moved C301 174.7 mm to (160.0, 87.6), turned to 90 degrees
- moved R803 173.8 mm to (123.8, 92.9), turned to 180 degrees
- moved R804 173.0 mm to (123.8, 80.2), turned to 180 degrees
- moved R802 163.9 mm to (123.8, 77.7), turned to 180 degrees
- moved R801 162.8 mm to (123.8, 85.3), turned to 180 degrees
- moved R602 157.2 mm to (151.9, 86.4), turned to 90 degrees
- moved R601 156.9 mm to (144.5, 84.7)
- moved C608 154.3 mm to (146.6, 70.6), turned to 180 degrees
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Connections:
- B701 pad 1: Net-(B701-Pad1) -> (no net)
- J801 pad 25: /Page 1/LCD_DC -> /Page 8/LCD_DC_R
- R805 pad 2: /Page 1/LCD_DC -> /Page 8/LCD_DC_R
- TP202 pad 1: (no net) -> +5V
- TP203 pad 1: (no net) -> +3V3
- U701 pad 3: Net-(B701-Pad1) -> /Page 7/RTCB+
Routing:
- net GND: track 68.8 -> 129.1 mm, vias 15 -> 20
- net +5V: track 59.4 -> 88.5 mm, vias 0 -> 1
- net /Page 8/LCD_SPI_CLK: track 0.00 -> 20.5 mm, vias 0 -> 2
- net VBUS: track 12.0 -> 29.5 mm, vias 0 -> 2
- net /Page 8/LCD_SPI_MOSI: track 0.00 -> 16.2 mm
- net /Page 7/RTCB+: track 0.00 -> 15.4 mm
- net /Page 1/LCD_nCS: track 0.00 -> 13.2 mm
- net /Page 8/LCD_DC_R: track 0.00 -> 13.0 mm
- net Net-(C703-Pad2): track 0.00 -> 12.2 mm
- net Net-(C702-Pad2): track 0.00 -> 12.2 mm
- net +3V3: track 7.74 -> 19.9 mm, vias 3 -> 7
- net Net-(C607-Pad2): track 0.00 -> 11.5 mm
- net Net-(C608-Pad2): track 0.00 -> 11.5 mm
- net /Page 8/LCD_SPI_MISO: track 0.00 -> 10.0 mm
- net /Page 1/XTAL2: track 0.00 -> 9.42 mm
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Other:
- net class Power Main: via_dia 0.8 -> 1; via_drill 0.4 -> 0.6

Commit message: PCB Update
Parts:
- C607, C608, R104, R502, R503, TP203, TP501, TP502, TP503, TP504, TP601, TP602, TP603, TP604, TP801, TP802, TP803, TP804, Y601: moved to B.Cu
- moved TP802 103.1 mm to (115.5, 73.6), turned to 270 degrees
- moved TP803 86.1 mm to (127.8, 87.7)
- moved TP603 72.3 mm to (174.2, 103.6)
- moved TP604 65.0 mm to (170.2, 103.6)
- moved TP602 63.6 mm to (150.3, 87.8)
- moved TP501 56.2 mm to (117.6, 109.3)
- moved TP601 53.2 mm to (147.8, 83.1)
- moved J101 38.8 mm to (127.5, 78.3), turned to 90 degrees
- moved R103 37.4 mm to (166.1, 108.9)
- moved R104 27.5 mm to (134.4, 96.2)
- moved R102 20.3 mm to (174.0, 112.8), turned to 180 degrees
- moved C605 17.8 mm to (161.8, 89.8), turned to 90 degrees
- moved TP203 17.0 mm to (147.2, 59.0)
- moved U602 13.7 mm to (165.2, 89.9), turned to 180 degrees
- moved C606 12.2 mm to (168.6, 90.1), turned to 270 degrees
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Connections:
- J801 pad 23: /Page 1/LCD_nCS -> /Page 8/LCD_nCS_R
- R806 pad 2: /Page 1/LCD_nCS -> /Page 8/LCD_nCS_R
- TP501 pad 1: (no net) -> /Page 5/SAMD11_nRST
Routing:
- net /Page 1/LED_IND: track 0.00 -> 62.6 mm, vias 0 -> 2
- net /Page 1/LCD_FONT_nSELECT: track 0.00 -> 56.0 mm, vias 0 -> 3
- net /Page 1/SPI_MOSI: track 0.00 -> 52.9 mm, vias 0 -> 2
- net /Page 1/SW1: track 11.5 -> 61.9 mm, vias 1 -> 2
- net /Page 1/SPI_CLK: track 0.00 -> 45.0 mm, vias 0 -> 1
- net /Page 1/SPI_MISO: track 0.00 -> 40.9 mm, vias 0 -> 2
- net /Page 1/SW2: track 11.5 -> 50.2 mm, vias 1 -> 2
- net /Page 1/LCD_DC: track 0.00 -> 33.9 mm, vias 0 -> 2
- net /Page 1/SDA: track 0.00 -> 32.7 mm, vias 0 -> 1
- net /Page 1/RTC_INT: track 0.00 -> 32.6 mm, vias 0 -> 3
- net /Page 1/LCD_nCS: track 13.2 -> 45.7 mm, vias 0 -> 4
- net /Page 1/MEGA_nRST: track 0.00 -> 31.6 mm, vias 0 -> 1
- net /Page 1/SAMD11_RX_MEGA_TX: track 0.00 -> 29.3 mm, vias 0 -> 1
- net /Page 1/SCL: track 0.00 -> 29.1 mm, vias 0 -> 1
- net /Page 1/SAMD11_TX_MEGA_RX: track 0.00 -> 27.1 mm, vias 0 -> 1
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
Commit message: PCB Tweaks
Parts:
- added ?: , , F.Cu at (17.2, 15.2)
- added ?: , , F.Cu at (168.1, 127.2)
- added ?: , , F.Cu at (55.0, 22.1)
- added ?: , , F.Cu at (123.4, 136.9)
- added ?: , , F.Cu at (123.7, 129.3)
- moved TP804 77.9 mm to (148.0, 95.1)
- moved TP801 68.5 mm to (151.2, 95.1)
- moved TP503 54.8 mm to (148.0, 88.5)
- moved TP502 53.5 mm to (136.0, 101.6)
- moved TP504 49.6 mm to (131.5, 87.8)
- moved TP203 39.5 mm to (183.5, 74.8)
- moved R103 8.27 mm to (174.2, 107.1), turned to 180 degrees
- moved C301 8.16 mm to (156.9, 84.6)
- moved TP601 7.88 mm to (141.5, 78.3)
- moved R102 2.97 mm to (174.2, 109.8)
- moved TP805 2.66 mm to (139.4, 101.6)
- moved TP501 1.90 mm to (119.4, 108.5)
- moved TP506 1.86 mm to (114.2, 104.9)
- moved TP505 1.73 mm to (119.3, 104.9)
- moved S201 1.52 mm to (117.0, 128.0)
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Routing:
- net /Page 1/SDA: track 32.7 -> 79.3 mm, vias 1 -> 4
- net /Page 1/SCL: track 29.1 -> 75.1 mm, vias 1 -> 4
- net /Page 1/SW5: track 11.6 -> 52.5 mm, vias 1 -> 3
- net /Page 1/SW4: track 11.4 -> 52.1 mm, vias 1 -> 3
- net /Page 1/IMU_INT: track 0.00 -> 35.9 mm, vias 0 -> 2
- net /Page 1/SW3: track 11.6 -> 45.2 mm, vias 1 -> 3
- net /Page 1/MEGA_nRST: track 31.6 -> 55.9 mm
- net /Page 1/BUZZER: track 0.00 -> 14.4 mm
- net /Page 1/SAMD11_TX_MEGA_RX: track 27.1 -> 37.4 mm, vias 1 -> 3
- net GND: track 114.1 -> 123.4 mm
- net /Page 1/SAMD11_RX_MEGA_TX: track 29.3 -> 35.6 mm
- net /Page 1/LCD_DC: track 33.9 -> 38.4 mm
- net +3V3: track 27.1 -> 31.1 mm, vias 10 -> 11
- net /Page 1/SPI_MISO: track 40.9 -> 44.6 mm
- net Net-(C301-Pad2): track 0.00 -> 3.19 mm
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Other:
- board text added: "+"
- board text added: "+ UP"
- board text added: "AWAY FROM BOARD"
- board text added: "OFF"
- board text added: "ON"
