File: Name Plate Class Project.kicad_pcb (KiCad board)
At the start: 2 copper layers, 83.5 x 66 mm, 129 parts, among them J101 Conn Header SMD, J201 Battery Connector, J501 USB_B_Mini, J502 SAMD11 Header, J801 DNP, Q201 BSS138, U101 ATmega328P-AU, U201 MIC5219-5.0YM5-TR, U202 MIC5219-3.3YM5-TR, U501 ATSAMD11C14A-SS, U601 BNO055, U602 BME280, U701 MCP7940N-xSN, Y101 16.00 MHz, Y601 32.7680 kHz, Y701 32.7680 kHz

Commit message: Before removing empty module entries from pcb
Other:
- board text removed: "+"
Changed lines of the file:
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@@
   (general
     (thickness 1.6)
-    (drawings 14)
+    (drawings 13)
     (tracks 871)
     (zones 0)
@@
     (35 F.Paste user)
     (36 B.SilkS user)
-    (37 F.SilkS user)
+    (37 F.SilkS user hide)
     (38 B.Mask user)
     (39 F.Mask user)
@@
     (46 B.CrtYd user)
     (47 F.CrtYd user)
-    (48 B.Fab user hide)
-    (49 F.Fab user hide)
+    (48 B.Fab user)
+    (49 F.Fab user)
   )
   (setup
@@
     (add_net VBUS)
   )
+  (module Name_Plate_Class_Project:BAT_BK-883 (layer B.Cu)
+    (at 164.81 122.62)
+    (fp_text reference B701 (at 0.05 -4.4) (layer B.SilkS)
+      (effects (font (size 1 1) (thickness 0.15)) (justify mirror))
+    )
+    (fp_text value BK-883 (at 0 -6.7) (layer B.Fab)
+      (effects (font (size 1 1) (thickness 0.15)) (justify mirror))
+    )
+    (fp_text user + (at 12.2 4.2) (layer B.SilkS)
+      (effects (font (size 1.25 1.25) (thickness 0.2)) (justify mirror))
+    )
+    (fp_text user - (at 0 4) (layer B.SilkS)
+      (effects (font (size 1.25 1.25) (thickness 0.2)) (justify mirror))
+    )
+    (fp_text user + (at -12.2 4.2) (layer B.SilkS)
+      (effects (font (size 1.25 1.25) (thickness 0.2)) (justify mirror))
+    )
+    (fp_line (start -10.805 9.49) (end -10.805 3.285) (layer B.CrtYd) (width 0.05))
+    (fp_line (start 10.805 9.49) (end -10.805 9.49) (layer B.CrtYd) (width 0.05))
+    (fp_line (start 10.805 3.285) (end 10.805 9.49) (layer B.CrtYd) (width 0.05))
+    (fp_line (start 15.615 3.285) (end 10.805 3.285) (layer B.CrtYd) (width 0.05))
+    (fp_line (start 15.615 -3.285) (end 15.615 3.285) (layer B.CrtYd) (width 0.05))
+    (fp_line (start 10.805 -3.285) (end 15.615 -3.285) (layer B.CrtYd) (width 0.05))
+    (fp_line (start 10.805 -10.82) (end 10.805 -3.285) (layer B.CrtYd) (width 0.05))
+    (fp_line (start -10.805 -10.82) (end 10.805 -10.82) (layer B.CrtYd) (width 0.05))
+    (fp_line (start -10.805 -3.285) (end -10.805 -10.82) (layer B.CrtYd) (width 0.05))
+    (fp_line (start -15.615 -3.285) (end -10.805 -3.285) (layer B.CrtYd) (width 0.05))
+    (fp_line (start -15.615 3.285) (end -15.615 -3.285) (layer B.CrtYd) (width 0.05))
+    (fp_line (start -10.805 3.285) (end -15.615 3.285) (layer B.CrtYd) (width 0.05))
+    (fp_line (start -10.555 7.5) (end -10.555 3.81) (layer B.SilkS) (width 0.12))
+    (fp_arc (start -8.222162 6.809786) (end -10.555 7.5) (angle -139.5) (layer B.SilkS) (width 0.12))
+    (fp_arc (start 0 12.001245) (end -6 7.8) (angle 110) (layer B.SilkS) (width 0.12))
+    (fp_arc (start 8.222162 6.809786) (end 6 7.8) (angle -139.5) (layer B.SilkS) (width 0.12))
+    (fp_line (start 10.555 3.81) (end 10.555 7.5) (layer B.SilkS) (width 0.12))
+    (fp_line (start 10.555 -4.58) (end 10.555 -3.81) (layer B.SilkS) (width 0.12))
+    (fp_line (start 4.5 -10.57) (end 10.555 -4.58) (layer B.SilkS) (width 0.12))
+    (fp_line (start -4.5 -10.57) (end 4.5 -10.57) (layer B.SilkS) (width 0.12))
+    (fp_line (start -10.555 -4.58) (end -4.5 -10.57) (layer B.SilkS) (width 0.12))
+    (fp_line (start -10.555 -3.81) (end -10.555 -4.58) (layer B.SilkS) (width 0.12))
+    (fp_line (start -10.555 2.54) (end -15.365 2.54) (layer B.Fab) (width 0.1))
+    (fp_line (start -10.555 7.5) (end -10.555 2.54) (layer B.Fab) (width 0.1))
+    (fp_arc (start -8.222162 6.809786) (end -10.555 7.5) (angle -139.5) (layer B.Fab) (width 0.1))
+    (fp_arc (start 0 12.001245) (end -6 7.8) (angle 110) (layer B.Fab) (width 0.1))
+    (fp_arc (start 8.222162 6.809786) (end 6 7.8) (angle -139.5) (layer B.Fab) (width 0.1))
+    (fp_line (start 10.555 2.54) (end 10.555 7.5) (layer B.Fab) (width 0.1))
+    (fp_line (start 15.365 2.54) (end 10.555 2.54) (layer B.Fab) (width 0.1))
+    (fp_line (start 15.365 -2.54) (end 15.365 2.54) (layer B.Fab) (width 0.1))
+    (fp_line (start 10.555 -2.54) (end 15.365 -2.54) (layer B.Fab) (width 0.1))
+    (fp_line (start 10.555 -4.58) (end 10.555 -2.54) (layer B.Fab) (width 0.1))
+    (fp_line (start 4.5 -10.57) (end 10.555 -4.58) (layer B.Fab) (width 0.1))
+    (fp_line (start -4.5 -10.57) (end 4.5 -10.57) (layer B.Fab) (width 0.1))
+    (fp_line (start -10.555 -4.58) (end -4.5 -10.57) (layer B.Fab) (width 0.1))
+    (fp_line (start -10.555 -2.54) (end -10.555 -4.58) (layer B.Fab) (width 0.1))
+    (fp_line (start -15.365 -2.54) (end -10.555 -2.54) (layer B.Fab) (width 0.1))
+    (fp_line (start -15.365 2.54) (end -15.365 -2.54) (layer B.Fab) (width 0.1))
+    (pad 1 smd rect (at -12.33 0) (size 6.07 6.07) (layers B.Cu B.Paste B.Mask))
+    (pad 3 smd rect (at 12.33 0) (size 6.07 6.07) (layers B.Cu B.Paste B.Mask)
+      (net 64 "/Page 7/RTCB+"))
+    (pad 2 smd rect (at 0 0) (size 6.07 6.07) (layers B.Cu B.Mask)
+      (net 1 GND))
+    (model "$(LE3DMOD)/BK-883.step"
+      (offset (xyz 0 -0.65 0))
+      (scale (xyz 1 1 1))
+      (rotate (xyz -90 0 180))
+    )
+  )
   (module Name_Plate_Class_Project:Molex_USB_Mini_B_548190572 (layer B.Cu)
     (at 114.708 95.696)
@@
       (effects (font (size 1.27 1.27) (thickness 0.15)))
     )
-    (fp_text user + (at 159.99 111.47 180) (layer B.SilkS)
-      (effects (font (size 1.25 1.25) (thickness 0.2)) (justify mirror))
-    )
   )
   (module "" (layer F.Cu)
@@
       (effects (font (size 1.27 1.27) (thickness 0.15)))
     )
-    (fp_text user - (at 109.8 104.36 180) (layer B.SilkS)
-      (effects (font (size 1.25 1.25) (thickness 0.2)) (justify mirror))
-    )
   )
   (module "" (layer F.Cu)
@@
     )
   )
-  (module Name_Plate_Class_Project:BAT_BK-883 (layer B.Cu)
-    (at 164.81 122.62)
-    (fp_text reference B701 (at 0.05 -4.4) (layer B.SilkS)
-      (effects (font (size 1 1) (thickness 0.15)) (justify mirror))
-    )
-    (fp_text value BK-883 (at 0 -6.7) (layer B.Fab)
-      (effects (font (size 1 1) (thickness 0.15)) (justify mirror))
-    )
-    (fp_line (start -10.805 9.49) (end -10.805 3.285) (layer B.CrtYd) (width 0.05))
-    (fp_line (start 10.805 9.49) (end -10.805 9.49) (layer B.CrtYd) (width 0.05))
-    (fp_line (start 10.805 3.285) (end 10.805 9.49) (layer B.CrtYd) (width 0.05))
-    (fp_line (start 15.615 3.285) (end 10.805 3.285) (layer B.CrtYd) (width 0.05))
-    (fp_line (start 15.615 -3.285) (end 15.615 3.285) (layer B.CrtYd) (width 0.05))
-    (fp_line (start 10.805 -3.285) (end 15.615 -3.285) (layer B.CrtYd) (width 0.05))
-    (fp_line (start 10.805 -10.82) (end 10.805 -3.285) (layer B.CrtYd) (width 0.05))
-    (fp_line (start -10.805 -10.82) (end 10.805 -10.82) (layer B.CrtYd) (width 0.05))
-    (fp_line (start -10.805 -3.285) (end -10.805 -10.82) (layer B.CrtYd) (width 0.05))
-    (fp_line (start -15.615 -3.285) (end -10.805 -3.285) (layer B.CrtYd) (width 0.05))
-    (fp_line (start -15.615 3.285) (end -15.615 -3.285) (layer B.CrtYd) (width 0.05))
-    (fp_line (start -10.805 3.285) (end -15.615 3.285) (layer B.CrtYd) (width 0.05))
-    (fp_line (start -10.555 7.5) (end -10.555 3.81) (layer B.SilkS) (width 0.12))
-    (fp_arc (start -8.222162 6.809786) (end -10.555 7.5) (angle -139.5) (layer B.SilkS) (width 0.12))
-    (fp_arc (start 0 12.001245) (end -6 7.8) (angle 110) (layer B.SilkS) (width 0.12))
-    (fp_arc (start 8.222162 6.809786) (end 6 7.8) (angle -139.5) (layer B.SilkS) (width 0.12))
-    (fp_line (start 10.555 3.81) (end 10.555 7.5) (layer B.SilkS) (width 0.12))
-    (fp_line (start 10.555 -4.58) (end 10.555 -3.81) (layer B.SilkS) (width 0.12))
-    (fp_line (start 4.5 -10.57) (end 10.555 -4.58) (layer B.SilkS) (width 0.12))
-    (fp_line (start -4.5 -10.57) (end 4.5 -10.57) (layer B.SilkS) (width 0.12))
-    (fp_line (start -10.555 -4.58) (end -4.5 -10.57) (layer B.SilkS) (width 0.12))
-    (fp_line (start -10.555 -3.81) (end -10.555 -4.58) (layer B.SilkS) (width 0.12))
-    (fp_line (start -10.555 2.54) (end -15.365 2.54) (layer B.Fab) (width 0.1))
-    (fp_line (start -10.555 7.5) (end -10.555 2.54) (layer B.Fab) (width 0.1))
-    (fp_arc (start -8.222162 6.809786) (end -10.555 7.5) (angle -139.5) (layer B.Fab) (width 0.1))
-    (fp_arc (start 0 12.001245) (end -6 7.8) (angle 110) (layer B.Fab) (width 0.1))
-    (fp_arc (start 8.222162 6.809786) (end 6 7.8) (angle -139.5) (layer B.Fab) (width 0.1))
-    (fp_line (start 10.555 2.54) (end 10.555 7.5) (layer B.Fab) (width 0.1))
-    (fp_line (start 15.365 2.54) (end 10.555 2.54) (layer B.Fab) (width 0.1))
-    (fp_line (start 15.365 -2.54) (end 15.365 2.54) (layer B.Fab) (width 0.1))
-    (fp_line (start 10.555 -2.54) (end 15.365 -2.54) (layer B.Fab) (width 0.1))
-    (fp_line (start 10.555 -4.58) (end 10.555 -2.54) (layer B.Fab) (width 0.1))
-    (fp_line (start 4.5 -10.57) (end 10.555 -4.58) (layer B.Fab) (width 0.1))
-    (fp_line (start -4.5 -10.57) (end 4.5 -10.57) (layer B.Fab) (width 0.1))
-    (fp_line (start -10.555 -4.58) (end -4.5 -10.57) (layer B.Fab) (width 0.1))
-    (fp_line (start -10.555 -2.54) (end -10.555 -4.58) (layer B.Fab) (width 0.1))
-    (fp_line (start -15.365 -2.54) (end -10.555 -2.54) (layer B.Fab) (width 0.1))
-    (fp_line (start -15.365 2.54) (end -15.365 -2.54) (layer B.Fab) (width 0.1))
-    (pad 1 smd rect (at -12.33 0) (size 6.07 6.07) (layers B.Cu B.Paste B.Mask))
-    (pad 3 smd rect (at 12.33 0) (size 6.07 6.07) (layers B.Cu B.Paste B.Mask)
-      (net 64 "/Page 7/RTCB+"))
-    (pad 2 smd rect (at 0 0) (size 6.07 6.07) (layers B.Cu B.Mask)
-      (net 1 GND) (thermal_width 1))
-    (model "$(LE3DMOD)/BK-883.step"
-      (offset (xyz 0 -0.65 0))
-      (scale (xyz 1 1 1))
-      (rotate (xyz -90 0 180))
-    )
-  )
   (module Name_Plate_Class_Project:LED_G-GX (layer F.Cu)
     (at 117.602 129.286 180)
@@
     (effects (font (size 1 1) (thickness 0.15)) (justify mirror))
   )
-  (gr_text + (at 152.32 126.71) (layer B.SilkS)
-    (effects (font (size 1.25 1.25) (thickness 0.2)) (justify mirror))
-  )
   (gr_text "+ UP" (at 164.63 130.29) (layer B.SilkS)

Commit message: Update
Parts:
- removed ? (x5): , 
Changed lines of the file:
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@@
     (tracks 871)
     (zones 0)
-    (modules 129)
+    (modules 124)
     (nets 66)
   )
@@
     (35 F.Paste user)
     (36 B.SilkS user)
-    (37 F.SilkS user hide)
+    (37 F.SilkS user)
     (38 B.Mask user)
     (39 F.Mask user)
@@
     (46 B.CrtYd user)
     (47 F.CrtYd user)
-    (48 B.Fab user)
-    (49 F.Fab user)
+    (48 B.Fab user hide)
+    (49 F.Fab user hide)
   )
   (setup
@@
     (visible_elements 7FFFFFFF)
     (pcbplotparams
-      (layerselection 0x010fc_ffffffff)
+      (layerselection 0x310fc_ffffffff)
       (usegerberextensions false)
       (usegerberattributes false)
@@
       (psa4output false)
       (plotreference true)
-      (plotvalue true)
+      (plotvalue false)
       (plotinvisibletext false)
       (padsonsilk false)
@@
       (outputformat 1)
       (mirror false)
-      (drillshape 1)
+      (drillshape 0)
       (scaleselection 1)
-      (outputdirectory ""))
+      (outputdirectory "Gerbers/2020-06-23/"))
   )
   (net 0 "")
@@
   (module Name_Plate_Class_Project:BAT_BK-883 (layer B.Cu)
     (at 164.81 122.62)
-    (fp_text reference B701 (at 0.05 -4.4) (layer B.SilkS)
+    (fp_text reference B701 (at -9.92 -7.78 90) (layer B.SilkS)
       (effects (font (size 1 1) (thickness 0.15)) (justify mirror))
     )
@@
     (descr "TFT LCD Screen")
     (attr smd)
-    (fp_text reference J801 (at 5.01 0.91 180) (layer F.SilkS)
+    (fp_text reference J801 (at -0.63 -28.18 270) (layer F.SilkS)
       (effects (font (size 1 1) (thickness 0.15)))
     )
@@
       (effects (font (size 1 1) (thickness 0.15)))
     )
-    (fp_text user 40 (at 5.9944 -54.864) (layer F.SilkS)
+    (fp_text user 40 (at 8.41 -53.42) (layer F.SilkS)
       (effects (font (size 1 1) (thickness 0.15)))
     )
-    (fp_text user 39 (at 3.5052 -54.864) (layer F.SilkS)
+    (fp_text user 39 (at 1.05 -53.48) (layer F.SilkS)
       (effects (font (size 1 1) (thickness 0.15)))
     )
-    (fp_text user 2 (at 5.9944 -1.016) (layer F.SilkS)
+    (fp_text user 2 (at 8.77 -2.49) (layer F.SilkS)
       (effects (font (size 1 1) (thickness 0.15)))
     )
-    (fp_text user 1 (at 3.5052 -1.016) (layer F.SilkS)
+    (fp_text user 1 (at 0.55 -2.42) (layer F.SilkS)
       (effects (font (size 1 1) (thickness 0.15)))
     )
@@
     )
   )
-  (module "" (layer F.Cu)
-    (at 17.17 15.16)
-    (fp_text reference "" (at 168.13 127.17) (layer F.SilkS)
-      (effects (font (size 1.27 1.27) (thickness 0.15)))
-    )
-    (fp_text value "" (at 168.13 127.17) (layer F.SilkS)
-      (effects (font (size 1.27 1.27) (thickness 0.15)))
-    )
-  )
-  (module "" (layer F.Cu)
-    (at 168.13 127.17)
-    (fp_text reference "" (at 123.444 136.906) (layer F.SilkS)
-      (effects (font (size 1.27 1.27) (thickness 0.15)))
-    )
-    (fp_text value "" (at 123.444 136.906) (layer F.SilkS)
-      (effects (font (size 1.27 1.27) (thickness 0.15)))
-    )
-  )
-  (module "" (layer F.Cu)
-    (at 54.97 22.13)
-    (fp_text reference "" (at 123.444 136.906) (layer F.SilkS)
-      (effects (font (size 1.27 1.27) (thickness 0.15)))
-    )
-    (fp_text value "" (at 123.444 136.906) (layer F.SilkS)
-      (effects (font (size 1.27 1.27) (thickness 0.15)))
-    )
-  )
-  (module "" (layer F.Cu)
-    (at 123.444 136.906)
-    (fp_text reference "" (at 111.47 124.7) (layer F.SilkS)
-      (effects (font (size 1.27 1.27) (thickness 0.15)))
-    )
-    (fp_text value "" (at 111.47 124.7) (layer F.SilkS)
-      (effects (font (size 1.27 1.27) (thickness 0.15)))
-    )
-  )
-  (module "" (layer F.Cu)
-    (at 123.698 129.286)
-    (fp_text reference "" (at 111.47 124.7) (layer F.SilkS)
-      (effects (font (size 1.27 1.27) (thickness 0.15)))
-    )
-    (fp_text value "" (at 111.47 124.7) (layer F.SilkS)
-      (effects (font (size 1.27 1.27) (thickness 0.15)))
-    )
-  )
   (module Resistor_SMD:R_0603_1608Metric_Pad1.05x0.95mm_HandSolder (layer F.Cu)
     (at 174.19 109.81 180)
@@
     (tags "resistor handsolder")
     (attr smd)
-    (fp_text reference R104 (at 0 1.43 90) (layer B.SilkS)
+    (fp_text reference R104 (at -0.035 -1.34 90) (layer B.SilkS)
       (effects (font (size 1 1) (thickness 0.15)) (justify mirror))
     )
@@
   (module Name_Plate_Class_Project:Switch_JS202011SCQN (layer B.Cu)
     (at 117.024 128)
-    (fp_text reference S201 (at 0 0) (layer B.SilkS)
+    (fp_text reference S201 (at -3.994 -3.54 90) (layer B.SilkS)
       (effects (font (size 1 1) (thickness 0.15)) (justify mirror))
     )
@@
     (at 128.62 103.59 270)
     (descr "translated Allegro footprint")
-    (fp_text reference J502 (at -0.03 -4.65 90) (layer B.SilkS)
+    (fp_text reference J502 (at -1.91 4.6 90) (layer B.SilkS)
       (effects (font (size 1 1) (thickness 0.15)) (justify mirror))
     )
@@
     (tags "connector JST PH top entry")
     (attr smd)
-    (fp_text reference J201 (at 1.74 -3.74 -180) (layer B.SilkS)
+    (fp_text reference J201 (at -3.26 7.16 90) (layer B.SilkS)
       (effects (font (size 1 1) (thickness 0.15)) (justify mirror))
     )
@@
   (module Name_Plate_Class_Project:Oscillator_MC-405_32.7680K-D__ROHS (layer B.Cu)
     (at 146.37 71.14 180)
-    (fp_text reference Y601 (at -0.03 -1.36) (layer B.SilkS)
+    (fp_text reference Y601 (at 7.02 0.07 90) (layer B.SilkS)
       (effects (font (size 1 1) (thickness 0.15)) (justify mirror))
     )
@@
   (module Name_Plate_Class_Project:T491A106K010AT (layer F.Cu)
     (at 134.11 122.524 90)
-    (fp_text reference C302 (at 0.005004 -1.8 270) (layer F.SilkS)
+    (fp_text reference C302 (at 0.014 -2.13 270) (layer F.SilkS)
       (effects (font (size 1 1) (thickness 0.15)))
     )
@@
     (tags "Surface mounted pin header SMD 2x03 2.54mm double row")
     (attr smd)
-    (fp_text reference J101 (at 5.03 -0.03) (layer B.SilkS)
+    (fp_text reference J101 (at -0.01 -5.16 90) (layer B.SilkS)
       (effects (font (size 1 1) (thickness 0.15)) (justify mirror))
     )
@@
     (tags "SOIC SO")
     (attr smd)
-    (fp_text reference U501 (at -0.5 0.04 270) (layer B.SilkS)
+    (fp_text reference U501 (at 4.42 -2.91 270) (layer B.SilkS)
       (effects (font (size 1 1) (thickness 0.15)) (justify mirror))
     )
@@
     (tags "SOIC SO")
     (attr smd)
-    (fp_text reference U701 (at -0.01 -0.01 270) (layer B.SilkS)
+    (fp_text reference U701 (at 4.35 0 270) (layer B.SilkS)
       (effects (font (size 1 1) (thickness 0.15)) (justify mirror))
     )
@@
     (tags "resistor handsolder")
     (attr smd)
-    (fp_text reference R202 (at 4.34 -0.2 270) (layer B.SilkS)
+    (fp_text reference R202 (at -0.06 1.33 270) (layer B.SilkS)
       (effects (font (size 1 1) (thickness 0.15)) (justify mirror))
     )
@@
     (tags "capacitor handsolder")
     (attr smd)
-    (fp_text reference C306 (at 0 -1.43 90) (layer F.SilkS)
+    (fp_text reference C306 (at 0.349 -1.41 90) (layer F.SilkS)
       (effects (font (size 1 1) (thickness 0.15)))
     )
@@
     (tags "capacitor handsolder")
     (attr smd)
-    (fp_text reference C303 (at 0.425 -1.53 270) (layer F.SilkS)
+    (fp_text reference C303 (at -0.021 -1.31 270) (layer F.SilkS)
       (effects (font (size 1 1) (thickness 0.15)))
     )
@@
     (tags "resistor handsolder")
     (attr smd)
-    (fp_text reference R302 (at -0.023 1.406) (layer F.SilkS)
+    (fp_text reference R302 (at 2.37 -0.61 90) (layer F.SilkS)
       (effects (font (size 1 1) (thickness 0.15)))
     )
@@
     (tags SOT-23)
     (attr smd)
-    (fp_text reference Q201 (at 0 2.5) (layer B.SilkS)
+    (fp_text reference Q201 (at 2.38 0.03 90) (layer B.SilkS)
       (effects (font (size 1 1) (thickness 0.15)) (justify mirror))
     )
