File: Name Plate Class Project.kicad_pcb (KiCad board)
At the start: 2 copper layers, 83.5 x 66 mm, 124 parts, among them J101 Conn Header SMD, J201 Battery Connector, J501 USB_B_Mini, J502 SAMD11 Header, J801 DNP, Q201 BSS138, U101 ATmega328P-AU, U201 MIC5219-5.0YM5-TR, U202 MIC5219-3.3YM5-TR, U501 ATSAMD11C14A-SS, U601 BNO055, U602 BME280, U701 MCP7940N-xSN, Y101 16.00 MHz, Y601 32.7680 kHz, Y701 32.7680 kHz

Commit message: Final Design Files
Final design files as submitted.
Parts:
- added NT1: Net-Tie_2, NetTie:NetTie-2_SMD_Pad0.5mm, F.Cu at (136.2, 102.3)
Connections:
- C101 pad 1: +3V3 -> /Page 1/MEGAVCC
- C102 pad 1: +3V3 -> /Page 1/MEGAVCC
- C105 pad 1: +3V3 -> /Page 1/MEGAVCC
- C106 pad 1: +3V3 -> /Page 1/MEGAVCC
- U101 pad 18: +3V3 -> /Page 1/MEGAVCC
- U101 pad 4: +3V3 -> /Page 1/MEGAVCC
- U101 pad 6: +3V3 -> /Page 1/MEGAVCC
Routing:
- net /Page 1/MEGAVCC: track 0.00 -> 28.6 mm
- net +3V3: track 31.1 -> 34.2 mm
- net /Page 1/IMU_INT: track 35.9 -> 36.6 mm
