File: Page 1.sch (KiCad schematic (older format))
At the start: 14 parts, among them J101 Conn Header SMD, U1 ATmega328P-AU, Y101 16.00 MHz

Commit message: Updates
Parts:
- R101: value R10K0 -> 10K0; Manufacturer (none) -> Yageo
- R102, R103: value R4k75 -> 4k75; Manufacturer (none) -> Yageo
- R104, R105: value R10K0 -> 10K0; DigiKey Part No. (none) -> 311-10KGRCT-ND; Manufacturer (none) -> Yageo
Changed lines of the file:
@@
 AR Path="/5EACA483/5EAD5874" Ref="R?"  Part="1"
 F 0 "R103" H 5970 1396 50  0000 L CNN
-F 1 "R4k75" H 5970 1305 50  0000 L CNN
+F 1 "4k75" H 5970 1305 50  0000 L CNN
 F 2 "Resistor_SMD:R_0603_1608Metric_Pad1.05x0.95mm_HandSolder" V 5830 1350 50  0001 C CNN
 F 3 "~" H 5900 1350 50  0001 C CNN
+F 4 "Yageo" H 5900 1350 50  0001 C CNN "Manufacturer"
 	1    5900 1350
 	1    0    0    -1
@@
 AR Path="/5EACA483/5EAD4B3A" Ref="R?"  Part="1"
 F 0 "R102" H 5520 1396 50  0000 L CNN
-F 1 "R4k75" H 5520 1305 50  0000 L CNN
+F 1 "4k75" H 5520 1305 50  0000 L CNN
 F 2 "Resistor_SMD:R_0603_1608Metric_Pad1.05x0.95mm_HandSolder" V 5380 1350 50  0001 C CNN
 F 3 "~" H 5450 1350 50  0001 C CNN
+F 4 "Yageo" H 5450 1350 50  0001 C CNN "Manufacturer"
 	1    5450 1350
 	1    0    0    -1
@@
 AR Path="/5EACA483/5EAC9991" Ref="R?"  Part="1"
 F 0 "R101" H 5070 1396 50  0000 L CNN
-F 1 "R10K0" H 5070 1305 50  0000 L CNN
+F 1 "10K0" H 5070 1305 50  0000 L CNN
 F 2 "Resistor_SMD:R_0603_1608Metric_Pad1.05x0.95mm_HandSolder" V 4930 1350 50  0001 C CNN
 F 3 "https://www.yageo.com/upload/media/product/productsearch/datasheet/rchip/PYu-RC_Group_51_RoHS_L_10.pdf" H 5000 1350 50  0001 C CNN
 F 4 "311-10KGRCT-ND" H 5000 1350 50  0001 C CNN "DigiKey Part No."
 F 5 "Yageo RC0603JR-0710KL" H 5000 1350 50  0001 C CNN "Mftr Part No."
+F 6 "Yageo" H 5000 1350 50  0001 C CNN "Manufacturer"
 	1    5000 1350
 	1    0    0    -1
@@
 AR Path="/5EACA483/5EC9D2F5" Ref="R?"  Part="1"
 F 0 "R104" H 6420 1396 50  0000 L CNN
-F 1 "R10K0" H 6420 1305 50  0000 L CNN
+F 1 "10K0" H 6420 1305 50  0000 L CNN
 F 2 "Resistor_SMD:R_0603_1608Metric_Pad1.05x0.95mm_HandSolder" V 6280 1350 50  0001 C CNN
 F 3 "~" H 6350 1350 50  0001 C CNN
+F 4 "311-10KGRCT-ND" H 6350 1350 50  0001 C CNN "DigiKey Part No."
+F 5 "Yageo" H 6350 1350 50  0001 C CNN "Manufacturer"
 	1    6350 1350
 	1    0    0    -1
@@
 AR Path="/5EACA483/5EC9D6B1" Ref="R?"  Part="1"
 F 0 "R105" H 6820 1396 50  0000 L CNN
-F 1 "R10K0" H 6820 1305 50  0000 L CNN
+F 1 "10K0" H 6820 1305 50  0000 L CNN
 F 2 "Resistor_SMD:R_0603_1608Metric_Pad1.05x0.95mm_HandSolder" V 6680 1350 50  0001 C CNN
 F 3 "~" H 6750 1350 50  0001 C CNN
+F 4 "311-10KGRCT-ND" H 6750 1350 50  0001 C CNN "DigiKey Part No."
+F 5 "Yageo" H 6750 1350 50  0001 C CNN "Manufacturer"
 	1    6750 1350
 	1    0    0    -1

Commit message: Updates to schematic
Switching to ATMega34UF chip.
Parts:
- C101, C105, C106: DigiKey Part No. (none) -> 311-1335-1-ND; Manufacturer (none) -> Yageo; Mftr Part No. Yageo CC0603KPX7R7BB104 -> CC0603KPX7R7BB104
- C102: DigiKey Part No. (none) -> 478-5161-1-ND; Manufacturer (none) -> AVX; Mftr Part No. AVX 08053C124KAT2A -> 08053C124KAT2A
- C103, C104: DigiKey Part No. (none) -> 399-1052-1-ND; Manufacturer (none) -> Kemet; Mftr Part No. Kemet C0603C180J5GACTU -> C0603C180J5GACTU
- J101: DigiKey Part No. (none) -> 0713085406-ND; Manufacturer (none) -> Molex; Mftr Part No. (none) -> 713085406
- R101: value 10K0 -> 10k; Mftr Part No. Yageo RC0603JR-0710KL -> RC0603JR-0710KL
- R102, R103: value 4k75 -> 4.75k; DigiKey Part No. (none) -> 311-10KGRCT-ND; Mftr Part No. (none) -> RC0603JR-074K7L
- R104, R105: value 10K0 -> 10k; Mftr Part No. (none) -> RC0603JR-0710KL
- U101: renamed from U1; DigiKey Part No. (none) -> ATMEGA328P-AURCT-ND; Manufacturer (none) -> Microchip; Mftr Part No. (none) -> ATMega328P-AU
- Y101: DigiKey Part No. (none) -> 535-9103-1-ND; Manufacturer (none) -> Abracon; Mftr Part No. (none) -> ABM3-16.000MHZ-B2-T
Connections:
- wire segments 93 -> 91
Other:
- moved on the sheet: J101

Commit message: Updates
Parts:
- J101: footprint Name Plate Class Project:Molex_PinHeader_2x03 -> Name_Plate_Class_Project:Molex_PinHeader_2x03
- Y101: footprint Name Plate Class Project:Oscillator_ABM3-16.000MHZ-B2-T -> Name_Plate_Class_Project:Oscillator_ABM3-16.000MHZ-B2-T; symbol Name~Plate~Class~Library:Oscillator_ABM3-16.000MHZ-B2-T -> Name_Plate_Class_Project:Oscillator_ABM3-16.000MHZ-B2-T
Changed lines of the file:
@@
 $EndComp
 $Comp
-L Name~Plate~Class~Library:Oscillator_ABM3-16.000MHZ-B2-T Y101
+L Name_Plate_Class_Project:Oscillator_ABM3-16.000MHZ-B2-T Y101
 U 1 1 5EC8A05A
 P 8550 1500
 F 0 "Y101" V 8504 1600 50  0000 L CNN
 F 1 "16.00 MHz" V 8595 1600 50  0000 L CNN
-F 2 "Name Plate Class Project:Oscillator_ABM3-16.000MHZ-B2-T" H 8500 1750 50  0001 L BNN
+F 2 "Name_Plate_Class_Project:Oscillator_ABM3-16.000MHZ-B2-T" H 8500 1750 50  0001 L BNN
 F 3 "https://abracon.com/Resonators/abm3.pdf" H 8450 1250 50  0001 L BNN
 F 4 "535-9103-1-ND" H 8550 1500 50  0001 C CNN "DigiKey Part No."
@@
 F 0 "J101" H 9250 3650 50  0000 R CNN
 F 1 "Conn Header SMD" H 9150 3150 50  0000 C CNN
-F 2 "Name Plate Class Project:Molex_PinHeader_2x03" H 9100 3400 50  0001 C CNN
+F 2 "Name_Plate_Class_Project:Molex_PinHeader_2x03" H 9100 3400 50  0001 C CNN
 F 3 "https://www.molex.com/pdm_docs/sd/713085404_sd.pdf" H 9100 3400 50  0001 C CNN
 F 4 "0713085406-ND" H 9100 3400 50  0001 C CNN "DigiKey Part No."

Commit message: Final Design Files
Final design files as submitted.
Parts:
- added NT1: Net-Tie_2, NetTie:NetTie-2_SMD_Pad0.5mm, symbol Device:Net-Tie_2
Connections:
- net +3V3: now also NT1.1; no longer C101.1, C102.1, C105.1, C106.1, U101.18 (AVCC), U101.4 (VCC), U101.6 (VCC)
- new net MEGAVCC: C101.1, C102.1, C105.1, C106.1, NT1.2, U101.18 (AVCC), U101.4 (VCC), U101.6 (VCC)
Changed lines of the file:
@@
 L power:+3.3V #PWR?
 U 1 1 5EAC9944
-P 2650 1000
+P 1000 1000
 AR Path="/5EAC9944" Ref="#PWR?"  Part="1"
 AR Path="/5EAC05C2/5EAC9944" Ref="#PWR04"  Part="1"
 AR Path="/5EACA483/5EAC9944" Ref="#PWR?"  Part="1"
-F 0 "#PWR04" H 2650 850 50  0001 C CNN
-F 1 "+3.3V" H 2665 1173 50  0000 C CNN
-F 2 "" H 2650 1000 50  0001 C CNN
-F 3 "" H 2650 1000 50  0001 C CNN
-	1    2650 1000
+F 0 "#PWR04" H 1000 850 50  0001 C CNN
+F 1 "+3.3V" H 1015 1173 50  0000 C CNN
+F 2 "" H 1000 1000 50  0001 C CNN
+F 3 "" H 1000 1000 50  0001 C CNN
+	1    1000 1000
 	1    0    0    -1
 $EndComp
@@
 Connection ~ 3000 1000
 Wire Wire Line
-	3000 1000 2650 1000
-Wire Wire Line
 	2300 1000 2300 1500
 Connection ~ 2300 1000
@@
 Wire Wire Line
 	1650 1000 1650 2800
-Connection ~ 2650 1000
-Wire Wire Line
-	2650 1000 2300 1000
 Wire Wire Line
 	3700 2400 5000 2400
@@
 Wire Wire Line
 	9850 3300 9850 3200
+Wire Wire Line
+	2300 1000 3000 1000
+$Comp
+L Device:Net-Tie_2 NT1
+U 1 1 5F05D7AF
+P 1200 1000
+F 0 "NT1" H 1200 1050 50  0000 C CNN
+F 1 "Net-Tie_2" H 1200 1090 50  0001 C CNN
+F 2 "NetTie:NetTie-2_SMD_Pad0.5mm" H 1200 1000 50  0001 C CNN
+F 3 "None" H 1200 1000 50  0001 C CNN
+F 4 "None" H 1200 1000 50  0001 C CNN "DigiKey Part No."
+F 5 "None" H 1200 1000 50  0001 C CNN "Manufacturer"
+F 6 "None" H 1200 1000 50  0001 C CNN "Mftr Part No."
+	1    1200 1000
+	1    0    0    -1
+$EndComp
+Wire Wire Line
+	1300 1000 1350 1000
+Connection ~ 1350 1000
+Wire Wire Line
+	1100 1000 1000 1000
+Text Label 1750 1000 0    50   ~ 0
+MEGAVCC
 $EndSCHEMATC
