File: Page 3.sch (KiCad schematic (older format))
At the start: 15 parts

Commit message: Updates to schematic
Switching to ATMega34UF chip.
Parts:
- C301, C302: DigiKey Part No. PCE4295CT-ND -> 399-11437-1-ND; Manufacturer (none) -> Kemet; Mftr Part No. Panasonic EEE-1VA2R2NR -> T491A106K010AT
- C303, C304, C305, C306: DigiKey Part No. (none) -> 311-1335-1-ND; Manufacturer (none) -> Yageo; Mftr Part No. Yageo CC0603KPX7R7BB104 -> CC0603KPX7R7BB104
- D305: DigiKey Part No. 754-1580-6-ND -> 475-2816-1-ND; Manufacturer (none) -> OSRAM Opto Semiconductors; Mftr Part No. Kingbright APA3010CGCK-GX -> LB Q39G-L2OO-35-1
- LS301: DigiKey Part No. (none) -> 668-1136-ND; Manufacturer (none) -> Pui Audio; Mftr Part No. (none) -> AST-03008MR-R
- R301: value 22K0 -> 22; DigiKey Part No. (none) -> A130081CT-ND; Mftr Part No. (none) -> CRGCQ0603J22R
- R302: value 470k -> 470; DigiKey Part No. (none) -> A130089CT-ND; Mftr Part No. (none) -> CRGCQ0603J470R
- TP301: symbol Connector:TestPoint -> Name~Plate~Class~Library:TestPoint; DigiKey Part No. (none) -> None; Manufacturer (none) -> None; Mftr Part No. (none) -> None
Changed lines of the file:
@@
 F 1 "BLUE LED" H 2550 4700 50  0000 R TNN
 F 2 "Name Plate Class Project:LED_G-GX" H 2500 4850 50  0001 C CNN
-F 3 "http://www.kingbrightusa.com/images/catalog/SPEC/APA3010CGCK-GX.pdf" H 2500 4850 50  0001 C CNN
-F 4 "754-1580-6-ND" H 2500 4850 50  0001 C CNN "DigiKey Part No."
-F 5 "Kingbright APA3010CGCK-GX" H 2500 4850 50  0001 C CNN "Mftr Part No."
+F 3 "https://media.digikey.com/pdf/Data%20Sheets/Osram%20PDFs/LB_Q39G_v1.4_9-1-15.pdf" H 2500 4850 50  0001 C CNN
+F 4 "475-2816-1-ND" H 2500 4850 50  0001 C CNN "DigiKey Part No."
+F 5 "LB Q39G-L2OO-35-1" H 2500 4850 50  0001 C CNN "Mftr Part No."
+F 6 "OSRAM Opto Semiconductors" H 2500 4850 50  0001 C CNN "Manufacturer"
 	1    2500 4850
 	-1   0    0    1
@@
 AR Path="/5ECEA271/5ECEB248" Ref="R302"  Part="1"
 F 0 "R302" V 2850 4750 50  0000 L BNN
-F 1 "470k" V 2950 4750 50  0000 L BNN
+F 1 "470" V 2950 4750 50  0000 L BNN
 F 2 "Resistor_SMD:R_0603_1608Metric_Pad1.05x0.95mm_HandSolder" V 2980 4850 50  0001 C CNN
-F 3 "~" H 3050 4850 50  0001 C CNN
+F 3 "https://www.te.com/commerce/DocumentDelivery/DDEController?Action=srchrtrv&DocNm=1773204-3&DocType=DS&DocLang=English" H 3050 4850 50  0001 C CNN
 F 4 "TE Connectivity " H 3050 4850 50  0001 C CNN "Manufacturer"
+F 5 "A130089CT-ND" H 3050 4850 50  0001 C CNN "DigiKey Part No."
+F 6 "CRGCQ0603J470R" H 3050 4850 50  0001 C CNN "Mftr Part No."
 	1    3050 4850
 	0    1    1    0
@@
 F 2 "Name Plate Class Project:Buzzer_TDK_PS1240P02BT_D12.2mm_H6.5mm" V 9325 5000 50  0001 C CNN
 F 3 "http://www.puiaudio.com/pdf/AST-03008MR-R.pdf" V 9325 5000 50  0001 C CNN
+F 4 "668-1136-ND" H 9350 4900 50  0001 C CNN "DigiKey Part No."
+F 5 "Pui Audio" H 9350 4900 50  0001 C CNN "Manufacturer"
+F 6 "AST-03008MR-R" H 9350 4900 50  0001 C CNN "Mftr Part No."
 	1    9350 4900
 	1    0    0    -1
@@
 F 3 "https://media.digikey.com/pdf/Data%20Sheets/Panasonic%20Electronic%20Components/S_Series,Type_V_Rev2018.pdf" H 8950 4800 50  0001 C CNN
 F 4 "Panasonic EEE-1VA2R2NR" H 8950 4800 50  0001 C CNN "Field4"
-F 5 "PCE4295CT-ND" H 8950 4800 50  0001 C CNN "DigiKey Part No."
-F 6 "Panasonic EEE-1VA2R2NR" H 8950 4800 50  0001 C CNN "Mftr Part No."
+F 5 "399-11437-1-ND" H 8950 4800 50  0001 C CNN "DigiKey Part No."
+F 6 "T491A106K010AT" H 8950 4800 50  0001 C CNN "Mftr Part No."
 F 7 "" H 8950 4800 50  0001 C CNN "URL"
+F 8 "Kemet" H 8950 4800 50  0001 C CNN "Manufacturer"
 	1    8950 4800
 	0    -1   -1   0
@@
 AR Path="/5ECEA271/5EB2ABF4" Ref="R301"  Part="1"
 F 0 "R301" V 3150 2350 50  0000 R CNN
-F 1 "22K0" V 3050 2350 50  0000 R CNN
+F 1 "22" V 3050 2350 50  0000 R CNN
 F 2 "Resistor_SMD:R_0603_1608Metric_Pad1.05x0.95mm_HandSolder" V 3180 2250 50  0001 C CNN
 F 3 "https://www.te.com/commerce/DocumentDelivery/DDEController?Action=srchrtrv&DocNm=1773204-3&DocType=DS&DocLang=English" H 3250 2250 50  0001 C CNN
 F 4 "TE Connectivity " H 3250 2250 50  0001 C CNN "Manufacturer"
+F 5 "CRGCQ0603J22R" H 3250 2250 50  0001 C CNN "Mftr Part No."
+F 6 "A130081CT-ND" H 3250 2250 50  0001 C CNN "DigiKey Part No."
 	1    3250 2250
 	0    -1   -1   0
 $EndComp
 $Comp
-L Connector:TestPoint TP?
+L Name~Plate~Class~Library:TestPoint TP?
 U 1 1 5EB2B88E
 P 2850 2250
@@
 AR Path="/5ECEA271/5EB2B88E" Ref="TP301"  Part="1"
 F 0 "TP301" H 2650 2550 50  0000 L CNN
-F 1 "Test Point" H 2650 2450 50  0000 L CNN
+F 1 "Test Point" H 2650 2450 50  0001 L CNN
 F 2 "Connector_Wire:SolderWirePad_1x01_SMD_5x10mm" H 3050 2250 50  0001 C CNN
 F 3 "None" H 3050 2250 50  0001 C CNN
-F 4 "TP_ADDR_LED" H 2850 2250 50  0001 C CNN "Name"
+F 4 "TP_ADDR_LED" H 2650 2450 50  0000 L CNN "Name"
+F 5 "None" H 2850 2250 50  0001 C CNN "DigiKey Part No."
+F 6 "None" H 2850 2250 50  0001 C CNN "Manufacturer"
+F 7 "None" H 2850 2250 50  0001 C CNN "Mftr Part No."
 	1    2850 2250
 	1    0    0    -1
@@
 F 2 "Capacitor_SMD:C_0603_1608Metric_Pad1.05x0.95mm_HandSolder" H 4388 2400 50  0001 C CNN
 F 3 "https://www.yageo.com/upload/media/product/productsearch/datasheet/mlcc/UPY-GPHC_X7R_6.3V-to-50V_18.pdf" H 4350 2550 50  0001 C CNN
-F 4 "Yageo CC0603KPX7R7BB104" H 4350 2550 50  0001 C CNN "Mftr Part No."
+F 4 "CC0603KPX7R7BB104" H 4350 2550 50  0001 C CNN "Mftr Part No."
+F 5 "Yageo" H 4350 2550 50  0001 C CNN "Manufacturer"
+F 6 "311-1335-1-ND" H 4350 2550 50  0001 C CNN "DigiKey Part No."
 	1    4350 2550
 	1    0    0    -1
@@
 F 2 "Capacitor_SMD:C_0603_1608Metric_Pad1.05x0.95mm_HandSolder" H 5538 2400 50  0001 C CNN
 F 3 "https://www.yageo.com/upload/media/product/productsearch/datasheet/mlcc/UPY-GPHC_X7R_6.3V-to-50V_18.pdf" H 5500 2550 50  0001 C CNN
-F 4 "Yageo CC0603KPX7R7BB104" H 5500 2550 50  0001 C CNN "Mftr Part No."
+F 4 "CC0603KPX7R7BB104" H 5500 2550 50  0001 C CNN "Mftr Part No."
+F 5 "Yageo" H 5500 2550 50  0001 C CNN "Manufacturer"
+F 6 "311-1335-1-ND" H 5500 2550 50  0001 C CNN "DigiKey Part No."
 	1    5500 2550
 	1    0    0    -1
@@
 F 2 "Capacitor_SMD:C_0603_1608Metric_Pad1.05x0.95mm_HandSolder" H 6688 2400 50  0001 C CNN
 F 3 "https://www.yageo.com/upload/media/product/productsearch/datasheet/mlcc/UPY-GPHC_X7R_6.3V-to-50V_18.pdf" H 6650 2550 50  0001 C CNN
-F 4 "Yageo CC0603KPX7R7BB104" H 6650 2550 50  0001 C CNN "Mftr Part No."
+F 4 "CC0603KPX7R7BB104" H 6650 2550 50  0001 C CNN "Mftr Part No."
+F 5 "Yageo" H 6650 2550 50  0001 C CNN "Manufacturer"
+F 6 "311-1335-1-ND" H 6650 2550 50  0001 C CNN "DigiKey Part No."
 	1    6650 2550
 	1    0    0    -1
@@
 F 2 "Capacitor_SMD:C_0603_1608Metric_Pad1.05x0.95mm_HandSolder" H 7838 2400 50  0001 C CNN
 F 3 "https://www.yageo.com/upload/media/product/productsearch/datasheet/mlcc/UPY-GPHC_X7R_6.3V-to-50V_18.pdf" H 7800 2550 50  0001 C CNN
-F 4 "Yageo CC0603KPX7R7BB104" H 7800 2550 50  0001 C CNN "Mftr Part No."
+F 4 "CC0603KPX7R7BB104" H 7800 2550 50  0001 C CNN "Mftr Part No."
+F 5 "Yageo" H 7800 2550 50  0001 C CNN "Manufacturer"
+F 6 "311-1335-1-ND" H 7800 2550 50  0001 C CNN "DigiKey Part No."
 	1    7800 2550
 	1    0    0    -1
@@
 F 3 "https://media.digikey.com/pdf/Data%20Sheets/Panasonic%20Electronic%20Components/S_Series,Type_V_Rev2018.pdf" H 8300 2200 50  0001 C CNN
 F 4 "Panasonic EEE-1VA2R2NR" H 8300 2200 50  0001 C CNN "Field4"
-F 5 "PCE4295CT-ND" H 8300 2200 50  0001 C CNN "DigiKey Part No."
-F 6 "Panasonic EEE-1VA2R2NR" H 8300 2200 50  0001 C CNN "Mftr Part No."
+F 5 "399-11437-1-ND" H 8300 2200 50  0001 C CNN "DigiKey Part No."
+F 6 "T491A106K010AT" H 8300 2200 50  0001 C CNN "Mftr Part No."
 F 7 "" H 8300 2200 50  0001 C CNN "URL"
+F 8 "Kemet" H 8300 2200 50  0001 C CNN "Manufacturer"
 	1    8300 2200
 	1    0    0    -1

Commit message: Updates
Parts:
- C301, C302: footprint Name Plate Class Project:CAP_430X430N -> Name_Plate_Class_Project:CAP_430X430N; Field4 Panasonic EEE-1VA2R2NR -> (none)
- D305: footprint Name Plate Class Project:LED_G-GX -> Name_Plate_Class_Project:LED_G-GX
- LS301: footprint Name Plate Class Project:Buzzer_TDK_PS1240P02BT_D12.2mm_H6.5mm -> Name_Plate_Class_Project:Buzzer_TDK_PS1240P02BT_D12.2mm_H6.5mm
- TP301: symbol Name~Plate~Class~Library:TestPoint -> Name_Plate_Class_Project:TestPoint
Changed lines of the file:
@@
 F 0 "D305" H 2550 4600 50  0000 R TNN
 F 1 "BLUE LED" H 2550 4700 50  0000 R TNN
-F 2 "Name Plate Class Project:LED_G-GX" H 2500 4850 50  0001 C CNN
+F 2 "Name_Plate_Class_Project:LED_G-GX" H 2500 4850 50  0001 C CNN
 F 3 "https://media.digikey.com/pdf/Data%20Sheets/Osram%20PDFs/LB_Q39G_v1.4_9-1-15.pdf" H 2500 4850 50  0001 C CNN
 F 4 "475-2816-1-ND" H 2500 4850 50  0001 C CNN "DigiKey Part No."
@@
 F 0 "LS301" H 9500 4950 50  0000 L CNN
 F 1 "Piezo Buzzer" H 9500 4850 50  0000 L CNN
-F 2 "Name Plate Class Project:Buzzer_TDK_PS1240P02BT_D12.2mm_H6.5mm" V 9325 5000 50  0001 C CNN
+F 2 "Name_Plate_Class_Project:Buzzer_TDK_PS1240P02BT_D12.2mm_H6.5mm" V 9325 5000 50  0001 C CNN
 F 3 "http://www.puiaudio.com/pdf/AST-03008MR-R.pdf" V 9325 5000 50  0001 C CNN
 F 4 "668-1136-ND" H 9350 4900 50  0001 C CNN "DigiKey Part No."
@@
 F 0 "C301" V 9202 4800 50  0000 C CNN
 F 1 "10uF" V 9111 4800 50  0000 C CNN
-F 2 "Name Plate Class Project:CAP_430X430N" H 8950 4800 50  0001 C CNN
+F 2 "Name_Plate_Class_Project:CAP_430X430N" H 8950 4800 50  0001 C CNN
 F 3 "https://media.digikey.com/pdf/Data%20Sheets/Panasonic%20Electronic%20Components/S_Series,Type_V_Rev2018.pdf" H 8950 4800 50  0001 C CNN
-F 4 "Panasonic EEE-1VA2R2NR" H 8950 4800 50  0001 C CNN "Field4"
-F 5 "399-11437-1-ND" H 8950 4800 50  0001 C CNN "DigiKey Part No."
-F 6 "T491A106K010AT" H 8950 4800 50  0001 C CNN "Mftr Part No."
-F 7 "" H 8950 4800 50  0001 C CNN "URL"
-F 8 "Kemet" H 8950 4800 50  0001 C CNN "Manufacturer"
+F 4 "399-11437-1-ND" H 8950 4800 50  0001 C CNN "DigiKey Part No."
+F 5 "T491A106K010AT" H 8950 4800 50  0001 C CNN "Mftr Part No."
+F 6 "Kemet" H 8950 4800 50  0001 C CNN "Manufacturer"
 	1    8950 4800
 	0    -1   -1   0
@@
 $EndComp
 $Comp
-L Name~Plate~Class~Library:TestPoint TP?
+L Name_Plate_Class_Project:TestPoint TP?
 U 1 1 5EB2B88E
 P 2850 2250
 AR Path="/5ECF32A9/5EB2B88E" Ref="TP?"  Part="1"
 AR Path="/5ECEA271/5EB2B88E" Ref="TP301"  Part="1"
+AR Path="/5EB2B88E" Ref="TP301"  Part="1"
 F 0 "TP301" H 2650 2550 50  0000 L CNN
 F 1 "Test Point" H 2650 2450 50  0001 L CNN
@@
 F 0 "C302" H 8350 2300 50  0000 L CNN
 F 1 "10uF" H 8350 2050 50  0000 L CNN
-F 2 "Name Plate Class Project:CAP_430X430N" H 8300 2200 50  0001 C CNN
+F 2 "Name_Plate_Class_Project:CAP_430X430N" H 8300 2200 50  0001 C CNN
 F 3 "https://media.digikey.com/pdf/Data%20Sheets/Panasonic%20Electronic%20Components/S_Series,Type_V_Rev2018.pdf" H 8300 2200 50  0001 C CNN
-F 4 "Panasonic EEE-1VA2R2NR" H 8300 2200 50  0001 C CNN "Field4"
-F 5 "399-11437-1-ND" H 8300 2200 50  0001 C CNN "DigiKey Part No."
-F 6 "T491A106K010AT" H 8300 2200 50  0001 C CNN "Mftr Part No."
-F 7 "" H 8300 2200 50  0001 C CNN "URL"
-F 8 "Kemet" H 8300 2200 50  0001 C CNN "Manufacturer"
+F 4 "399-11437-1-ND" H 8300 2200 50  0001 C CNN "DigiKey Part No."
+F 5 "T491A106K010AT" H 8300 2200 50  0001 C CNN "Mftr Part No."
+F 6 "Kemet" H 8300 2200 50  0001 C CNN "Manufacturer"
 	1    8300 2200
 	1    0    0    -1

Commit message: PCB Layout
Parts:
- C301, C302: footprint Name_Plate_Class_Project:CAP_430X430N -> Name_Plate_Class_Project:T491A106K010AT; DigiKey Part No. 399-11437-1-ND -> 399-3684-1-ND
- TP301: footprint Connector_Wire:SolderWirePad_1x01_SMD_5x10mm -> FrequentlyUsed:Pad_2.5-2.5
Connections:
- net ADDR_LED: no longer TP301.1
- net at D301.4 (DIN), R301.2: now also TP301.1
Other:
- moved on the sheet: R301, TP301
Changed lines of the file:
@@
 F 0 "C301" V 9202 4800 50  0000 C CNN
 F 1 "10uF" V 9111 4800 50  0000 C CNN
-F 2 "Name_Plate_Class_Project:CAP_430X430N" H 8950 4800 50  0001 C CNN
-F 3 "https://media.digikey.com/pdf/Data%20Sheets/Panasonic%20Electronic%20Components/S_Series,Type_V_Rev2018.pdf" H 8950 4800 50  0001 C CNN
-F 4 "399-11437-1-ND" H 8950 4800 50  0001 C CNN "DigiKey Part No."
+F 2 "Name_Plate_Class_Project:T491A106K010AT" H 8950 4800 50  0001 C CNN
+F 3 "https://content.kemet.com/datasheets/KEM_T2005_T491.pdf" H 8950 4800 50  0001 C CNN
+F 4 "399-3684-1-ND" H 8950 4800 50  0001 C CNN "DigiKey Part No."
 F 5 "T491A106K010AT" H 8950 4800 50  0001 C CNN "Mftr Part No."
 F 6 "Kemet" H 8950 4800 50  0001 C CNN "Manufacturer"
@@
 	8800 4800 8600 4800
 Wire Wire Line
-	3550 2250 3400 2250
+	3550 2250 3300 2250
 $Comp
 L Device:R R?
 U 1 1 5EB2ABF4
-P 3250 2250
+P 2900 2250
 AR Path="/5EB2ABF4" Ref="R?"  Part="1"
 AR Path="/5EAC05C2/5EB2ABF4" Ref="R?"  Part="1"
@@
 AR Path="/5ECF32A9/5EB2ABF4" Ref="R?"  Part="1"
 AR Path="/5ECEA271/5EB2ABF4" Ref="R301"  Part="1"
-F 0 "R301" V 3150 2350 50  0000 R CNN
-F 1 "22" V 3050 2350 50  0000 R CNN
-F 2 "Resistor_SMD:R_0603_1608Metric_Pad1.05x0.95mm_HandSolder" V 3180 2250 50  0001 C CNN
-F 3 "https://www.te.com/commerce/DocumentDelivery/DDEController?Action=srchrtrv&DocNm=1773204-3&DocType=DS&DocLang=English" H 3250 2250 50  0001 C CNN
-F 4 "TE Connectivity " H 3250 2250 50  0001 C CNN "Manufacturer"
-F 5 "CRGCQ0603J22R" H 3250 2250 50  0001 C CNN "Mftr Part No."
-F 6 "A130081CT-ND" H 3250 2250 50  0001 C CNN "DigiKey Part No."
-	1    3250 2250
+F 0 "R301" V 2800 2350 50  0000 R CNN
+F 1 "22" V 2700 2350 50  0000 R CNN
+F 2 "Resistor_SMD:R_0603_1608Metric_Pad1.05x0.95mm_HandSolder" V 2830 2250 50  0001 C CNN
+F 3 "https://www.te.com/commerce/DocumentDelivery/DDEController?Action=srchrtrv&DocNm=1773204-3&DocType=DS&DocLang=English" H 2900 2250 50  0001 C CNN
+F 4 "TE Connectivity " H 2900 2250 50  0001 C CNN "Manufacturer"
+F 5 "CRGCQ0603J22R" H 2900 2250 50  0001 C CNN "Mftr Part No."
+F 6 "A130081CT-ND" H 2900 2250 50  0001 C CNN "DigiKey Part No."
+	1    2900 2250
 	0    -1   -1   0
 $EndComp
@@
 L Name_Plate_Class_Project:TestPoint TP?
 U 1 1 5EB2B88E
-P 2850 2250
+P 3300 2250
 AR Path="/5ECF32A9/5EB2B88E" Ref="TP?"  Part="1"
 AR Path="/5ECEA271/5EB2B88E" Ref="TP301"  Part="1"
 AR Path="/5EB2B88E" Ref="TP301"  Part="1"
-F 0 "TP301" H 2650 2550 50  0000 L CNN
-F 1 "Test Point" H 2650 2450 50  0001 L CNN
-F 2 "Connector_Wire:SolderWirePad_1x01_SMD_5x10mm" H 3050 2250 50  0001 C CNN
-F 3 "None" H 3050 2250 50  0001 C CNN
-F 4 "TP_ADDR_LED" H 2650 2450 50  0000 L CNN "Name"
-F 5 "None" H 2850 2250 50  0001 C CNN "DigiKey Part No."
-F 6 "None" H 2850 2250 50  0001 C CNN "Manufacturer"
-F 7 "None" H 2850 2250 50  0001 C CNN "Mftr Part No."
-	1    2850 2250
-	1    0    0    -1
-$EndComp
-Wire Wire Line
-	3100 2250 2850 2250
-Wire Wire Line
-	2850 2250 2550 2250
-Connection ~ 2850 2250
+F 0 "TP301" H 3100 2550 50  0000 L CNN
+F 1 "Test Point" H 3100 2450 50  0001 L CNN
+F 2 "FrequentlyUsed:Pad_2.5-2.5" H 3500 2250 50  0001 C CNN
+F 3 "None" H 3500 2250 50  0001 C CNN
+F 4 "TP_ADDR_LED" H 3100 2450 50  0000 L CNN "Name"
+F 5 "None" H 3300 2250 50  0001 C CNN "DigiKey Part No."
+F 6 "None" H 3300 2250 50  0001 C CNN "Manufacturer"
+F 7 "None" H 3300 2250 50  0001 C CNN "Mftr Part No."
+	1    3300 2250
+	1    0    0    -1
+$EndComp
 Wire Wire Line
 	3850 1950 3850 1750
@@
 	3850 1550 5000 1550
 Wire Wire Line
-	8300 1550 8300 1400
+	8400 1550 8400 1450
 Connection ~ 7800 2850
 NoConn ~ 7600 2250
@@
 L power:+5V #PWR0101
 U 1 1 5EB43851
-P 8300 1400
-F 0 "#PWR0101" H 8300 1250 50  0001 C CNN
-F 1 "+5V" H 8315 1573 50  0000 C CNN
-F 2 "" H 8300 1400 50  0001 C CNN
-F 3 "" H 8300 1400 50  0001 C CNN
-	1    8300 1400
+P 8400 1450
+F 0 "#PWR0101" H 8400 1300 50  0001 C CNN
+F 1 "+5V" H 8415 1623 50  0000 C CNN
+F 2 "" H 8400 1450 50  0001 C CNN
+F 3 "" H 8400 1450 50  0001 C CNN
+	1    8400 1450
 	1    0    0    -1
 $EndComp
@@
 L power:GND #PWR0102
 U 1 1 5EB44FF3
-P 8300 3050
-F 0 "#PWR0102" H 8300 2800 50  0001 C CNN
-F 1 "GND" H 8305 2877 50  0000 C CNN
-F 2 "" H 8300 3050 50  0001 C CNN
-F 3 "" H 8300 3050 50  0001 C CNN
-	1    8300 3050
+P 8400 2950
+F 0 "#PWR0102" H 8400 2700 50  0001 C CNN
+F 1 "GND" H 8405 2777 50  0000 C CNN
+F 2 "" H 8400 2950 50  0001 C CNN
+F 3 "" H 8400 2950 50  0001 C CNN
+	1    8400 2950
 	1    0    0    -1
 $EndComp
@@
 	1    0    0    -1
 $EndComp
-Connection ~ 8300 1550
 Connection ~ 6150 2850
 Connection ~ 5500 2850
@@
 	5500 2850 6150 2850
 Wire Wire Line
-	8300 2850 8300 3050
-Connection ~ 8300 2850
+	8400 2850 8400 2950
 Text Notes 5350 3400 0    98   ~ 20
 2812 LEDs
@@
 F 0 "C302" H 8350 2300 50  0000 L CNN
 F 1 "10uF" H 8350 2050 50  0000 L CNN
-F 2 "Name_Plate_Class_Project:CAP_430X430N" H 8300 2200 50  0001 C CNN
-F 3 "https://media.digikey.com/pdf/Data%20Sheets/Panasonic%20Electronic%20Components/S_Series,Type_V_Rev2018.pdf" H 8300 2200 50  0001 C CNN
-F 4 "399-11437-1-ND" H 8300 2200 50  0001 C CNN "DigiKey Part No."
+F 2 "Name_Plate_Class_Project:T491A106K010AT" H 8300 2200 50  0001 C CNN
+F 3 "https://content.kemet.com/datasheets/KEM_T2005_T491.pdf" H 8300 2200 50  0001 C CNN
+F 4 "399-3684-1-ND" H 8300 2200 50  0001 C CNN "DigiKey Part No."
 F 5 "T491A106K010AT" H 8300 2200 50  0001 C CNN "Mftr Part No."
 F 6 "Kemet" H 8300 2200 50  0001 C CNN "Manufacturer"
@@
 	1    0    0    -1
 $EndComp
+Text Label 7900 1550 0    50   ~ 0
+LEDVCC
+Text Label 7900 2850 0    50   ~ 0
+LEDGND
+Connection ~ 8300 1550
+Connection ~ 8300 2850
+Wire Wire Line
+	8300 2850 8400 2850
+Wire Wire Line
+	8300 1550 8400 1550
+Connection ~ 3300 2250
+Wire Wire Line
+	3300 2250 3050 2250
+Wire Wire Line
+	2550 2250 2750 2250
 $EndSCHEMATC

Commit message: Final Design Files
Final design files as submitted.
Parts:
- D301, D302, D303, D304: DigiKey Part No. (none) -> 1528-2388-ND; Manufacturer (none) -> Adafruit Industries LLC; Mftr Part No. (none) -> 3094
- LS301: DigiKey Part No. 668-1136-ND -> 668-1448-ND; Mftr Part No. AST-03008MR-R -> AB1541B-LW100-R
Changed lines of the file:
@@
 F 1 "Piezo Buzzer" H 9500 4850 50  0000 L CNN
 F 2 "Name_Plate_Class_Project:Buzzer_TDK_PS1240P02BT_D12.2mm_H6.5mm" V 9325 5000 50  0001 C CNN
-F 3 "http://www.puiaudio.com/pdf/AST-03008MR-R.pdf" V 9325 5000 50  0001 C CNN
-F 4 "668-1136-ND" H 9350 4900 50  0001 C CNN "DigiKey Part No."
+F 3 "http://www.puiaudio.com/pdf/AB1541B-LW100-R.pdf" V 9325 5000 50  0001 C CNN
+F 4 "668-1448-ND" H 9350 4900 50  0001 C CNN "DigiKey Part No."
 F 5 "Pui Audio" H 9350 4900 50  0001 C CNN "Manufacturer"
-F 6 "AST-03008MR-R" H 9350 4900 50  0001 C CNN "Mftr Part No."
+F 6 "AB1541B-LW100-R" H 9350 4900 50  0001 C CNN "Mftr Part No."
 	1    9350 4900
 	1    0    0    -1
@@
 F 1 "WS2812B" H 5100 2550 50  0000 L CNN
 F 2 "LED_SMD:LED_WS2812B_PLCC4_5.0x5.0mm_P3.2mm" H 5050 1950 50  0001 L TNN
-F 3 "https://cdn-shop.adafruit.com/datasheets/WS2812B.pdf" H 5100 1875 50  0001 L TNN
+F 3 "https://cdn-shop.adafruit.com/product-files/1138/SK6812+LED+datasheet+.pdf" H 5100 1875 50  0001 L TNN
+F 4 "1528-2388-ND" H 5000 2250 50  0001 C CNN "DigiKey Part No."
+F 5 "Adafruit Industries LLC" H 5000 2250 50  0001 C CNN "Manufacturer"
+F 6 "3094" H 5000 2250 50  0001 C CNN "Mftr Part No."
 	1    5000 2250
 	1    0    0    -1
@@
 F 1 "WS2812B" H 6250 2550 50  0000 L CNN
 F 2 "LED_SMD:LED_WS2812B_PLCC4_5.0x5.0mm_P3.2mm" H 6200 1950 50  0001 L TNN
-F 3 "https://cdn-shop.adafruit.com/datasheets/WS2812B.pdf" H 6250 1875 50  0001 L TNN
+F 3 "https://cdn-shop.adafruit.com/product-files/1138/SK6812+LED+datasheet+.pdf" H 6250 1875 50  0001 L TNN
+F 4 "1528-2388-ND" H 6150 2250 50  0001 C CNN "DigiKey Part No."
+F 5 "Adafruit Industries LLC" H 6150 2250 50  0001 C CNN "Manufacturer"
+F 6 "3094" H 6150 2250 50  0001 C CNN "Mftr Part No."
 	1    6150 2250
 	1    0    0    -1
@@
 F 1 "WS2812B" H 7400 2550 50  0000 L CNN
 F 2 "LED_SMD:LED_WS2812B_PLCC4_5.0x5.0mm_P3.2mm" H 7350 1950 50  0001 L TNN
-F 3 "https://cdn-shop.adafruit.com/datasheets/WS2812B.pdf" H 7400 1875 50  0001 L TNN
+F 3 "https://cdn-shop.adafruit.com/product-files/1138/SK6812+LED+datasheet+.pdf" H 7400 1875 50  0001 L TNN
+F 4 "1528-2388-ND" H 7300 2250 50  0001 C CNN "DigiKey Part No."
+F 5 "Adafruit Industries LLC" H 7300 2250 50  0001 C CNN "Manufacturer"
+F 6 "3094" H 7300 2250 50  0001 C CNN "Mftr Part No."
 	1    7300 2250
 	1    0    0    -1
@@
 F 1 "WS2812B" H 3950 2550 50  0000 L CNN
 F 2 "LED_SMD:LED_WS2812B_PLCC4_5.0x5.0mm_P3.2mm" H 3900 1950 50  0001 L TNN
-F 3 "https://cdn-shop.adafruit.com/datasheets/WS2812B.pdf" H 3950 1875 50  0001 L TNN
+F 3 "https://cdn-shop.adafruit.com/product-files/1138/SK6812+LED+datasheet+.pdf" H 3950 1875 50  0001 L TNN
+F 4 "1528-2388-ND" H 3850 2250 50  0001 C CNN "DigiKey Part No."
+F 5 "Adafruit Industries LLC" H 3850 2250 50  0001 C CNN "Manufacturer"
+F 6 "3094" H 3850 2250 50  0001 C CNN "Mftr Part No."
 	1    3850 2250
 	1    0    0    -1
